File: nixie-clock/nixie-clock.kicad_pcb (KiCad board)
At the start: 2 copper layers, 69 parts, among them J1 Barrel_Jack, J2 Conn_01x02, J3 Conn_01x02, Q1 2N7002, Q2 2N7002, Q3 2N7002, Q4 2N7002, Q5 2N7002, Q6 Q_Photo_NPN, Q7 PSMN014-80YL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

Commit message: Top layer ground plane and stitching
Parts:
- added G***: LOGO, custom-parts:ProjectName125-800, F.Cu at (350.1, 207.9)
- added G***: LOGO, custom-parts:VersionString125-800, F.Cu at (399.1, 208.0)
- added J4: Conn_01x01_MountingPin, custom-parts:4MM_Mounting_Hole, F.Cu at (162.9, 207.9)
- added J5: Conn_01x01_MountingPin, custom-parts:4MM_Mounting_Hole, F.Cu at (446.9, 167.9)
- added J6: Conn_01x01_MountingPin, custom-parts:4MM_Mounting_Hole, F.Cu at (446.9, 207.9)
- added J7: Conn_01x01_MountingPin, custom-parts:4MM_Mounting_Hole, F.Cu at (162.9, 167.9)
- added J8: Conn_01x01_MountingPin, custom-parts:4MM_Mounting_Hole, F.Cu at (304.9, 179.1)
- U6: footprint Package_SO:SOIC-16W_7.5x10.3mm_P1.27mm -> Package_SO:SO-8_5.3x6.2mm_P1.27mm
- moved C9 165.4 mm to (220.7, 202.6), turned to 270 degrees
- moved C4 165.0 mm to (389.7, 203.1), turned to 90 degrees
- moved U5 160.4 mm to (225.3, 200.5), turned to 90 degrees
- moved U7 159.5 mm to (385.0, 201.1), turned to 90 degrees
- moved C15 154.6 mm to (380.3, 203.2), turned to 270 degrees
- moved C14 151.5 mm to (230.0, 202.6), turned to 90 degrees
- moved R23 81.4 mm to (403.4, 201.4), turned to 180 degrees
- moved V1 80.0 mm to (207.4, 187.9)
- moved V6 80.0 mm to (402.4, 187.9)
- moved R18 79.2 mm to (208.4, 201.5), turned to 180 degrees
- moved J1 49.5 mm to (264.8, 198.6)
- moved R4 47.9 mm to (273.6, 178.6)
- moved Q4 45.9 mm to (273.6, 175.8), turned to 270 degrees
- moved R20 45.9 mm to (288.4, 201.5), turned to 180 degrees
- moved V3 45.0 mm to (287.4, 187.9)
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Connections:
- R8 pad 2: /RTL_SDA -> /RTC_SDA
- U1 pad 37: /RTC_INT -> Net-(U1-Pad37)
- U1 pad 39: (no net) -> GND
- U1 pad 9: Net-(U1-Pad9) -> /RTC_INT
- U2 pad 28: Net-(Q1-Pad3) -> Net-(Q2-Pad3)
- U2 pad 32: Net-(Q2-Pad3) -> Net-(Q1-Pad3)
- U3 pad 28: Net-(Q1-Pad3) -> Net-(Q2-Pad3)
- U6 pad 2: +3V3 -> GND
- U6 pad 4: /RTL_RST -> /RTC_RST
- U6 pad 6: GND -> +3V3
- U6 pad 7: GND -> /RTC_SDA
- U6 pad 8: GND -> /RTC_SCL
Routing:
- net /HVDIS: track 0.00 -> 270.1 mm
- net +170V: track 0.00 -> 255.4 mm, vias 0 -> 30
- net +5V: track 0.00 -> 218.7 mm, vias 0 -> 19
- net +3V3: track 0.00 -> 189.4 mm, vias 0 -> 2
- net Net-(C7-Pad1): track 0.00 -> 151.7 mm, vias 0 -> 4
- net Net-(U3-Pad12): track 0.00 -> 144.1 mm
- net Net-(U3-Pad11): track 0.00 -> 144.0 mm
- net Net-(U2-Pad43): track 0.00 -> 132.8 mm
- net Net-(U2-Pad44): track 0.00 -> 130.3 mm
- net Net-(U3-Pad13): track 0.00 -> 120.4 mm
- net /SCLK: track 0.00 -> 113.4 mm
- net Net-(U2-Pad42): track 0.00 -> 108.6 mm
- net Net-(Q3-Pad3): track 0.00 -> 106.7 mm, vias 0 -> 4
- net /POL: track 0.00 -> 101.9 mm
- net /MOSI: track 0.00 -> 100.0 mm
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- added copper zone on F.Cu, net +170V
- added copper zone on B.Cu, net GND
- added copper zone on F.Cu, net GND
- added copper zone on F.Cu, net Net-(C11-Pad1)
- added copper zone on F.Cu, net Net-(C2-Pad1)
- added copper zone on F.Cu, net Net-(C5-Pad1)
- added copper zone on F.Cu, net Net-(C5-Pad2)
- added copper zone on F.Cu, net Net-(C6-Pad1)
- added copper zone on F.Cu, net Net-(D1-Pad1)
- added copper zone on F.Cu, net Net-(D2-Pad2)
- added copper zone on F.Cu, net Net-(D3-Pad1)
- added copper zone on F.Cu, net Net-(Q7-Pad1)
- added copper zone on F.Cu, net Net-(Q7-Pad4)
- added copper zone on F.Cu, net VDD
Other:
- board outline added: 294.1 x 50 mm
- net class +170V added: clearance 0.4, trace_width 0.29, via_dia 0.8, via_drill 0.4
- net class Default: trace_width 0.25 -> 0.29
