File: nixie-clock/nixie-clock.sch (KiCad schematic (older format))
At the start: 72 parts, among them J1 Barrel_Jack, J2 Conn_01x02, J3 Conn_01x02, J4 Conn_01x01_MountingPin, J5 Conn_01x01_MountingPin, J6 Conn_01x01_MountingPin, J7 Conn_01x01_MountingPin, J8 Conn_01x01_MountingPin, Q1 2N7002, Q2 2N7002, Q3 2N7002, Q4 2N7002, Q5 2N7002, Q6 Q_Photo_NPN, Q7 BUK7Y9R9-80EX, T1 NA5920-AL, U1 ESP32-WROOM-32D, U2 HV5523, U3 HV5523, U4 TPS40210, U5 LDL1117, U6 DS3231M, U7 LDL1117

Commit message: Tweak couple things before sending to fab
Parts:
- U2, U3: footprint Package_DFN_QFN:QFN-44-1EP_7x7mm_P0.5mm_EP5.15x5.15mm -> Package_DFN_QFN:QFN-44-1EP_7x7mm_P0.5mm_EP5.15x5.15mm_ThermalVias
Changed lines of the file:
@@
 F 0 "U2" H 9000 5300 50  0000 C CNN
 F 1 "HV5523" H 9100 5200 50  0000 C CNN
-F 2 "Package_DFN_QFN:QFN-44-1EP_7x7mm_P0.5mm_EP5.15x5.15mm" H 9450 4100 50  0001 C CNN
+F 2 "Package_DFN_QFN:QFN-44-1EP_7x7mm_P0.5mm_EP5.15x5.15mm_ThermalVias" H 9450 4100 50  0001 C CNN
 F 3 "" H 9450 4100 50  0001 C CNN
 	1    9450 3150
@@
 F 0 "U3" H 9000 10450 50  0000 C CNN
 F 1 "HV5523" H 9100 10350 50  0000 C CNN
-F 2 "Package_DFN_QFN:QFN-44-1EP_7x7mm_P0.5mm_EP5.15x5.15mm" H 9450 9250 50  0001 C CNN
+F 2 "Package_DFN_QFN:QFN-44-1EP_7x7mm_P0.5mm_EP5.15x5.15mm_ThermalVias" H 9450 9250 50  0001 C CNN
 F 3 "" H 9450 9250 50  0001 C CNN
 	1    9450 8300

Commit message: Fixes from v1.0
Parts:
- removed J2, J3: Conn_01x02, Connector_PinHeader_1.00mm:PinHeader_1x02_P1.00mm_Vertical, symbol Connector_Generic:Conn_01x02
- removed Q1, Q2, Q3, Q4, Q5: 2N7002, Package_TO_SOT_SMD:SOT-23, symbol Transistor_FET:2N7002
- removed R1, R2, R3, R4, R5: 10K, Resistor_SMD:R_0805_2012Metric_Pad1.15x1.40mm_HandSolder, symbol Device:R
- added C1: 100uF, Capacitor_SMD:C_0805_2012Metric_Pad1.15x1.40mm_HandSolder, symbol Device:C
- added C16, C17, C19: 0.1uF, symbol Device:C_Small
- added C18: 4.7uF, symbol Device:C_Small
- added J2: USB_B_Mini, custom-parts:54819-0589, symbol Connector:USB_B_Mini
- added R12: 22.1K, symbol Device:R_Small
- added R13: 47.5K, symbol Device:R_Small
- added R14: 1K, symbol Device:R_Small
- added R6: 10K, symbol Device:R_Small
- added U6: TXB0108PWR, Package_SO:TSSOP-20_4.4x6.5mm_P0.65mm, symbol Logic_LevelTranslator:TXS0108EPW
- added U7: CP2102N-A01-GQFN24, Package_DFN_QFN:QFN-24-1EP_4x4mm_P0.5mm_EP2.6x2.6mm, symbol Interface_USB:CP2102N-A01-GQFN24
- C2: renamed from C1; value 10uF -> 1uF
- R17: renamed from R18; value 3.3k -> 7.3k
- R18: renamed from R19; value 3.3k -> 7.3k
- R19: renamed from R20; value 3.3k -> 7.3k
- R20: renamed from R21; value 3.3k -> 7.3k
- R21: renamed from R22; value 3.3k -> 7.3k
- R22: renamed from R23; value 3.3k -> 7.3k
- U4: renamed from U6; footprint Package_SO:SO-8_5.3x6.2mm_P1.27mm -> Package_SO:SOIC-8_3.9x4.9mm_P1.27mm
- renumbered C9 to C10, C10 to C11, C11 to C12, C12 to C13, C13 to C14, C14 to C15, C15 to C20, C16 to C21, C17 to C22, C18 to C23, C19 to C24, C2 to C3, C3 to C4, C4 to C5, C5 to C6, C6 to C7, C7 to C8, C8 to C9, D3 to D1, J4 to J3, J5 to J4, J6 to J5, J7 to J6, J8 to J7, Q6 to Q1, Q7 to Q2, R6 to R1, R14 to R10, R15 to R11, R16 to R15, R17 to R16, R7 to R2, R8 to R3, R9 to R4, R10 to R5, R11 to R7, R12 to R8, R13 to R9, U4 to U2, U5 to U3, U7 to U5, U2 to U8, U3 to U9
Connections:
- net +3V3: now also C1.1, C16.1, C17.1, C18.1, R14.1, R6.2, U6.10 (OE), U6.2 (VCCA), U7.5 (VIO), U7.6 (VDD), U7.7 (REGIN)
- net +5V: now also C19.2, U6.19 (VCCB)
- net BL: now also U6.6 (A5)
- net GND: now also C1.2, C16.2, C17.2, C18.2, C19.1, J2.5 (GND), J2.6 (Shield), R13.2, U6.11 (GND), U7.2 (GND), U7.25 (GND)
- net HVDIS: now also R6.1
- net LE: now also U6.4 (A3)
- net MOSI: now also U6.1 (A1)
- net POL: now also U6.5 (A4)
- net SCLK: now also U6.3 (A2)
- net BOOT_MODE: now reaches U1.25 (IO0)
- net BOOT_MODE: now also U7.23 (DTR)
- net ESP_EN: now reaches R2.2, U1.3 (EN)
- net ESP_EN: now also U7.19 (RTS)
- net RX: now reaches U1.34 (RXD0/IO3)
- net RX: now also U7.21 (TXD)
- net TX: now reaches U1.35 (TXD0/IO1)
- net TX: now also U7.20 (RXD)
- net at U8.27 (~POL), U9.27 (~POL): now also U6.16 (B4)
- net at U8.28 (CLK), U9.28 (CLK): now also U6.18 (B2)
- net at U8.31 (~LE), U9.31 (~LE): now also U6.17 (B3)
- net at U8.32 (DATA_IN): now also U6.20 (B1)
- net at U8.33 (~BL), U9.33 (~BL): now also U6.15 (B5)
- new net: J2.3 (D+), U7.3 (D+)
- new net: J2.2 (D-), U7.4 (D-)
- new net: R12.2, R13.1, U7.8 (VBUS)
- new net: R14.2, U7.9 (~RSTb)
- new net: J2.1 (VBUS), R12.1

Commit message: Annotate remaining footprints
Parts:
- C16, C17, C18, C19: footprint (none) -> Capacitor_SMD:C_0805_2012Metric_Pad1.15x1.40mm_HandSolder
- R12, R13, R14, R6: footprint (none) -> Resistor_SMD:R_0805_2012Metric_Pad1.15x1.40mm_HandSolder
Changed lines of the file:
@@
 F 0 "C19" V 5721 1550 50  0000 C CNN
 F 1 "0.1uF" V 5812 1550 50  0000 C CNN
-F 2 "" H 5950 1550 50  0001 C CNN
+F 2 "Capacitor_SMD:C_0805_2012Metric_Pad1.15x1.40mm_HandSolder" H 5950 1550 50  0001 C CNN
 F 3 "~" H 5950 1550 50  0001 C CNN
 	1    5950 1550
@@
 F 0 "C16" V 4571 1550 50  0000 C CNN
 F 1 "0.1uF" V 4662 1550 50  0000 C CNN
-F 2 "" H 4800 1550 50  0001 C CNN
+F 2 "Capacitor_SMD:C_0805_2012Metric_Pad1.15x1.40mm_HandSolder" H 4800 1550 50  0001 C CNN
 F 3 "~" H 4800 1550 50  0001 C CNN
 	1    4800 1550
@@
 F 0 "R6" H 2959 2696 50  0000 L CNN
 F 1 "10K" H 2959 2605 50  0000 L CNN
-F 2 "" H 2900 2650 50  0001 C CNN
+F 2 "Resistor_SMD:R_0805_2012Metric_Pad1.15x1.40mm_HandSolder" H 2900 2650 50  0001 C CNN
 F 3 "~" H 2900 2650 50  0001 C CNN
 	1    2900 2650
@@
 F 0 "R14" H 6059 7396 50  0000 L CNN
 F 1 "1K" H 6059 7305 50  0000 L CNN
-F 2 "" H 6000 7350 50  0001 C CNN
+F 2 "Resistor_SMD:R_0805_2012Metric_Pad1.15x1.40mm_HandSolder" H 6000 7350 50  0001 C CNN
 F 3 "~" H 6000 7350 50  0001 C CNN
 	1    6000 7350
@@
 F 0 "C18" H 5342 7646 50  0000 L CNN
 F 1 "4.7uF" H 5342 7555 50  0000 L CNN
-F 2 "" H 5250 7600 50  0001 C CNN
+F 2 "Capacitor_SMD:C_0805_2012Metric_Pad1.15x1.40mm_HandSolder" H 5250 7600 50  0001 C CNN
 F 3 "~" H 5250 7600 50  0001 C CNN
 	1    5250 7600
@@
 F 0 "C17" H 4892 7646 50  0000 L CNN
 F 1 "0.1uF" H 4892 7555 50  0000 L CNN
-F 2 "" H 4800 7600 50  0001 C CNN
+F 2 "Capacitor_SMD:C_0805_2012Metric_Pad1.15x1.40mm_HandSolder" H 4800 7600 50  0001 C CNN
 F 3 "~" H 4800 7600 50  0001 C CNN
 	1    4800 7600
@@
 F 0 "R12" H 5309 8146 50  0000 L CNN
 F 1 "22.1K" H 5309 8055 50  0000 L CNN
-F 2 "" H 5250 8100 50  0001 C CNN
+F 2 "Resistor_SMD:R_0805_2012Metric_Pad1.15x1.40mm_HandSolder" H 5250 8100 50  0001 C CNN
 F 3 "~" H 5250 8100 50  0001 C CNN
 	1    5250 8100
@@
 F 0 "R13" H 5309 8446 50  0000 L CNN
 F 1 "47.5K" H 5309 8355 50  0000 L CNN
-F 2 "" H 5250 8400 50  0001 C CNN
+F 2 "Resistor_SMD:R_0805_2012Metric_Pad1.15x1.40mm_HandSolder" H 5250 8400 50  0001 C CNN
 F 3 "~" H 5250 8400 50  0001 C CNN
 	1    5250 8400

Commit message: Fix footprint in schematic
Parts:
- C1: footprint Capacitor_SMD:C_0805_2012Metric_Pad1.15x1.40mm_HandSolder -> Capacitor_SMD:C_1206_3216Metric_Pad1.42x1.75mm_HandSolder
Changed lines of the file:
@@
 F 0 "C1" H 765 2796 50  0000 L CNN
 F 1 "100uF" H 765 2705 50  0000 L CNN
-F 2 "Capacitor_SMD:C_0805_2012Metric_Pad1.15x1.40mm_HandSolder" H 688 2600 50  0001 C CNN
+F 2 "Capacitor_SMD:C_1206_3216Metric_Pad1.42x1.75mm_HandSolder" H 688 2600 50  0001 C CNN
 F 3 "~" H 650 2750 50  0001 C CNN
 	1    650  2750
