File: davis-receiver/davis-receiver.sch (KiCad schematic (older format))
At the start: 48 parts, among them U1 TM4C129ENCZADI3R, U2 CC1125RHBR, U3 FXPS7115D4

Commit message: Davis Receiver RF Trans Captured
Parts:
- added C? (x3): 10nF, symbol Device:C
- added C?: 2.2uF, symbol Device:C
- added C? (x2): 100nF, symbol Device:C
- added C?: 22pF, symbol Device:C
- added C? (x11): 47nF, symbol Device:C
- added C?: 1.8nF, symbol Device:C
- added C? (x2): 3.3pF, symbol Device:C
- added C?: 15pF, symbol Device:C
- added C?: 1pF, symbol Device:C
- added C?: 2.2pF, symbol Device:C
- added C?: 3pF, symbol Device:C
- added C?: 33pF, symbol Device:C
- added C?: 100pF, symbol Device:C
- added C?: 220nF, symbol Device:C
- added J?: Conn_Coaxial, symbol Connector:Conn_Coaxial
- added L?: 15nH, symbol Device:L
- added L? (x4): 12nH, symbol Device:L
- added L?: 10nH, symbol Device:L
- added L?: 7.5nH, symbol Device:L
- added L?: 18nH, symbol Device:L
- added R?: 10, symbol Device:R
- added R?: 56K, symbol Device:R
- added U?: TPS79930DDCR, Custom:SOT-23-Thin-5, symbol Custom:TPS79930
- added X?: ECS-2520MV-400-AY-TR, Oscillator:Oscillator_SMD_ECS_2520MV-xxx-xx-4Pin_2.5x2.0mm, symbol Oscillator:ECS-2520MV-xxx-xx
Connections:
- net +3V3: now also C?.1, U?.1 (IN), U?.3 (EN)
- net GND: now also U2.30 (XOSC_Q1), U2.33 (EPAD), C?.1, C?.1, C?.1, C?.1, C?.1, C?.2, C?.2, C?.2, C?.2, C?.2, C?.2, C?.2, C?.2, C?.2, C?.2, C?.2, C?.2, C?.2, C?.2, C?.2, C?.2, J?.2 (Ext), L?.2, R?.2, U?.2 (GND), X?.2 (GND)
- net +3V0: now reaches U2.1 (VDD_GUARD)
- net +3V0: now also U2.12 (DVDD), U2.13 (AVDD_IF), U2.15 (AVDD_RF), U2.22 (AVDD_SYNTH1), U2.25 (AVDD_PFD_CHP), U2.27 (AVDD_SYNTH2), U2.28 (AVDD_XOSC), U2.5 (DVDD), C?.1, C?.1, C?.1, C?.1, C?.1, C?.1, C?.1, C?.1, C?.1, C?.1, C?.2, C?.2, C?.2, C?.2, R?.2, U?.5 (OUT), X?.4 (VDD)
- net RF_GPIO0: now reaches U2.10 (GPIO0)
- net RF_CS: now reaches U2.11 (CSN)
- net at U2.14 (RBIAS): now also R?.1
- net at U2.17 (PA): now also C?.1, L?.1
- net at U2.18 (TRX_SW): now also C?.1, L?.2
- net at U2.19 (LNA_P): now also C?.1, L?.1, L?.2
- net RF_RESET: now reaches U2.2 (RESET_N)
- net at U2.20 (LNA_N): now also C?.1, L?.1, L?.1
- net at U2.21 (DCPL_VCO): now also C?.1
- net at U2.23 (LPF0): now also C?.2
- net at U2.24 (LPF1): now also C?.1
- net at U2.26 (DCPL_PFD_CHP): now also C?.2
- net at U2.29 (DCPL_XOSC): now also C?.2
- net RF_GPIO3: now reaches U2.3 (GPIO3)
- net at U2.32 (EXT_XOSC): now also C?.2
- net RF_GPIO2: now reaches U2.4 (GPIO2)
- net at U2.6 (DCPL): now also C?.1
- net RF_SI: now reaches U2.7 (SI)
- net RF_SCLK: now reaches U2.8 (SCLK)
- net RF_SO_GPIO1: now reaches U2.9 (SOGPIO1)
- new net: J?.1 (In), L?.2
- new net: C?.1, U?.4 (NR)
- new net: C?.1, X?.3 (OUT)
- new net: C?.2, L?.1, L?.2
- new net: C?.1, L?.2, R?.1
- new net: C?.1, C?.2, L?.1
- new net: C?.2, C?.2, L?.1, L?.2
- new net: C?.1, L?.1, L?.2
Other:
- note added: "RF Tranceiver"
- moved on the sheet: D1, U2

Commit message: Davis Receiver Captures
More capture for the Davis receiver.
Parts:
- added C? (x5): 100nF, symbol Device:C
- added C? (x16): 0.1uF, symbol Device:C
- added C? (x2): 1uF, symbol Device:C
- added C?: 2.2uF, symbol Device:C
- added C?: 01.uF, symbol Device:C
- added C? (x2): 22pF, symbol Device:C
- added R?: 4.87K, symbol Device:R
- added R? (x4): 49.9, symbol Device:R
- added R? (x2): 330, symbol Device:R
- added R?: 51, symbol Device:R
- added R?: 10K, symbol Device:R
- added R? (x4): 100, symbol Device:R
- added SW?: MCU_RESET, symbol Switch:SW_Push
- added Y?: LFXTAL071758CUTT, symbol Device:Crystal_GND24
Connections:
- net RF_SI is gone; now on net RF_MOSI: U2.7 (SI)
- net RF_SO_GPIO1 is gone; now on net RF_MISO: U2.9 (SOGPIO1)
- net +3V3: now also D1.1 (A), J?.3 (CT), U3.1 (VCC), U3.13 (VCCIO), U3.16 (VCC), C?.1, C?.1, C?.1, C?.1, C?.1, C?.1, C?.1, C?.1, C?.1, C?.1, C?.1, C?.1, C?.1, C?.1, C?.1, C?.1, C?.1, C?.1, C?.2, C?.2, R?.1, R?.1, R?.1, R?.1, R?.1, R?.1
- net GND: now also J?.SHD (Sheild), U1.E19 (OSC0), U1.U18 (WAKE_N), U3.15 (VSS), U3.17 (VSS), U3.4 (VSS), C?.1, C?.1, C?.2, C?.2, C?.2, C?.2, C?.2, C?.2, C?.2, C?.2, C?.2, C?.2, C?.2, C?.2, C?.2, C?.2, C?.2, C?.2, C?.2, C?.2, C?.2, C?.2, C?.2, C?.2, C?.2, C?.2, C?.2, R?.2, R?.2, R?.2, SW?.1, Y?.2, Y?.4
- net PairOneNeg: now also J?.8 (V1-)
- net PairOnePos: now also J?.7 (V1+)
- net PairTwoNeg: now also J?.10 (V2-)
- net PairTwoPos: now also J?.9 (V2+)
- net RF_CS: now also U1.C6 (PB4)
- net RF_GPIO0: now also U1.E3 (PQ0)
- net RF_GPIO2: now also U1.E2 (PQ1)
- net RF_GPIO3: now also U1.H4 (PQ2)
- net RF_RESET: now also U1.M4 (PQ3)
- net RF_SCLK: now also U1.B6 (PB5)
- net RF_MOSI: now reaches U1.A5 (PE4)
- net RF_MISO: now reaches U1.B5 (PE5)
- net BAR_INT: now reaches U1.C2 (PD0)
- net BAR_INT: now also U3.3 (INT)
- net BAR_SCLK: now reaches U1.T6 (PA2)
- net BAR_SCLK: now also U3.9 (SCLK/SCL)
- net BAR_CS: now reaches U1.U5 (PA3)
- net BAR_CS: now also U3.8 (SS_B)
- net ETH_LED1: now reaches U1.U6 (PF0)
- net ETH_LED1: now also J?.11 (LED1)
- net UART_RX: now reaches U1.V3 (PA0)
- net BAR_MOSI: now reaches U1.V4 (PA4)
- net BAR_MOSI: now also U3.10 (MOSI)
- net ETH_LED3: now reaches U1.V7 (PF4)
- net ETH_LED3: now also J?.13 (LED3)
- net UART_TX: now reaches U1.W3 (PA1)
- net BAR_MISO: now reaches U1.W4 (PA5)
- net BAR_MISO: now also U3.11 (MISO/SDA)
- net at U1.P18 (RST_N): now also C?.1, R?.1, R?.2
- net at U1.T18 (XOSC0): now also C?.1, Y?.1
- net at U1.T19 (XOSC1): now also C?.1, Y?.3
- net at U1.V13 (EN0RXIN): now also J?.5 (RD-), R?.2
- net at U1.V14 (EN0TXON): now also J?.2 (TD-), R?.2
- net at U1.V15 (EN0TXOP): now also J?.1 (TD+), R?.2
- net at U1.W13 (EN0RXIP): now also J?.4 (RD+), R?.2
- net at U1.W15 (RBIAS): now also R?.1
- net IND_G: now reaches U1.N2 (PR2)
- net IND_G: now also R?.2
- net IND_R: now reaches U1.N5 (PR0)
- net IND_R: now also R?.2
- net IND_B: now reaches U1.P3 (PR4)
- net IND_B: now also R?.2
- net at U1.E10 (VDDC): now also U1.H16 (VDDC), C?.1, C?.1, C?.1
- net at U1.P19 (VBAT): now also C?.1, R?.2
- net at D1.2 (BK): now also R?.1
- net at D1.3 (GK): now also R?.1
- net at D1.4 (RK): now also R?.1
- net ETH_LED2: now reaches J?.12 (LED2)
- net ETH_LED2: now also R?.1
- net ETH_LED4: now reaches J?.14 (LED4)
- net ETH_LED4: now also R?.1
- new net: R?.2, SW?.2
Other:
- note added: "BAROMETER"
- note added: "uC - XTAL / E-NET"
- note added: "uC Power"
- moved on the sheet: D1, J?, U1A, U1B, U1C, U1D, U3

Commit message: Davis Receiver Capture Complete
Captured the rest of the Davis Receiver schematic. Captured all necessary footprints. Assigned all footprints. Onto PCB layout...
Parts:
- added J3: JTAG, Custom:TC2050-IDC-FP, symbol Custom:TC-2050-Cortex-JTAG
- added J4: UART, Custom:TC2030-IDC-FP, symbol Custom:TC2030-UART
- added J5: SPI-BARO, Custom:TC2030-IDC-FP, symbol Custom:TC2030-GPIO
- added J6: SPI-RF, Custom:TC2030-IDC-FP, symbol Custom:TC2030-GPIO
- added TP1, TP10, TP11, TP2, TP3, TP4, TP5, TP6, TP7, TP8, TP9: TestPoint, TestPoint:TestPoint_Pad_D2.0mm, symbol Connector:TestPoint
- C1, C10, C11, C12, C13, C14, C15, C16, C17, C18, C19, C2, C20, C21, C22, C23, C24, C25, C26, C27, C28, C29, C3, C30, C31, C32, C33, C35, C36, C37, C38, C39, C4, C40, C41, C42, C43, C44, C46, C47, C48, C49, C5, C50, C51, C52, C53, C54, C55, C56, C57, C58, C59, C6, C60, C61, C62, C63, C64, C65, C66, C67, C68, C69, C7, C70, C8, C9: renamed from C?; footprint (none) -> Capacitor_SMD:C_0805_2012Metric
- C34: renamed from C?; footprint (none) -> Capacitor_SMD:C_2220_5650Metric
- C45: renamed from C?; footprint (none) -> Capacitor_SMD:C_1206_3216Metric
- D2: renamed from D?; footprint (none) -> Custom:SMAJ58A
- D3, D4, D5: renamed from D?; footprint (none) -> Custom:RFN2LAM6STF
- D6: renamed from D?; footprint (none) -> Custom:CFP15
- J1: renamed from J?; footprint (none) -> Custom:CONREVSMA003.062-G
- L1, L2, L3, L4, L5, L6, L7, L8: renamed from L?; footprint (none) -> Inductor_SMD:L_0805_2012Metric
- L9: renamed from L?; value 4.7uH -> 4.7uH SDR7030; footprint (none) -> Custom:SDR7030
- R1, R10, R11, R12, R13, R14, R15, R16, R17, R18, R19, R2, R20, R21, R22, R23, R25, R26, R27, R28, R29, R3, R30, R4, R5, R6, R7, R8, R9: renamed from R?; footprint (none) -> Resistor_SMD:R_0805_2012Metric
- R24: renamed from R?; value 0.56 0.1W -> 0.56 0.25W; footprint (none) -> Resistor_SMD:R_0805_2012Metric
- SW1: renamed from SW?; footprint (none) -> Custom:PTS636
- U2: footprint RHB32_3P45X3P45_TEX -> Davis Receiver Footprints:CC1125RHBR
- Y1: renamed from Y?; footprint (none) -> Custom:LFXTAL071758CUTT
- gave numbers to parts that had none: 10
Connections:
- net +3V0: now also TP1.1
- net +3V3: now also TP10.1
- net BAR_CS: now also J5.3
- net BAR_MISO: now also J5.4
- net BAR_MOSI: now also J5.5
- net BAR_SCLK: now also J5.2
- net GND: now also J3.3 (GND), J4.1 (GND), J5.1, J6.1, TP11.1
- net RF_CS: now also J6.3
- net RF_MISO: now also J6.4
- net RF_MOSI: now also J6.5
- net RF_SCLK: now also J6.2
- net UART_RX: now also J4.4 (TX)
- net UART_TX: now also J4.5 (RX)
- net JTAG_TCK: now reaches U1.B15 (PC0_TCK_SWCLK)
- net JTAG_TCK: now also J3.4 (TCK)
- net JTAG_TDO: now reaches U1.C14 (PC3_TDO_SWO)
- net JTAG_TDO: now also J3.6 (TDO)
- net JTAG_TMS: now reaches U1.C15 (PC1_TMS_SWDIO)
- net JTAG_TMS: now also J3.2 (TMS)
- net JTAG_TDI: now reaches U1.D14 (PC2_TDI)
- net JTAG_TDI: now also J3.8 (TDI)
- net at C17.1, R5.1, R7.2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: now also TP2.1
- net at C38.2, R19.1, U7.1 (CTL)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: now also TP5.1
- net at C39.1, R14.2, R19.2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: now also TP8.1
- net at C40.1, C43.1, D3.1 (K)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: now also TP7.1
- net at R22.1, U7.5 (GATE): now also TP6.1
- net at C14.2, D2.2, R10.2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: now also TP4.1
- net at C14.1, C34.1, D2.1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: now also TP3.1
- net at D4.2 (A), Q1.1 (D), Q1.2 (D)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: now also TP9.1
- net JTAG_RESET: now reaches R5.2, SW1.2
- net JTAG_RESET: now also J3.10 (RST)
- new net: J3.5 (NC), J3.9 (NC)
Other:
- note added: "Barometer"
- note added: "JTAG / Debug Conns"
- note added: "Main uC"
- note removed: "BAROMETER"
- moved on the sheet: C1, C10, C11, C12, C13, C14, C15, C16, C17, C18, C19, C2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

Commit message: Davis Receiver v1.0
Parts:
- added H1, H2, H3, H4: MountingHole, MountingHole:MountingHole_4.3mm_M4_Pad_Via, symbol Mechanical:MountingHole
- C1, C2, C35, C37, C41, C44, C7: value 100nF -> 0.1uF
- C11, C12, C22, C25, C28, C3, C31, C32, C5, C8: value 47nF -> 0.047uF
- C15, C9: value 10nF -> 0.01uF
- C52: value 6.8nF -> 6800pF
Connections:
- net GND: no longer J2.SHD (Sheild)
- net GND1: now also J2.SHD (Sheild)
- net ETH_RX_N: now reaches J2.5 (RD-), R16.2, U1.V13 (EN0RXIN)
- net ETH_TX_N: now reaches J2.2 (TD-), R13.2, U1.V14 (EN0TXON)
- net ETH_TX_P: now reaches J2.1 (TD+), R12.2, U1.V15 (EN0TXOP)
- net ETH_RX_P: now reaches J2.4 (RD+), R15.2, U1.W13 (EN0RXIP)
Changed lines of the file:
@@
 P 20300 15400
 F 0 "C52" V 20552 15400 50  0000 C CNN
-F 1 "6.8nF" V 20461 15400 50  0000 C CNN
+F 1 "6800pF" V 20461 15400 50  0000 C CNN
 F 2 "Capacitor_SMD:C_0805_2012Metric" H 20338 15250 50  0001 C CNN
 F 3 "~" H 20300 15400 50  0001 C CNN
@@
 P 3850 26000
 F 0 "C2" H 3965 26046 50  0000 L CNN
-F 1 "100nF" H 3965 25955 50  0000 L CNN
+F 1 "0.1uF" H 3965 25955 50  0000 L CNN
 F 2 "Capacitor_SMD:C_0805_2012Metric" H 3888 25850 50  0001 C CNN
 F 3 "~" H 3850 26000 50  0001 C CNN
@@
 P 5400 26200
 F 0 "C9" H 5515 26246 50  0000 L CNN
-F 1 "10nF" H 5515 26155 50  0000 L CNN
+F 1 "0.01uF" H 5515 26155 50  0000 L CNN
 F 2 "Capacitor_SMD:C_0805_2012Metric" H 5438 26050 50  0001 C CNN
 F 3 "~" H 5400 26200 50  0001 C CNN
@@
 P 2450 20250
 F 0 "C1" H 2565 20296 50  0000 L CNN
-F 1 "100nF" H 2565 20205 50  0000 L CNN
+F 1 "0.1uF" H 2565 20205 50  0000 L CNN
 F 2 "Capacitor_SMD:C_0805_2012Metric" H 2488 20100 50  0001 C CNN
 F 3 "~" H 2450 20250 50  0001 C CNN
@@
 P 11200 19950
 F 0 "C22" H 11315 19996 50  0000 L CNN
-F 1 "47nF" H 11315 19905 50  0000 L CNN
+F 1 "0.047uF" H 11315 19905 50  0000 L CNN
 F 2 "Capacitor_SMD:C_0805_2012Metric" H 11238 19800 50  0001 C CNN
 F 3 "~" H 11200 19950 50  0001 C CNN
@@
 P 11650 19950
 F 0 "C25" H 11765 19996 50  0000 L CNN
-F 1 "47nF" H 11765 19905 50  0000 L CNN
+F 1 "0.047uF" H 11765 19905 50  0000 L CNN
 F 2 "Capacitor_SMD:C_0805_2012Metric" H 11688 19800 50  0001 C CNN
 F 3 "~" H 11650 19950 50  0001 C CNN
@@
 P 12100 19950
 F 0 "C28" H 12215 19996 50  0000 L CNN
-F 1 "47nF" H 12215 19905 50  0000 L CNN
+F 1 "0.047uF" H 12215 19905 50  0000 L CNN
 F 2 "Capacitor_SMD:C_0805_2012Metric" H 12138 19800 50  0001 C CNN
 F 3 "~" H 12100 19950 50  0001 C CNN
@@
 P 12550 19950
 F 0 "C31" H 12665 19996 50  0000 L CNN
-F 1 "47nF" H 12665 19905 50  0000 L CNN
+F 1 "0.047uF" H 12665 19905 50  0000 L CNN
 F 2 "Capacitor_SMD:C_0805_2012Metric" H 12588 19800 50  0001 C CNN
 F 3 "~" H 12550 19950 50  0001 C CNN
@@
 P 13000 19950
 F 0 "C32" H 13115 19996 50  0000 L CNN
-F 1 "47nF" H 13115 19905 50  0000 L CNN
+F 1 "0.047uF" H 13115 19905 50  0000 L CNN
 F 2 "Capacitor_SMD:C_0805_2012Metric" H 13038 19800 50  0001 C CNN
 F 3 "~" H 13000 19950 50  0001 C CNN
@@
 P 10450 27150
 F 0 "C15" H 10565 27196 50  0000 L CNN
-F 1 "10nF" H 10565 27105 50  0000 L CNN
+F 1 "0.01uF" H 10565 27105 50  0000 L CNN
 F 2 "Capacitor_SMD:C_0805_2012Metric" H 10488 27000 50  0001 C CNN
 F 3 "~" H 10450 27150 50  0001 C CNN
@@
 P 6700 22800
 F 0 "C12" H 6815 22846 50  0000 L CNN
-F 1 "47nF" H 6815 22755 50  0000 L CNN
+F 1 "0.047uF" H 6815 22755 50  0000 L CNN
 F 2 "Capacitor_SMD:C_0805_2012Metric" H 6738 22650 50  0001 C CNN
 F 3 "~" H 6700 22800 50  0001 C CNN
@@
 P 6000 22800
 F 0 "C11" H 6115 22846 50  0000 L CNN
-F 1 "47nF" H 6115 22755 50  0000 L CNN
+F 1 "0.047uF" H 6115 22755 50  0000 L CNN
 F 2 "Capacitor_SMD:C_0805_2012Metric" H 6038 22650 50  0001 C CNN
 F 3 "~" H 6000 22800 50  0001 C CNN
@@
 P 5300 22800
 F 0 "C8" H 5415 22846 50  0000 L CNN
-F 1 "47nF" H 5415 22755 50  0000 L CNN
+F 1 "0.047uF" H 5415 22755 50  0000 L CNN
 F 2 "Capacitor_SMD:C_0805_2012Metric" H 5338 22650 50  0001 C CNN
 F 3 "~" H 5300 22800 50  0001 C CNN
@@
 P 4600 22800
 F 0 "C5" H 4715 22846 50  0000 L CNN
-F 1 "47nF" H 4715 22755 50  0000 L CNN
+F 1 "0.047uF" H 4715 22755 50  0000 L CNN
 F 2 "Capacitor_SMD:C_0805_2012Metric" H 4638 22650 50  0001 C CNN
 F 3 "~" H 4600 22800 50  0001 C CNN
@@
 P 3950 22800
 F 0 "C3" H 4065 22846 50  0000 L CNN
-F 1 "47nF" H 4065 22755 50  0000 L CNN
+F 1 "0.047uF" H 4065 22755 50  0000 L CNN
 F 2 "Capacitor_SMD:C_0805_2012Metric" H 3988 22650 50  0001 C CNN
 F 3 "~" H 3950 22800 50  0001 C CNN
@@
 P 5050 10950
 F 0 "C7" H 5165 10996 50  0000 L CNN
-F 1 "100nF" H 5165 10905 50  0000 L CNN
+F 1 "0.1uF" H 5165 10905 50  0000 L CNN
 F 2 "Capacitor_SMD:C_0805_2012Metric" H 5088 10800 50  0001 C CNN
 F 3 "~" H 5050 10950 50  0001 C CNN
@@
 P 15350 3450
 F 0 "C41" H 15465 3496 50  0000 L CNN
-F 1 "100nF" H 15465 3405 50  0000 L CNN
+F 1 "0.1uF" H 15465 3405 50  0000 L CNN
 F 2 "Capacitor_SMD:C_0805_2012Metric" H 15388 3300 50  0001 C CNN
 F 3 "~" H 15350 3450 50  0001 C CNN
@@
 P 15850 3450
 F 0 "C44" H 15965 3496 50  0000 L CNN
-F 1 "100nF" H 15965 3405 50  0000 L CNN
+F 1 "0.1uF" H 15965 3405 50  0000 L CNN
 F 2 "Capacitor_SMD:C_0805_2012Metric" H 15888 3300 50  0001 C CNN
 F 3 "~" H 15850 3450 50  0001 C CNN
@@
 	15200 5550 15700 5550
 $Comp
-L power:GND #PWR063
+L power:GND1 #PWR063
 U 1 1 62E4313E
 P 15600 5900
 F 0 "#PWR063" H 15600 5650 50  0001 C CNN
-F 1 "GND" H 15605 5727 50  0000 C CNN
+F 1 "GND1" H 15605 5727 50  0000 C CNN
 F 2 "" H 15600 5900 50  0001 C CNN
 F 3 "" H 15600 5900 50  0001 C CNN
@@
 P 13650 2400
 F 0 "C35" H 13765 2446 50  0000 L CNN
-F 1 "100nF" H 13765 2355 50  0000 L CNN
+F 1 "0.1uF" H 13765 2355 50  0000 L CNN
 F 2 "Capacitor_SMD:C_0805_2012Metric" H 13688 2250 50  0001 C CNN
 F 3 "~" H 13650 2400 50  0001 C CNN
@@
 P 14200 2400
 F 0 "C37" H 14315 2446 50  0000 L CNN
-F 1 "100nF" H 14315 2355 50  0000 L CNN
+F 1 "0.1uF" H 14315 2355 50  0000 L CNN
 F 2 "Capacitor_SMD:C_0805_2012Metric" H 14238 2250 50  0001 C CNN
 F 3 "~" H 14200 2400 50  0001 C CNN
@@
 Wire Wire Line
 	5300 25550 5800 25550
+$Comp
+L Mechanical:MountingHole H1
+U 1 1 6064B59A
+P 21850 19300
+F 0 "H1" H 21950 19346 50  0000 L CNN
+F 1 "MountingHole" H 21950 19255 50  0000 L CNN
+F 2 "MountingHole:MountingHole_4.3mm_M4_Pad_Via" H 21850 19300 50  0001 C CNN
+F 3 "~" H 21850 19300 50  0001 C CNN
+	1    21850 19300
+	1    0    0    -1
+$EndComp
+$Comp
+L Mechanical:MountingHole H2
+U 1 1 6064BF41
+P 21850 19600
+F 0 "H2" H 21950 19646 50  0000 L CNN
+F 1 "MountingHole" H 21950 19555 50  0000 L CNN
+F 2 "MountingHole:MountingHole_4.3mm_M4_Pad_Via" H 21850 19600 50  0001 C CNN
+F 3 "~" H 21850 19600 50  0001 C CNN
+	1    21850 19600
+	1    0    0    -1
+$EndComp
+$Comp
+L Mechanical:MountingHole H3
+U 1 1 6064DDFF
+P 21850 19900
+F 0 "H3" H 21950 19946 50  0000 L CNN
+F 1 "MountingHole" H 21950 19855 50  0000 L CNN
+F 2 "MountingHole:MountingHole_4.3mm_M4_Pad_Via" H 21850 19900 50  0001 C CNN
+F 3 "~" H 21850 19900 50  0001 C CNN
+	1    21850 19900
+	1    0    0    -1
+$EndComp
+$Comp
+L Mechanical:MountingHole H4
+U 1 1 6064FD8B
+P 21850 20200
+F 0 "H4" H 21950 20246 50  0000 L CNN
+F 1 "MountingHole" H 21950 20155 50  0000 L CNN
+F 2 "MountingHole:MountingHole_4.3mm_M4_Pad_Via" H 21850 20200 50  0001 C CNN
+F 3 "~" H 21850 20200 50  0001 C CNN
+	1    21850 20200
+	1    0    0    -1
+$EndComp
+Text Label 14800 4250 0    50   ~ 0
+ETH_TX_P
+Text Label 14800 4350 0    50   ~ 0
+ETH_TX_N
+Text Label 14800 4550 0    50   ~ 0
+ETH_RX_P
+Text Label 14800 4650 0    50   ~ 0
+ETH_RX_N
 $EndSCHEMATC

Commit message: Davis Receiver v1.1
Parts:
- C52: value 6800pF -> 11900pF
- R18: value 49.9K 0.1W -> 80K 0.1W
- R29: value 13.3K -> 24.3K
Changed lines of the file:
@@
 P 14750 11350
 F 0 "R18" H 14820 11396 50  0000 L CNN
-F 1 "49.9K 0.1W" H 14820 11305 50  0000 L CNN
+F 1 "80K 0.1W" H 14820 11305 50  0000 L CNN
 F 2 "Resistor_SMD:R_0805_2012Metric" V 14680 11350 50  0001 C CNN
 F 3 "~" H 14750 11350 50  0001 C CNN
@@
 P 21100 16350
 F 0 "R29" H 21030 16304 50  0000 R CNN
-F 1 "13.3K" H 21030 16395 50  0000 R CNN
+F 1 "24.3K" H 21030 16395 50  0000 R CNN
 F 2 "Resistor_SMD:R_0805_2012Metric" V 21030 16350 50  0001 C CNN
 F 3 "~" H 21100 16350 50  0001 C CNN
@@
 $EndComp
 $Comp
-L Device:C C52
-U 1 1 60AC2D7F
-P 20300 15400
-F 0 "C52" V 20552 15400 50  0000 C CNN
-F 1 "6800pF" V 20461 15400 50  0000 C CNN
-F 2 "Capacitor_SMD:C_0805_2012Metric" H 20338 15250 50  0001 C CNN
-F 3 "~" H 20300 15400 50  0001 C CNN
-	1    20300 15400
-	0    -1   -1   0
-$EndComp
-$Comp
 L Device:C C46
 U 1 1 60ACC076
@@
 Text Label 14800 4650 0    50   ~ 0
 ETH_RX_N
+$Comp
+L Device:C C52
+U 1 1 60AC2D7F
+P 20300 15400
+F 0 "C52" V 20552 15400 50  0000 C CNN
+F 1 "11900pF" V 20461 15400 50  0000 C CNN
+F 2 "Capacitor_SMD:C_0805_2012Metric" H 20338 15250 50  0001 C CNN
+F 3 "~" H 20300 15400 50  0001 C CNN
+	1    20300 15400
+	0    -1   -1   0
+$EndComp
+Text Label 15300 6000 0    50   ~ 0
+SHLD
+Wire Wire Line
+	15300 6000 15600 6000
+Connection ~ 15600 6000
 $EndSCHEMATC

Commit message: Updates and new projects
Parts:
- J3: symbol Custom:TC-2050-Cortex-JTAG -> davis-receiver-rescue:TC-2050-Cortex-JTAG-Custom
Changed lines of the file:
@@
 	6250 2600 6350 2600
 $Comp
-L Custom:TC-2050-Cortex-JTAG J3
+L davis-receiver-rescue:TC-2050-Cortex-JTAG-Custom J3
 U 1 1 606A9E30
 P 18150 19300
