File: davis-receiver/davis-receiver-kc6.kicad_pcb (KiCad board)
At the start: 4 copper layers, 110 x 70 mm, 153 parts, among them J1 Conn_Coaxial, J2 Wurth_74982104400, J3 JTAG, J4 UART, J5 SPI-BARO, J6 SPI-RF, J7 GPIO-RF, Q1 FDC2512, SW1 MCU_RESET, T1 POE70P-33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

Commit message: Davis RX and Weir Controller changes
Parts:
- U2: value CC1125RHBR -> RHB32_3P45X3P45_TEX
