File: sea-led/sea-led.sch (KiCad schematic (older format))
At the start: 113 parts

Commit message: Lots of footprint updates
Parts:
- C1, C11, C12, C16, C18, C19, C20, C21, C22, C23, C24, C25, C26, C27, C28, C29, C3, C30, C31, C32, C33, C34, C35, C36, C37, C38, C39, C4, C40, C41, C6, C9: renamed from C?; footprint (none) -> Capacitor_SMD:C_0805_2012Metric
- C10, C13, C14, C8: renamed from C?; footprint (none) -> Capacitor_SMD:C_1206_3216Metric
- C15: renamed from C?; footprint (none) -> Capacitor_SMD:C_1812_4532Metric
- C17: renamed from C?; footprint (none) -> Capacitor_Tantalum_SMD:CP_EIA-7343-30_AVX-N_Pad2.25x2.55mm_HandSolder
- C2, C5: renamed from C?; value C_Small -> 22pF; footprint (none) -> Capacitor_SMD:C_0805_2012Metric
- C7: renamed from C?; footprint (none) -> Custom:Panasonic-Electrolytic-K16; symbol Device:C_Small -> Device:CP_Small
- D1, D2: renamed from D?; footprint (none) -> Custom:SMAJ30CA
- D3: renamed from D?; footprint (none) -> LED_SMD:LED_Cree-PLCC4_2x2mm_CW
- D4: renamed from D?; value D_Schottky -> PMEG045V100EPD; footprint (none) -> Custom:CFP15
- D5: renamed from D?; value BLUE -> BLUE - HSMN-C150; footprint (none) -> LED_SMD:LED_1206_3216Metric_Castellated
- D6: renamed from D?; value GREEN -> GREEN - HSMM-C150; footprint (none) -> LED_SMD:LED_1206_3216Metric_Castellated
- F1: renamed from F?; footprint (none) -> Custom:Keystone-3568
- F2: renamed from F?; footprint (none) -> Custom:2016L075_60MR
- H1, H2, H3, H4, H5, H6: renamed from H?; footprint (none) -> MountingHole:MountingHole_3.5mm_Pad_Via
- J3: renamed from J?; footprint (none) -> Custom:PhoenixContact-PTS-1_5-2POS-1703084
- J4: renamed from J?; footprint (none) -> Custom:PhoenixContact-PTS-1_5-5POS-1792892
- J5: renamed from J?; footprint custom-parts:Wurth_74980104400 -> Custom:Wurth_74980104400
- L1: renamed from L?; value 15uH -> 15uH SRP1265A-150M; footprint (none) -> Custom:SRP1265A-150M
- Q1: renamed from Q?; footprint (none) -> Package_TO_SOT_SMD:SOT-23; symbol Device:Q_NMOS_DGS -> Device:Q_NMOS_GSD
- R1, R10, R11, R12, R13, R14, R15, R16, R17, R18, R19, R2, R20, R21, R22, R23, R24, R25, R26, R27, R28, R29, R3, R30, R31, R32, R33, R4, R5, R6, R7, R8, R9: renamed from R?; footprint (none) -> Resistor_SMD:R_0805_2012Metric
- SW1, SW2, SW3: renamed from SW?; footprint (none) -> Custom:PTS636
- TP1, TP2, TP3, TP4, TP5, TP6: renamed from TP?; footprint (none) -> TestPoint:TestPoint_Pad_D1.5mm
- U1: renamed from U?; footprint ZAD0212A -> TM4C:TM4C129ENCZADI3R
- U3: renamed from U?; footprint (none) -> Custom:VQFN-24
- Y1: renamed from Y?; footprint (none) -> Custom:LFXTAL071758CUTT
- gave numbers to parts that had none: 5
Connections:
- net GND: now also Q1.2 (S); no longer Q1.3 (S)
- net PWR_SW_CTL: now also Q1.1 (G); no longer Q1.2 (G)
- net at F2.2: now also Q1.3 (D); no longer Q1.1 (D)

Commit message: Sea LED Routing Complete
Parts:
- removed TP2, TP3: TestPoint, TestPoint:TestPoint_Pad_D1.5mm, symbol Connector:TestPoint
- added R34: 100, Resistor_SMD:R_0805_2012Metric, symbol Device:R_Small
- added TP10, TP11, TP15, TP16, TP17, TP18, TP19, TP20, TP21, TP7, TP8, TP9: TestPoint, TestPoint:TestPoint_Pad_D1.5mm, symbol Connector:TestPoint
- C10, C13, C14, C8: value 100uF -> 0.1uF; footprint Capacitor_SMD:C_1206_3216Metric -> Capacitor_SMD:C_0805_2012Metric
- C2, C5: value 22pF -> 8pF
- D3: symbol Custom:LED_ABGR -> Device:LED_RABG
Connections:
- net +12V: now also TP18.1
- net +3V3: now also D3.2 (A), J2.1 (VCC); no longer D3.1 (A), R1.1
- net +5V: now also TP20.1
- net GND: now also R1.2, SW2.1, SW3.1, U1.T18 (XOSC0), TP21.1; no longer SW2.2, SW3.2, U1.E19 (OSC0)
- net IND_B: now also TP10.1
- net IND_G: now also R6.1, TP9.1; no longer R5.1
- net IND_R: now also R5.1, TP8.1; no longer R6.1
- net JTAG_RESET: now also R8.2, SW1.2; no longer C3.1, R12.2, R8.1, TP4.1, U1.P18 (RST_N)
- net PWR_SW_CTL: now also U1.B3 (PD6), R34.2, TP16.1; no longer Q1.1 (G), R13.1, U1.B2 (PD7)
- net DMX_TX_EN: now reaches U1.D2 (PD2)
- net DMX_TX_EN: now also R1.1, U2.3 (DE), TP7.1
- net DIVSCLK: now reaches U1.A13 (PQ4)
- net DIVSCLK: now also TP11.1
- net at U1.D19 (OSC1): now also C5.1, Y1.3
- net at C2.1, Y1.1: now also U1.E19 (OSC0); no longer U1.T18 (XOSC0)
- net ETH_RX_N: now reaches J5.6 (RD-), R21.2, U1.V13 (EN0RXIN)
- net ETH_TX_N: now reaches J5.2 (TD-), R19.2, U1.V14 (EN0TXON)
- net ETH_TX_P: now reaches J5.1 (TD+), R18.2, U1.V15 (EN0TXOP)
- net ETH_RX_P: now reaches J5.3 (RD+), R20.2, U1.W13 (EN0RXIP)
- net at C4.1, F1.1, R9.1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: now also TP15.1
- net at C16.1, D4.1 (K), L1.1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: now also TP19.1
- net at R31.2: now also SW2.2; no longer SW2.1
- net at R33.2: now also SW3.2; no longer SW3.1
- net at R7.2: now also D3.3 (BK); no longer D3.2 (BK)
- net at R5.2: now also D3.1 (RK); no longer D3.3 (GK)
- net at F2.2, Q1.3 (D): now also TP17.1
- new net: C3.1, R12.2, R8.1, TP4.1, U1.P18 (RST_N)
- new net: Q1.1 (G), R13.1, R34.1
- now unconnected: U1.T19 (XOSC1)
Other:
- moved on the sheet: C3, R1, R12, R8, SW1, SW2, SW3, TP4

Commit message: Updates to DavisReceiver
Parts:
- R15: value 2.4k -> 5.5K
Changed lines of the file:
@@
 P 14350 3100
 F 0 "R15" H 14409 3146 50  0000 L CNN
-F 1 "2.4k" H 14409 3055 50  0000 L CNN
+F 1 "5.5K" H 14409 3055 50  0000 L CNN
 F 2 "Resistor_SMD:R_0805_2012Metric" H 14350 3100 50  0001 C CNN
 F 3 "~" H 14350 3100 50  0001 C CNN
