File: usb-c_pd_powersupply/usb-c_pd_powersupply.kicad_pcb (KiCad board)
At the start: 4 copper layers, 55 x 57 mm, 79 parts, among them J1 USB_C_Receptacle, J2 TC2030-SWD, J3 Conn_01x02, J4 Conn_01x02, U1 STM32L011, U2 PTN5110, U3 AOZ1375DI, U4 LT3685, U5 LT3685, U6 LT3685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

Commit message: Cleanup + bugfixes
Parts:
- D3: footprint LED_SMD:LED_RGB_Wuerth-PLCC4_3.2x2.8mm_150141M173100 -> LED_SMD:LED_Cree-PLCC4_3.2x2.8mm_CCW
- R27: value 500 -> 1.5k
- R28: value 500 -> 1k
- turned D3 to -90 degrees
Routing:
- net Net-(D3-Pad1): track 5.29 -> 1.95 mm
- net +3V3: track 123.9 -> 125.5 mm
Other:
- board text added: "USB-C PD 35W 15V"
- board text removed: "USB-C PD 30W"
Changed lines of the file:
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@@
       (effects (font (size 1 1) (thickness 0.15)))
     )
-    (fp_text value "500" (at 0 1.65 90) (layer "F.Fab")
+    (fp_text value "1k" (at 0 1.65 90) (layer "F.Fab")
       (effects (font (size 1 1) (thickness 0.15)))
     )
@@
       (effects (font (size 1 1) (thickness 0.15)))
     )
-    (fp_text value "500" (at 0 1.65 90) (layer "F.Fab")
+    (fp_text value "1.5k" (at 0 1.65 90) (layer "F.Fab")
       (effects (font (size 1 1) (thickness 0.15)))
     )
@@
     (property "Sheetname" "")
     (attr exclude_from_pos_files)
-    (fp_text reference "TP1" (at -0.8 -2.1) (layer "F.SilkS")
+    (fp_text reference "TP1" (at -0.657337 -2.287401) (layer "F.SilkS")
       (effects (font (size 1 1) (thickness 0.15)))
     )
@@
     )
   )
-  (footprint "LED_SMD:LED_RGB_Wuerth-PLCC4_3.2x2.8mm_150141M173100" (layer "F.Cu")
-    (at 67.7 50.1 90)
-    (descr "3.2mm x 2.8mm PLCC4 LED, https://www.we-online.de/katalog/datasheet/150141M173100.pdf")
-    (tags "LED RGB Wurth PLCC-4")
+  (footprint "LED_SMD:LED_Cree-PLCC4_3.2x2.8mm_CCW" (layer "F.Cu")
+    (at 67.7 50.1 -90)
+    (descr "3.2mm x 2.8mm PLCC4 LED, http://www.cree.com/led-components/media/documents/CLV1AFKB(874).pdf")
+    (tags "LED Cree PLCC-4")
     (property "Sheetfile" "usb-c_pd_powersupply.kicad_sch")
     (property "Sheetname" "")
     (attr smd)
-    (fp_text reference "D3" (at 1.3 -2.4 90) (layer "F.SilkS")
+    (fp_text reference "D3" (at 0 -2.65 90) (layer "F.SilkS")
       (effects (font (size 1 1) (thickness 0.15)))
     )
-    (fp_text value "LED_RABG" (at 0 2.5 90) (layer "F.Fab")
+    (fp_text value "LED_RABG" (at 0 2.65 90) (layer "F.Fab")
       (effects (font (size 1 1) (thickness 0.15)))
     )
@@
       (effects (font (size 0.5 0.5) (thickness 0.075)))
     )
-    (fp_line (start -2.3 1.51) (end 2.3 1.51) (layer "F.SilkS") (width 0.12))
-    (fp_line (start -2.5 -0.7) (end -2.5 -1.51) (layer "F.SilkS") (width 0.12))
-    (fp_line (start -2.5 -1.51) (end 2.3 -1.51) (layer "F.SilkS") (width 0.12))
-    (fp_line (start 2.55 -1.65) (end -2.55 -1.65) (layer "F.CrtYd") (width 0.05))
-    (fp_line (start 2.55 1.65) (end 2.55 -1.65) (layer "F.CrtYd") (width 0.05))
-    (fp_line (start -2.55 -1.65) (end -2.55 1.65) (layer "F.CrtYd") (width 0.05))
-    (fp_line (start -2.55 1.65) (end 2.55 1.65) (layer "F.CrtYd") (width 0.05))
-    (fp_line (start 1.6 1.4) (end 1.6 -1.4) (layer "F.Fab") (width 0.1))
-    (fp_line (start 1.6 -1.4) (end -1.6 -1.4) (layer "F.Fab") (width 0.1))
+    (fp_line (start -1.95 -0.7) (end -1.95 -1.5) (layer "F.SilkS") (width 0.12))
+    (fp_line (start -1.95 -1.5) (end 1.95 -1.5) (layer "F.SilkS") (width 0.12))
+    (fp_line (start -1.95 1.5) (end 1.95 1.5) (layer "F.SilkS") (width 0.12))
+    (fp_line (start -2.2 1.75) (end 2.2 1.75) (layer "F.CrtYd") (width 0.05))
+    (fp_line (start 2.2 1.75) (end 2.2 -1.75) (layer "F.CrtYd") (width 0.05))
+    (fp_line (start 2.2 -1.75) (end -2.2 -1.75) (layer "F.CrtYd") (width 0.05))
+    (fp_line (start -2.2 -1.75) (end -2.2 1.75) (layer "F.CrtYd") (width 0.05))
     (fp_line (start -1.6 -1.4) (end -1.6 1.4) (layer "F.Fab") (width 0.1))
-    (fp_line (start -0.6 -1.4) (end -1.6 -0.4) (layer "F.Fab") (width 0.1))
     (fp_line (start -1.6 1.4) (end 1.6 1.4) (layer "F.Fab") (width 0.1))
+    (fp_line (start 1.6 -1.4) (end -1.6 -1.4) (layer "F.Fab") (width 0.1))
+    (fp_line (start 1.6 1.4) (end 1.6 -1.4) (layer "F.Fab") (width 0.1))
+    (fp_line (start -0.6 -1.4) (end -1.6 -0.4) (layer "F.Fab") (width 0.1))
     (fp_circle (center 0 0) (end 1.12 0) (layer "F.Fab") (width 0.1) (fill none))
-    (pad "1" smd rect locked (at 1.55 -0.7 90) (size 1.5 0.9) (layers "F.Cu" "F.Paste" "F.Mask")
+    (pad "1" smd rect locked (at -1.25 -0.7 270) (size 1 0.8) (layers "F.Cu" "F.Paste" "F.Mask")
       (net 16 "Net-(D3-Pad1)") (pinfunction "RK") (pintype "passive"))
-    (pad "2" smd rect locked (at 1.55 0.7 90) (size 1.5 0.9) (layers "F.Cu" "F.Paste" "F.Mask")
+    (pad "2" smd rect locked (at -1.25 0.7 270) (size 1 0.8) (layers "F.Cu" "F.Paste" "F.Mask")
       (net 3 "+3V3") (pinfunction "A") (pintype "passive"))
-    (pad "3" smd rect locked (at -1.55 -0.7 90) (size 1.5 0.9) (layers "F.Cu" "F.Paste" "F.Mask")
+    (pad "3" smd rect locked (at 1.25 0.7 270) (size 1 0.8) (layers "F.Cu" "F.Paste" "F.Mask")
       (net 15 "Net-(D3-Pad3)") (pinfunction "BK") (pintype "passive"))
-    (pad "4" smd rect locked (at -1.55 0.7 90) (size 1.5 0.9) (layers "F.Cu" "F.Paste" "F.Mask")
+    (pad "4" smd rect locked (at 1.25 -0.7 270) (size 1 0.8) (layers "F.Cu" "F.Paste" "F.Mask")
       (net 17 "Net-(D3-Pad4)") (pinfunction "GK") (pintype "passive"))
-    (model "${KICAD6_3DMODEL_DIR}/LED_SMD.3dshapes/LED_RGB_Wuerth-PLCC4_3.2x2.8mm_150141M173100.wrl"
+    (model "${KICAD6_3DMODEL_DIR}/LED_SMD.3dshapes/LED_Cree-PLCC4_3.2x2.8mm_CCW.wrl"
       (offset (xyz 0 0 0))
       (scale (xyz 1 1 1))
@@
     (effects (font (size 2 2) (thickness 0.25) italic))
   )
-  (gr_text "USB-C PD\n30W\n" (at 46 25 90) (layer "F.SilkS")
+  (gr_text "USB-C PD\n35W 15V\n" (at 46.1 24.7 90) (layer "F.SilkS")
     (effects (font (size 1 1) (thickness 0.15)) (justify right))
   )
@@
   (segment (start 68.569112 26.769112) (end 67.026636 26.769112) (width 0.2) (layer "B.Cu") (net 2))
   (segment (start 74.624 38.076) (end 74.8 37.9) (width 0.25) (layer "F.Cu") (net 3))
-  (segment (start 68.4 48.55) (end 68.4 47.1) (width 0.4) (layer "F.Cu") (net 3))
   (segment (start 74.70625 37.9) (end 74.8 37.9) (width 0.4) (layer "F.Cu") (net 3))
   (segment (start 72.8 44.8125) (end 72.8 46.3) (width 1) (layer "F.Cu") (net 3))
   (segment (start 69.8 33.5875) (end 69.8125 33.6) (width 1) (layer "F.Cu") (net 3))
+  (segment (start 72.8 46.3) (end 68 46.3) (width 0.4) (layer "F.Cu") (net 3))
   (segment (start 46.3775 37.238) (end 45 37.238) (width 1) (layer "F.Cu") (net 3))
   (segment (start 38.66 37.1575) (end 39.9275 37.1575) (width 0.3) (layer "F.Cu") (net 3))
@@
   (segment (start 27.3 48.4) (end 30.0375 48.4) (width 1) (layer "F.Cu") (net 3))
   (segment (start 67.976 38.576) (end 67.8 38.4) (width 0.25) (layer "F.Cu") (net 3))
+  (segment (start 68 46.3) (end 67 47.3) (width 0.4) (layer "F.Cu") (net 3))
   (segment (start 60 46.4) (end 60 45.042) (width 1) (layer "F.Cu") (net 3))
   (segment (start 71.124 38.576) (end 71.624 38.076) (width 0.25) (layer "F.Cu") (net 3))
@@
   (segment (start 69.5875 33.8) (end 69.8 33.5875) (width 0.2) (layer "F.Cu") (net 3))
   (segment (start 42.99 37.51) (end 41.99 37.51) (width 1) (layer "F.Cu") (net 3))
-  (segment (start 68.4 47.1) (end 69.2 46.3) (width 0.4) (layer "F.Cu") (net 3))
   (segment (start 39.9275 37.1575) (end 40.28 37.51) (width 0.3) (layer "F.Cu") (net 3))
   (segment (start 72.846 38.076) (end 74.624 38.076) (width 0.25) (layer "F.Cu") (net 3))
@@
   (segment (start 31.93 44.1075) (end 31.93 45.8075) (width 0.3) (layer "F.Cu") (net 3))
   (segment (start 69.8125 33.6) (end 72.7 33.6) (width 1) (layer "F.Cu") (net 3))
+  (segment (start 67 47.3) (end 67 48.85) (width 0.4) (layer "F.Cu") (net 3))
   (segment (start 35.1175 41) (end 36.1 41) (width 0.3) (layer "F.Cu") (net 3))
-  (segment (start 69.2 46.3) (end 72.8 46.3) (width 0.4) (layer "F.Cu") (net 3))
   (segment (start 65.6 33.8) (end 69.5875 33.8) (width 0.2) (layer "F.Cu") (net 3))
   (segment (start 32.01 44.1075) (end 35.1175 41) (width 0.3) (layer "F.Cu") (net 3))
@@
   (segment (start 54.28 61.84875) (end 52.79 60.35875) (width 0.3) (layer "B.Cu") (net 14))
   (segment (start 61.3 63.87875) (end 56.31 63.87875) (width 0.3) (layer "B.Cu") (net 14))
-  (segment (start 67.3 53) (end 67 52.7) (width 0.3) (layer "F.Cu") (net 15))
-  (segment (start 70.2875 53) (end 67.3 53) (width 0.3) (layer "F.Cu") (net 15))
-  (segment (start 67 52.7) (end 67 51.65) (width 0.3) (layer "F.Cu") (net 15))
-  (segment (start 69.2 49.4) (end 69.2 49.8) (width 0.3) (layer "F.Cu") (net 16))
-  (segment (start 69.2 49.8) (end 68.9 50.1) (width 0.3) (layer "F.Cu") (net 16))
-  (segment (start 67.4 50.1) (end 67 49.7) (width 0.3) (layer "F.Cu") (net 16))
-  (segment (start 70.2875 49) (end 69.6 49) (width 0.3) (layer "F.Cu") (net 16))
-  (segment (start 67 49.7) (end 67 48.55) (width 0.3) (layer "F.Cu") (net 16))
-  (segment (start 69.6 49) (end 69.2 49.4) (width 0.3) (layer "F.Cu") (net 16))
-  (segment (start 68.9 50.1) (end 67.4 50.1) (width 0.3) (layer "F.Cu") (net 16))
-  (segment (start 69.6 51) (end 68.95 51.65) (width 0.3) (layer "F.Cu") (net 17))
-  (segment (start 68.95 51.65) (end 68.4 51.65) (width 0.3) (layer "F.Cu") (net 17))
-  (segment (start 70.2875 51) (end 69.6 51) (width 0.3) (layer "F.Cu") (net 17))
+  (segment (start 67 51.35) (end 67 52.1) (width 0.4) (layer "F.Cu") (net 15))
+  (segment (start 67 52.1) (end 67.9 53) (width 0.4) (layer "F.Cu") (net 15))
+  (segment (start 67.9 53) (end 70.2875 53) (width 0.4) (layer "F.Cu") (net 15))
+  (segment (start 70.1375 48.85) (end 70.2875 49) (width 0.4) (layer "F.Cu") (net 16))
+  (segment (start 68.4 48.85) (end 70.1375 48.85) (width 0.4) (layer "F.Cu") (net 16))
+  (segment (start 68.4 51.35) (end 69.9375 51.35) (width 0.4) (layer "F.Cu") (net 17))
+  (segment (start 69.9375 51.35) (end 70.2875 51) (width 0.4) (layer "F.Cu") (net 17))
   (segment (start 59.4 39.1) (end 57.95 37.65) (width 0.2) (layer "F.Cu") (net 20))
   (segment (start 58.1 35.8) (end 58.1 36.85) (width 0.25) (layer "F.Cu") (net 20))

Commit message: Fixes
Connections:
- J2 pad 2: /SWDIO -> /nRESET
- J2 pad 3: /nRESET -> GND
- J2 pad 4: /SWDCLK -> unconnected-(J2-Pad4)
- J2 pad 5: GND -> /SWDCLK
- J2 pad 6: unconnected-(J2-Pad6) -> /SWDIO
Routing:
- net +3V3: track 125.5 -> 132.6 mm, vias 11 -> 13
- net /SWDCLK: track 32.7 -> 25.8 mm
- net /nRESET: track 23.0 -> 18.9 mm
- net /OUT_EN: track 104.2 -> 103.3 mm
- net /SWDIO: track 16.9 -> 16.2 mm
- net GND: vias 190 -> 208

Commit message: Tweaks
Other:
- board text added: "+"
- board text added: "-"
Changed lines of the file:
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@@
     (property "Sheetname" "")
     (attr through_hole)
-    (fp_text reference "J3" (at 5.9 -2.4 unlocked) (layer "F.SilkS")
+    (fp_text reference "J3" (at -3.2 5.7 unlocked) (layer "F.SilkS")
       (effects (font (size 1 1) (thickness 0.15)))
     )
@@
     (property "Sheetname" "")
     (attr through_hole)
-    (fp_text reference "J4" (at 5.85 -2.5 unlocked) (layer "F.SilkS")
+    (fp_text reference "J4" (at -3.55 5.8 unlocked) (layer "F.SilkS")
       (effects (font (size 1 1) (thickness 0.15)))
     )
@@
   (gr_arc (start 75 24) (mid 78.535534 25.464466) (end 80 29) (layer "Edge.Cuts") (width 0.1))
   (gr_line (start 25 76) (end 25 29) (layer "Edge.Cuts") (width 0.1))
-  (gr_text "12V@2A" (at 51.3 74.6 90) (layer "F.SilkS")
+  (gr_text "+" (at 59.5 79.5) (layer "F.SilkS")
+    (effects (font (size 1.5 1.5) (thickness 0.3)))
+  )
+  (gr_text "+" (at 40 79.5) (layer "F.SilkS")
+    (effects (font (size 1.5 1.5) (thickness 0.3)))
+  )
+  (gr_text "-" (at 70 79.5) (layer "F.SilkS")
+    (effects (font (size 1.5 1.5) (thickness 0.3)))
+  )
+  (gr_text "12V@2A" (at 50.9 72 90) (layer "F.SilkS")
     (effects (font (size 2 2) (thickness 0.25) italic))
   )
-  (gr_text "5V@2A" (at 70.7 75.4 90) (layer "F.SilkS")
+  (gr_text "5V@2A" (at 70.5 71.9 90) (layer "F.SilkS")
     (effects (font (size 2 2) (thickness 0.25) italic))
   )
@@
     (effects (font (size 1 1) (thickness 0.15)) (justify right))
   )
+  (gr_text "-" (at 50.5 79.75 180) (layer "F.SilkS")
+    (effects (font (size 1.5 1.5) (thickness 0.3)))
+  )
   (gr_text "USB-C PD\nPower Supply" (at 75.6 73 90) (layer "F.Mask")
