File: usb-c_pd_powersupply/usb-c_pd_powersupply.kicad_sch (KiCad schematic)
At the start: 72 parts, among them J1 USB_C_Receptacle, J2 TC2030-SWD, J3 Conn_01x02, J4 Conn_01x02, U1 STM32L011, U2 PTN5110, U3 AOZ1375DI, U4 LT3685, U5 LT3685, U6 LT3685, U7 CDSOT23-0502B

Commit message: Finished USB C PD Supply Layout
Parts:
- added R27, R28, R29: 500, Resistor_SMD:R_0805_2012Metric, symbol Device:R
Connections:
- net GND: now also R27.1, R28.1, R29.1; no longer D7.2 (A), D8.2 (A), D9.2 (A)
- net VBUS_SW: now reaches C10.1, C11.1, C9.1, R14.2, U3.9 (CSP), U4.4 (Vin), U5.4 (Vin), U6.4 (Vin), U6.5 (RUN/SS)
- net 12V_SW: now reaches C15.2, D4.1 (K), L1.1, U4.3 (SW)
- net VBUS: now reaches C1.2, C6.1, J1.A4 (VBUS), J1.A9 (VBUS), J1.B4 (VBUS), J1.B9 (VBUS), U2.15 (VBUS), U3.1 (VBUS)
- net 3V3_SW: now reaches C17.2, D6.1 (K), L3.1, U6.3 (SW)
- net 5V_SW: now reaches C16.2, D5.1 (K), L2.1, U5.3 (SW)
- net OUT_EN: now reaches U5.5 (RUN/SS)
- net OUT_EN: now also U1.8 (PA5), U4.5 (RUN/SS)
- new net: D7.2 (A), R27.2
- new net: D9.2 (A), R29.2
- new net: D8.2 (A), R28.2
Changed lines of the file:
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@@
     (stroke (width 0) (type default) (color 0 0 0 0))
   )
+  (wire (pts (xy 361.95 64.77) (xy 361.95 68.58))
+    (stroke (width 0) (type default) (color 0 0 0 0))
+  )
   (wire (pts (xy 363.22 199.39) (xy 353.06 199.39))
     (stroke (width 0) (type default) (color 0 0 0 0))
@@
     (stroke (width 0) (type default) (color 0 0 0 0))
   )
+  (wire (pts (xy 289.56 52.07) (xy 298.45 52.07))
+    (stroke (width 0) (type default) (color 0 0 0 0))
+  )
   (wire (pts (xy 201.93 64.77) (xy 201.93 68.58))
     (stroke (width 0) (type default) (color 0 0 0 0))
@@
     (stroke (width 0) (type default) (color 0 0 0 0))
   )
+  (wire (pts (xy 363.22 193.04) (xy 363.22 199.39))
+    (stroke (width 0) (type default) (color 0 0 0 0))
+  )
   (wire (pts (xy 361.95 40.64) (xy 351.79 40.64))
     (stroke (width 0) (type default) (color 0 0 0 0))
@@
     (stroke (width 0) (type default) (color 0 0 0 0))
   )
+  (wire (pts (xy 361.95 76.2) (xy 361.95 82.55))
+    (stroke (width 0) (type default) (color 0 0 0 0))
+  )
   (wire (pts (xy 72.39 120.65) (xy 83.82 120.65))
     (stroke (width 0) (type default) (color 0 0 0 0))
@@
     (stroke (width 0) (type default) (color 0 0 0 0))
   )
+  (wire (pts (xy 290.83 110.49) (xy 299.72 110.49))
+    (stroke (width 0) (type default) (color 0 0 0 0))
+  )
   (wire (pts (xy 153.67 85.09) (xy 153.67 87.63))
     (stroke (width 0) (type default) (color 0 0 0 0))
@@
     (stroke (width 0) (type default) (color 0 0 0 0))
   )
-  (wire (pts (xy 361.95 82.55) (xy 361.95 64.77))
+  (wire (pts (xy 363.22 123.19) (xy 363.22 127))
     (stroke (width 0) (type default) (color 0 0 0 0))
   )
@@
     (stroke (width 0) (type default) (color 0 0 0 0))
   )
+  (wire (pts (xy 363.22 134.62) (xy 363.22 140.97))
+    (stroke (width 0) (type default) (color 0 0 0 0))
+  )
   (wire (pts (xy 153.67 97.79) (xy 142.24 97.79))
     (stroke (width 0) (type default) (color 0 0 0 0))
@@
     (stroke (width 0) (type default) (color 0 0 0 0))
   )
-  (wire (pts (xy 363.22 123.19) (xy 363.22 140.97))
-    (stroke (width 0) (type default) (color 0 0 0 0))
-  )
   (wire (pts (xy 342.9 78.74) (xy 342.9 82.55))
     (stroke (width 0) (type default) (color 0 0 0 0))
@@
     (stroke (width 0) (type default) (color 0 0 0 0))
   )
+  (wire (pts (xy 363.22 181.61) (xy 363.22 185.42))
+    (stroke (width 0) (type default) (color 0 0 0 0))
+  )
   (wire (pts (xy 113.03 217.17) (xy 115.57 217.17))
     (stroke (width 0) (type default) (color 0 0 0 0))
@@
     (stroke (width 0) (type default) (color 0 0 0 0))
   )
-  (wire (pts (xy 363.22 181.61) (xy 363.22 199.39))
-    (stroke (width 0) (type default) (color 0 0 0 0))
-  )
   (wire (pts (xy 278.13 199.39) (xy 287.02 199.39))
     (stroke (width 0) (type default) (color 0 0 0 0))
@@
     (stroke (width 0) (type default) (color 0 0 0 0))
   )
+  (wire (pts (xy 85.09 133.35) (xy 92.71 133.35))
+    (stroke (width 0) (type default) (color 0 0 0 0))
+  )
   (wire (pts (xy 217.17 59.69) (xy 220.98 59.69))
     (stroke (width 0) (type default) (color 0 0 0 0))
@@
     (effects (font (size 1.27 1.27)) (justify left bottom))
   )
+  (label "OUT_EN" (at 290.83 110.49 0)
+    (effects (font (size 1.27 1.27)) (justify left bottom))
+  )
+  (label "3V3_SW" (at 330.2 172.72 0)
+    (effects (font (size 1.27 1.27)) (justify left bottom))
+  )
+  (label "OUT_EN" (at 289.56 52.07 0)
+    (effects (font (size 1.27 1.27)) (justify left bottom))
+  )
   (label "IND_R" (at 85.09 125.73 0)
     (effects (font (size 1.27 1.27)) (justify left bottom))
@@
     (effects (font (size 1.27 1.27)) (justify left bottom))
   )
+  (label "5V_SW" (at 330.2 114.3 0)
+    (effects (font (size 1.27 1.27)) (justify left bottom))
+  )
+  (label "OUT_EN" (at 85.09 133.35 0)
+    (effects (font (size 1.27 1.27)) (justify left bottom))
+  )
   (label "IND_G" (at 107.95 229.87 270)
     (effects (font (size 1.27 1.27)) (justify right bottom))
@@
     (effects (font (size 1.27 1.27)) (justify left bottom))
   )
+  (label "VBUS" (at 138.43 40.64 0)
+    (effects (font (size 1.27 1.27)) (justify left bottom))
+  )
   (label "VBUS_FAULT" (at 85.09 81.28 0)
     (effects (font (size 1.27 1.27)) (justify left bottom))
@@
     (effects (font (size 1.27 1.27)) (justify left bottom))
   )
+  (label "VBUS_SW" (at 255.27 40.64 0)
+    (effects (font (size 1.27 1.27)) (justify left bottom))
+  )
   (label "SWDIO" (at 129.54 125.73 0)
     (effects (font (size 1.27 1.27)) (justify left bottom))
@@
     (effects (font (size 1.27 1.27)) (justify left bottom))
   )
+  (label "12V_SW" (at 328.93 55.88 0)
+    (effects (font (size 1.27 1.27)) (justify left bottom))
+  )
   (label "EN_SINK" (at 132.08 66.04 0)
     (effects (font (size 1.27 1.27)) (justify left bottom))
@@
     (pin "2")
   )
+  (symbol (lib_id "Device:R") (at 361.95 72.39 180) (unit 1)
+    (in_bom yes) (on_board yes) (fields_autoplaced)
+    (property "Reference" "R27" (id 0) (at 363.728 71.4815 0)
+      (effects (font (size 1.27 1.27)) (justify right))
+    )
+    (property "Value" "500" (id 1) (at 363.728 74.2566 0)
+      (effects (font (size 1.27 1.27)) (justify right))
+    )
+    (property "Footprint" "Resistor_SMD:R_0805_2012Metric" (id 2) (at 363.728 72.39 90)
+      (effects (font (size 1.27 1.27)) hide)
+    )
+    (property "Datasheet" "~" (id 3) (at 361.95 72.39 0)
+      (effects (font (size 1.27 1.27)) hide)
+    )
+    (pin "1")
+    (pin "2")
+  )
   (symbol (lib_id "Device:C") (at 287.02 193.04 0) (unit 1)
     (in_bom yes) (on_board yes) (fields_autoplaced)
@@
     (pin "2")
   )
+  (symbol (lib_id "Device:R") (at 363.22 189.23 180) (unit 1)
+    (in_bom yes) (on_board yes) (fields_autoplaced)
+    (property "Reference" "R29" (id 0) (at 364.998 188.3215 0)
+      (effects (font (size 1.27 1.27)) (justify right))
+    )
+    (property "Value" "500" (id 1) (at 364.998 191.0966 0)
+      (effects (font (size 1.27 1.27)) (justify right))
+    )
+    (property "Footprint" "Resistor_SMD:R_0805_2012Metric" (id 2) (at 364.998 189.23 90)
+      (effects (font (size 1.27 1.27)) hide)
+    )
+    (property "Datasheet" "~" (id 3) (at 363.22 189.23 0)
+      (effects (font (size 1.27 1.27)) hide)
+    )
+    (pin "1")
+    (pin "2")
+  )
   (symbol (lib_id "power:GND") (at 152.4 144.78 0) (unit 1)
     (in_bom yes) (on_board yes) (fields_autoplaced)
@@
     (pin "1")
   )
+  (symbol (lib_id "Device:R") (at 363.22 130.81 180) (unit 1)
+    (in_bom yes) (on_board yes) (fields_autoplaced)
+    (property "Reference" "R28" (id 0) (at 364.998 129.9015 0)
+      (effects (font (size 1.27 1.27)) (justify right))
+    )
+    (property "Value" "500" (id 1) (at 364.998 132.6766 0)
+      (effects (font (size 1.27 1.27)) (justify right))
+    )
+    (property "Footprint" "Resistor_SMD:R_0805_2012Metric" (id 2) (at 364.998 130.81 90)
+      (effects (font (size 1.27 1.27)) hide)
+    )
+    (property "Datasheet" "~" (id 3) (at 363.22 130.81 0)
+      (effects (font (size 1.27 1.27)) hide)
+    )
+    (pin "1")
+    (pin "2")
+  )
   (symbol (lib_id "Device:C") (at 285.75 76.2 0) (unit 1)
     (in_bom yes) (on_board yes) (fields_autoplaced)
@@
       (reference "R26") (unit 1) (value "100k") (footprint "Resistor_SMD:R_0805_2012Metric")
     )
+    (path "/1cc0cee9-b5cd-46f1-be4e-672b3110c552"
+      (reference "R27") (unit 1) (value "500") (footprint "Resistor_SMD:R_0805_2012Metric")
+    )
+    (path "/fc9cd7a2-6fe8-492c-8d6e-695482a195f3"
+      (reference "R28") (unit 1) (value "500") (footprint "Resistor_SMD:R_0805_2012Metric")
+    )
+    (path "/c452d50b-4fb0-427b-9da6-1adb0c8dc035"
+      (reference "R29") (unit 1) (value "500") (footprint "Resistor_SMD:R_0805_2012Metric")
+    )
     (path "/3ee7c52f-c6ea-40d3-ad07-9ca566f1f580"

Commit message: Cleanup + bugfixes
Parts:
- D3: footprint LED_SMD:LED_RGB_Wuerth-PLCC4_3.2x2.8mm_150141M173100 -> LED_SMD:LED_Cree-PLCC4_3.2x2.8mm_CCW
- R27: value 500 -> 1.5k
- R28: value 500 -> 1k
Changed lines of the file:
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@@
   (symbol (lib_id "Device:R") (at 361.95 72.39 180) (unit 1)
     (in_bom yes) (on_board yes) (fields_autoplaced)
-    (property "Reference" "R27" (id 0) (at 363.728 71.4815 0)
-      (effects (font (size 1.27 1.27)) (justify right))
-    )
-    (property "Value" "500" (id 1) (at 363.728 74.2566 0)
+    (property "Reference" "R27" (id 0) (at 364.49 71.1199 0)
+      (effects (font (size 1.27 1.27)) (justify right))
+    )
+    (property "Value" "1.5k" (id 1) (at 364.49 73.6599 0)
       (effects (font (size 1.27 1.27)) (justify right))
     )
@@
   (symbol (lib_id "Device:R") (at 153.67 91.44 0) (unit 1)
     (in_bom yes) (on_board yes) (fields_autoplaced)
-    (property "Reference" "R8" (id 0) (at 155.448 90.5315 0)
-      (effects (font (size 1.27 1.27)) (justify left))
-    )
-    (property "Value" "10k" (id 1) (at 155.448 93.3066 0)
+    (property "Reference" "R8" (id 0) (at 156.21 90.1699 0)
+      (effects (font (size 1.27 1.27)) (justify left))
+    )
+    (property "Value" "10k" (id 1) (at 156.21 92.7099 0)
       (effects (font (size 1.27 1.27)) (justify left))
     )
@@
   (symbol (lib_id "Device:R") (at 161.29 91.44 0) (unit 1)
     (in_bom yes) (on_board yes) (fields_autoplaced)
-    (property "Reference" "R9" (id 0) (at 163.068 90.5315 0)
-      (effects (font (size 1.27 1.27)) (justify left))
-    )
-    (property "Value" "10k" (id 1) (at 163.068 93.3066 0)
+    (property "Reference" "R9" (id 0) (at 163.83 90.1699 0)
+      (effects (font (size 1.27 1.27)) (justify left))
+    )
+    (property "Value" "10k" (id 1) (at 163.83 92.7099 0)
       (effects (font (size 1.27 1.27)) (justify left))
     )
@@
       (effects (font (size 1.27 1.27)) (justify right))
     )
-    (property "Footprint" "LED_SMD:LED_RGB_Wuerth-PLCC4_3.2x2.8mm_150141M173100" (id 2) (at 109.22 209.55 0)
+    (property "Footprint" "LED_SMD:LED_Cree-PLCC4_3.2x2.8mm_CCW" (id 2) (at 109.22 209.55 0)
       (effects (font (size 1.27 1.27)) hide)
     )
@@
   (symbol (lib_id "Device:R") (at 363.22 130.81 180) (unit 1)
     (in_bom yes) (on_board yes) (fields_autoplaced)
-    (property "Reference" "R28" (id 0) (at 364.998 129.9015 0)
-      (effects (font (size 1.27 1.27)) (justify right))
-    )
-    (property "Value" "500" (id 1) (at 364.998 132.6766 0)
+    (property "Reference" "R28" (id 0) (at 365.76 129.5399 0)
+      (effects (font (size 1.27 1.27)) (justify right))
+    )
+    (property "Value" "1k" (id 1) (at 365.76 132.0799 0)
       (effects (font (size 1.27 1.27)) (justify right))
     )
@@
     )
     (path "/745d332d-7784-4552-8b64-cb4a3d7b8912"
-      (reference "D3") (unit 1) (value "LED_RABG") (footprint "LED_SMD:LED_RGB_Wuerth-PLCC4_3.2x2.8mm_150141M173100")
+      (reference "D3") (unit 1) (value "LED_RABG") (footprint "LED_SMD:LED_Cree-PLCC4_3.2x2.8mm_CCW")
     )
     (path "/07ec2586-54ed-4889-ba31-71ec8d273741"
@@
     )
     (path "/1cc0cee9-b5cd-46f1-be4e-672b3110c552"
-      (reference "R27") (unit 1) (value "500") (footprint "Resistor_SMD:R_0805_2012Metric")
+      (reference "R27") (unit 1) (value "1.5k") (footprint "Resistor_SMD:R_0805_2012Metric")
     )
     (path "/fc9cd7a2-6fe8-492c-8d6e-695482a195f3"
-      (reference "R28") (unit 1) (value "500") (footprint "Resistor_SMD:R_0805_2012Metric")
+      (reference "R28") (unit 1) (value "1k") (footprint "Resistor_SMD:R_0805_2012Metric")
     )
     (path "/c452d50b-4fb0-427b-9da6-1adb0c8dc035"

Commit message: Fixes
Parts:
- R8, R9: value 10k -> 2k
Connections:
- net GND: now also J2.3 (GND); no longer J2.5 (GND)
- net IND_B: now also U1.15 (PA10); no longer U1.7 (PA4)
- net PD_PHY_SCL: now also U1.18 (PB6); no longer U1.14 (PA9)
- net PD_PHY_SDA: now also U1.19 (PB7); no longer U1.15 (PA10)
- net SWDCLK: now also J2.5 (SWDCLK); no longer J2.4 (SWCLK)
- net SWDIO: now also J2.6 (SWDIO); no longer J2.2 (SWDIO)
- net nRESET: now also J2.2 (nRESET); no longer J2.3 (nRESET)
Other:
- moved on the sheet: R6, R7
