File: starlink-pd-supply/starlink-pd-supply.kicad_pcb (KiCad board)
At the start: 4 copper layers, 93 x 90 mm, 92 parts, among them J1 USB_C_Receptacle, J2 USB_C_Receptacle, J3 TC2030-SWD, J4 RJE59-188-54A1, J5 RJE59-188-54A1, Q1 PSMN014-80YL, Q2 PSMN014-80YL, Q3 PSMN014-80YL, U1 CDSOT23-0502B, U10 LT3757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

Commit message: Fixes
Parts:
- added R34: NP, Resistor_SMD:R_0805_2012Metric, F.Cu at (49.5, 76.4)
- added R35: 10k, Resistor_SMD:R_0805_2012Metric, F.Cu at (49.5, 78.4)
Connections:
- U5 pad 20: unconnected-(U5-Pad20) -> Net-(R34-Pad2)
Routing:
- net Net-(R34-Pad2): track 0.00 -> 12.2 mm, vias 0 -> 2
- net +3V3: track 225.4 -> 227.3 mm
- net /EN_SINK_B: track 18.2 -> 19.1 mm
- net GND: vias 163 -> 187
Other:
- board text added: "Starlink PD Supply"
- board text removed: "USB-C PD Dishy Power Supply"
