File: starlink-pd-supply/starlink-pd-supply.kicad_pcb (KiCad board)
At the start: 4 copper layers, 93 x 90 mm, 94 parts, among them J1 USB_C_Receptacle, J2 USB_C_Receptacle, J3 TC2030-SWD, J4 RJE59-188-54A1, J5 RJE59-188-54A1, Q1 PSMN014-80YL, Q2 PSMN014-80YL, Q3 PSMN014-80YL, U1 CDSOT23-0502B, U10 LT3757, U11 7490220123, U2 CDSOT23-0502B, U3 PTN5110, U4 PTN5110, U5 STM32L011, U6 AOZ1375DI, U7 AOZ1375DI, U8 LT3685, U9 LT4355

Commit message: Updates to starlink PD design
Parts:
- removed TP1: TestPoint, TestPoint:TestPoint_Pad_D2.0mm
- added C29: 22000 pF, Capacitor_SMD:C_0805_2012Metric, F.Cu at (133.6, 142.7)
- added C30: 10uF 50V, Capacitor_SMD:C_1210_3225Metric, F.Cu at (110.5, 148.9)
- added C31: 10uF 50V, Capacitor_SMD:C_1210_3225Metric, F.Cu at (104.0, 158.9)
- added C32: 0.1uF, Capacitor_SMD:C_0805_2012Metric, F.Cu at (118.4, 156.3)
- added C33: 1uF, Capacitor_SMD:C_0805_2012Metric, F.Cu at (106.8, 165.5)
- added C34: 1uF, Capacitor_SMD:C_0805_2012Metric, F.Cu at (124.9, 150.2)
- added D10: BZX384-C10,115, Custom:SOD-323, F.Cu at (127.2, 158.9)
- added D6: D_Schottky, Diode_SMD:D_SMB, F.Cu at (103.5, 149.7)
- added D7: D_Schottky, Diode_SMD:D_SMB, F.Cu at (112.2, 141.0)
- added D8: BZX384-C10,115, Custom:SOD-323, F.Cu at (142.4, 142.5)
- added D9: LED GREEN, LED_SMD:LED_0805_2012Metric, F.Cu at (111.3, 164.4)
- added Q4: 2N7002NXAKR, Package_TO_SOT_SMD:SOT-23, F.Cu at (115.8, 148.0)
- added Q5: BUK6Y33-60P, Package_TO_SOT_SMD:LFPAK56, F.Cu at (97.0, 158.7)
- added Q6: 2N7002NXAKR, Package_TO_SOT_SMD:SOT-23, F.Cu at (109.3, 157.7)
- added Q7: BSH201,215, Package_TO_SOT_SMD:SOT-23, F.Cu at (115.8, 152.4)
- added R36: 100, Resistor_SMD:R_0805_2012Metric, F.Cu at (127.2, 156.1)
- added R37: 1.3k, Resistor_SMD:R_0805_2012Metric, F.Cu at (142.5, 139.7)
- added U12: MAX4080SAUA+, Custom:uMAX-8, F.Cu at (96.2, 164.2)
- added U13: TLV70327DBVR, Package_TO_SOT_SMD:SOT-23-5, F.Cu at (110.2, 153.2)
- C1, C2, C5, C6, C7: value 2.2uF -> 0.1uF
- C10: value 0.1uF -> 1uF
- C11: value 10uF -> 0.1uF 50V
- C12: value 0.001uF -> 0.1uF 50V
- C13: value 0.001uF -> 22000 pF
- C3: value 0.1uF -> 10uF 50V; footprint Capacitor_SMD:C_0805_2012Metric -> Capacitor_SMD:C_1210_3225Metric
- C4: value 2.2uF -> 10uF 50V; footprint Capacitor_SMD:C_0805_2012Metric -> Capacitor_SMD:C_1210_3225Metric
- C8: value 10uF -> 0.1uF
- C9: value 10uF -> 4.7uF
- L2: footprint Custom:PQ2614BLA-BHA -> Custom:SRP1513CA
- R10: value 20k -> 10k
- R11, R9: value 30k -> 10k
- R12: value 10k -> 0.025 1% 1W; footprint Resistor_SMD:R_0805_2012Metric -> Resistor_SMD:R_1206_3216Metric
- R13: value 10k -> 10K
- R16, R17: value 10m -> 10k; footprint Resistor_SMD:R_1206_3216Metric -> Resistor_SMD:R_0805_2012Metric
- R2: value 10k -> 3k
- R28: value 10k -> 158k
- R34: value NP -> 10k
- R6: value 2k -> 3k
- R7: value 2k -> 1k
- R8: value 20k -> 1k
- U3, U4: value PTN5110 -> MAX5418; footprint Custom:HX2QFN16 -> Custom:TDFN-8
- U5: value STM32L011 -> STM32G0B1CEU6; footprint Custom:UFQFPN-20 -> Custom:UFQFPN-48
- U6, U7: value AOZ1375DI -> TPS1HC30-Q1; footprint Custom:DFN-12L -> Custom:TSSOP-14
- moved R9 118.7 mm to (115.7, 165.2), turned to 0 degrees
- moved R10 117.0 mm to (120.1, 162.2)
- moved R8 113.1 mm to (138.1, 139.7)
- moved C1 112.6 mm to (111.3, 161.4), turned to 0 degrees
- moved R14 111.9 mm to (129.3, 151.6)
- moved U4 110.6 mm to (102.2, 164.3), turned to 0 degrees
- moved R34 110.6 mm to (138.1, 142.7), turned to 0 degrees
- moved C8 108.3 mm to (124.9, 147.2), turned to 0 degrees
- moved R13 107.7 mm to (124.8, 153.2), turned to 0 degrees
- moved R12 106.9 mm to (119.2, 144.1), turned to 0 degrees
- moved R35 106.8 mm to (115.7, 162.2)
- moved R2 106.2 mm to (138.1, 145.6), turned to 0 degrees
- moved R16 105.6 mm to (129.3, 145.7), turned to 0 degrees
- moved C12 104.3 mm to (124.2, 144.2), turned to 0 degrees
- moved C5 104.0 mm to (106.8, 162.5), turned to 0 degrees
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Connections:
- C1 pad 1: /VBUS_A -> /nRESET
- C11 pad 1: +3V3 -> /VBUS_B
- C12 pad 1: Net-(C12-Pad1) -> /VBUS_A
- C13 pad 1: Net-(C13-Pad1) -> /VBUS_B_SW
- C14 pad 1: /VBUS_OR -> Net-(C14-Pad1)
- C2 pad 1: /VBUS_B -> +3V3
- C3 pad 1: GND -> /VBUS_B
- C3 pad 2: /nRESET -> GND
- C4 pad 1: GND -> /VBUS_A
- C4 pad 2: +3V3 -> GND
- C5 pad 1: GND -> +3V3
- C5 pad 2: +3V3 -> GND
- C6 pad 1: Net-(C6-Pad1) -> +3V3
- C7 pad 1: Net-(C7-Pad1) -> +3V3
- C8 pad 1: /VBUS_A -> +3V3
- C9 pad 1: /VBUS_B -> +3V3
- R1 pad 1: /TCPC_ALERT_N -> +3V3
- R1 pad 2: +3V3 -> /nRESET
- R10 pad 1: GND -> /VBUS_A_EN
- R10 pad 2: Net-(R10-Pad2) -> GND
- R11 pad 1: GND -> /VBUS_A_EN
- R11 pad 2: Net-(R11-Pad2) -> GND
- R12 pad 1: /EN_SINK_A -> Net-(D8-Pad1)
- R12 pad 2: GND -> +48V
- R13 pad 1: /EN_SINK_B -> GND
- R13 pad 2: GND -> /48V_EN
- R14 pad 1: /VBUS_FAULT_A -> GND
- R14 pad 2: +3V3 -> /DISHY_POWER_EN
- R15 pad 1: /VBUS_FAULT_B -> Net-(Q4-Pad2)
- R15 pad 2: +3V3 -> Net-(D8-Pad2)
- R16 pad 1: Net-(R16-Pad1) -> GND
- R16 pad 2: /VBUS_A_SW -> Net-(D9-Pad2)
- R17 pad 1: Net-(R17-Pad1) -> /DISHY_SENSE_HIGH_SIDE
- R17 pad 2: /VBUS_B_SW -> GND
- R2 pad 1: /nRESET -> +3V3
- R2 pad 2: +3V3 -> /DIGIPOT_SCL
- R28 pad 1: /~{OUT_EN} -> /DISHY_48V
- R28 pad 2: +3V3 -> /DISHY_SENSE_HIGH_SIDE
- R34 pad 1: +3V3 -> GND
- R34 pad 2: Net-(R34-Pad2) -> /DISHY_SENSE_EN
- R35 pad 1: Net-(R34-Pad2) -> Net-(Q6-Pad2)
- R35 pad 2: GND -> Net-(D10-Pad2)
- R6 pad 2: /TCPC_SCL -> /DIGIPOT_SDA
- R7 pad 1: +3V3 -> Net-(R7-Pad1)
- R7 pad 2: /TCPC_SDA -> GND
- R8 pad 1: GND -> Net-(R8-Pad1)
- R8 pad 2: Net-(R8-Pad2) -> GND
- R9 pad 1: GND -> /SWDCLK
- R9 pad 2: Net-(R9-Pad2) -> GND
- U10 pad 9: /~{OUT_EN} -> /48V_EN
- U11 pad 21: +48V -> /DISHY_48V
- U11 pad 24: +48V -> /DISHY_48V
- U3 pad 1: unconnected-(U3-Pad1) -> +3V3
- U3 pad 2: /EN_SINK_A -> /DIGIPOT_SCL
- U3 pad 3: +3V3 -> /DIGIPOT_SDA
- U3 pad 4: Net-(C6-Pad1) -> +3V3
- U3 pad 5: unconnected-(U3-Pad5) -> GND
- U3 pad 6: unconnected-(U3-Pad6) -> GND
- U3 pad 7: /TCPC_SDA -> Net-(U3-Pad7)
- U3 pad 8: /TCPC_SCL -> Net-(U3-Pad7)
- U3 pad 9: unconnected-(U3-Pad9) -> GND
- U4 pad 1: unconnected-(U4-Pad1) -> +3V3
- U4 pad 2: /EN_SINK_B -> /DIGIPOT_SCL
- U4 pad 3: +3V3 -> /DIGIPOT_SDA
- U4 pad 4: Net-(C7-Pad1) -> GND
- U4 pad 6: unconnected-(U4-Pad6) -> GND
- U4 pad 7: /TCPC_SDA -> Net-(U4-Pad7)
- U4 pad 8: /TCPC_SCL -> Net-(U4-Pad7)
- U4 pad 9: unconnected-(U4-Pad9) -> GND
- U5 pad 10: /TCPC_ALERT_N -> /nRESET
- U5 pad 11: unconnected-(U5-Pad11) -> /48V_EN
- U5 pad 12: GND -> /DISHY_CURRENT_SENSE
- U5 pad 13: +3V3 -> /DISHY_SENSE_HIGH_SIDE
- U5 pad 14: unconnected-(U5-Pad14) -> /DISHY_SENSE_LOW_SIDE
- U5 pad 15: /IND_B -> /DISHY_POWER_EN
- U5 pad 16: /SWDIO -> /DISHY_SENSE_EN
- U5 pad 17: /SWDCLK -> /VBUS_A_EN
- U5 pad 18: /TCPC_SCL -> /VBUS_B_EN
- U5 pad 19: /TCPC_SDA -> unconnected-(U5-Pad19)
- U5 pad 20: Net-(R34-Pad2) -> unconnected-(U5-Pad20)
- U5 pad 3: /nRESET -> unconnected-(U5-Pad3)
- U5 pad 5: /IND_R -> +3V3
- U5 pad 6: /IND_G -> +3V3
- U5 pad 7: /~{OUT_EN} -> GND
- U5 pad 8: unconnected-(U5-Pad8) -> (no net)
- U6 pad 1: /VBUS_A -> GND
- U6 pad 10: Net-(R16-Pad1) -> /VBUS_A_SW
- U6 pad 11: Net-(R16-Pad1) -> Net-(U6-Pad11)
- U6 pad 13: GND -> /VBUS_A
- U6 pad 3: Net-(R8-Pad2) -> GND
- U6 pad 4: /VBUS_FAULT_A -> GND
- U6 pad 5: /EN_SINK_A -> GND
- U6 pad 6: GND -> Net-(R8-Pad1)
- U6 pad 7: Net-(C12-Pad1) -> Net-(U4-Pad7)
- U6 pad 8: Net-(R9-Pad2) -> Net-(U6-Pad11)
- U7 pad 1: /VBUS_B -> GND
- U7 pad 10: Net-(R17-Pad1) -> /VBUS_B_SW
- U7 pad 11: Net-(R17-Pad1) -> Net-(U7-Pad11)
- U7 pad 13: GND -> /VBUS_B
- U7 pad 3: Net-(R10-Pad2) -> GND
- U7 pad 4: /VBUS_FAULT_B -> GND
- U7 pad 5: /EN_SINK_B -> GND
- U7 pad 6: GND -> Net-(R7-Pad1)
- U7 pad 7: Net-(C13-Pad1) -> Net-(U3-Pad7)
- U7 pad 8: Net-(R11-Pad2) -> Net-(U7-Pad11)
- U8 pad 4: /VBUS_OR -> Net-(C14-Pad1)
- U8 pad 5: /VBUS_OR -> Net-(C14-Pad1)
Routing:
- net (no net): track 0.00 -> 499.7 mm, vias 0 -> 19
- net /TCPC_SDA: track 138.6 -> 0.00 mm, vias 3 -> 0
- net /TCPC_ALERT_N: track 131.7 -> 0.00 mm, vias 3 -> 0
- net /TCPC_SCL: track 131.3 -> 0.00 mm, vias 3 -> 0
- net Net-(C14-Pad1): track 0.00 -> 32.7 mm
- net /VBUS_OR: track 41.3 -> 8.60 mm
- net /~{OUT_EN}: track 28.6 -> 0.00 mm, vias 2 -> 0
- net /48V_EN: track 0.00 -> 28.6 mm, vias 0 -> 2
- net /EN_SINK_B: track 19.1 -> 0.00 mm, vias 2 -> 0
- net /EN_SINK_A: track 18.6 -> 0.00 mm, vias 2 -> 0
- net /VBUS_FAULT_B: track 13.6 -> 0.00 mm, vias 2 -> 0
- net /VBUS_FAULT_A: track 12.5 -> 0.00 mm, vias 2 -> 0
- net Net-(R34-Pad2): track 12.2 -> 0.00 mm, vias 2 -> 0
- net Net-(C6-Pad1): track 3.48 -> 0.00 mm
- net Net-(R10-Pad2): track 3.44 -> 0.00 mm
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- added copper zone on F.Cu, net (none)
- removed copper zone on F.Cu, net Net-(R16-Pad1)
- removed copper zone on F.Cu, net Net-(R17-Pad1)

Commit message: Finish layout
Parts:
- removed C5: 0.1uF, Capacitor_SMD:C_0805_2012Metric
- moved U4 113.4 mm to (63.1, 57.8)
- moved R8 113.2 mm to (63.1, 54.8), turned to 180 degrees
- moved C4 109.8 mm to (74.6, 48.8), turned to 180 degrees
- moved C7 109.0 mm to (59.8, 55.7), turned to 90 degrees
- moved R2 106.7 mm to (47.1, 89.9), turned to -90 degrees
- moved C12 104.7 mm to (75.2, 51.6), turned to 180 degrees
- moved C11 103.1 mm to (102.8, 51.7), turned to 180 degrees
- moved C29 102.6 mm to (73.6, 59.5), turned to 180 degrees
- moved D6 101.5 mm to (80.7, 50.9), turned to 90 degrees
- moved C31 101.2 mm to (73.3, 62.4), turned to 180 degrees
- moved R7 101.0 mm to (91.4, 55.1), turned to 180 degrees
- moved R6 100.3 mm to (47.1, 93.4), turned to 90 degrees
- moved U6 99.1 mm to (70.2, 55.5), turned to -90 degrees
- moved R10 96.6 mm to (62.4, 84.7)
- moved C6 95.9 mm to (88.2, 56.0), turned to 90 degrees
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Connections:
- net Net-(C14-Pad1) renamed /3V3_OR
- net Net-(D8-Pad1) renamed /DISHY_48V_HIGH
- R10 pad 1: /VBUS_A_EN -> /VBUS_B_EN
- U12 pad 3: Net-(U12-Pad3) -> unconnected-(U12-Pad3)
- U12 pad 6: Net-(U12-Pad3) -> unconnected-(U12-Pad6)
- U12 pad 7: Net-(U12-Pad3) -> unconnected-(U12-Pad7)
- U5 pad 17: /VBUS_A_EN -> unconnected-(U5-Pad17)
- U5 pad 18: /VBUS_B_EN -> unconnected-(U5-Pad18)
- U5 pad 22: /IND_G -> unconnected-(U5-Pad22)
- U5 pad 23: /IND_B -> /VBUS_A_EN
- U5 pad 24: unconnected-(U5-Pad24) -> /VBUS_B_EN
- U5 pad 30: GND -> unconnected-(U5-Pad30)
- U5 pad 31: (no net) -> unconnected-(U5-Pad31)
- U5 pad 32: +3V3 -> /CC2_A
- U5 pad 42: /IND_R -> unconnected-(U5-Pad42)
- U5 pad 43: unconnected-(U5-Pad43) -> /IND_R
- U5 pad 44: unconnected-(U5-Pad44) -> /IND_G
- U5 pad 45: /DIGIPOT_SCL -> /IND_B
- U5 pad 46: /DIGIPOT_SDA -> unconnected-(U5-Pad46)
- U5 pad 47: unconnected-(U5-Pad47) -> /DIGIPOT_SCL
- U5 pad 48: unconnected-(U5-Pad48) -> /DIGIPOT_SDA
- U5 pad 8: (no net) -> unconnected-(U5-Pad8)
- U6 pad 11: Net-(U6-Pad11) -> unconnected-(U6-Pad11)
- U6 pad 14: Net-(U6-Pad11) -> unconnected-(U6-Pad14)
- U6 pad 8: Net-(U6-Pad11) -> unconnected-(U6-Pad8)
- U7 pad 11: Net-(U7-Pad11) -> unconnected-(U7-Pad11)
- U7 pad 14: Net-(U7-Pad11) -> unconnected-(U7-Pad14)
- U7 pad 8: Net-(U7-Pad11) -> unconnected-(U7-Pad8)
Routing:
- net (no net): track 499.7 -> 0.00 mm, vias 19 -> 0
- net /CC2_B: track 16.8 -> 116.9 mm, vias 1 -> 2
- net /CC1_B: track 13.6 -> 111.3 mm, vias 2 -> 4
- net /DIGIPOT_SDA: track 0.00 -> 91.7 mm, vias 0 -> 3
- net /DISHY_48V: track 0.00 -> 90.0 mm, vias 0 -> 2
- net /DIGIPOT_SCL: track 0.00 -> 86.6 mm, vias 0 -> 3
- net +48V: track 82.2 -> 12.5 mm
- net /DISHY_POWER_EN: track 0.00 -> 68.9 mm, vias 0 -> 2
- net +3V3: track 227.3 -> 295.4 mm, vias 8 -> 4
- net /VBUS_B_EN: track 0.00 -> 67.2 mm, vias 0 -> 2
- net /DISHY_SENSE_EN: track 0.00 -> 59.1 mm, vias 0 -> 3
- net /DISHY_CURRENT_SENSE: track 0.00 -> 57.8 mm, vias 0 -> 2
- net /CC2_A: track 15.3 -> 71.8 mm, vias 1 -> 2
- net /CC1_A: track 12.6 -> 64.5 mm, vias 2 -> 4
- net /DISHY_SENSE_LOW_SIDE: track 0.00 -> 46.9 mm, vias 0 -> 2
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- added copper zone on F.Cu, net /3V3_OR
- added copper zone on F.Cu, net /DISHY_48V
- added copper zone on F.Cu, net /DISHY_48V_HIGH
- removed copper zone on F.Cu, net (none)
Other:
- board text removed: "EIA / TIA 568B Term. Only"

Commit message: Update Version
Connections:
- net Net-(C26-Pad1) renamed /SHIELD_C
- net Net-(C28-Pad1) renamed /SHIELD_D
Routing:
- net /VBUS_B_EN: track 67.2 -> 70.1 mm
- net /48V_EN: track 29.2 -> 30.3 mm
- net /CC2_A: track 71.8 -> 72.8 mm
- net +48V: track 12.5 -> 11.5 mm
- net /DISHY_POWER_EN: track 68.9 -> 68.0 mm
- net /CC1_B: track 111.3 -> 111.9 mm
- net /DISHY_CURRENT_SENSE: track 57.8 -> 57.3 mm
- net GND: vias 104 -> 308
Other:
- outline, holes or cut-outs redrawn
- board text added: "v1.1"
- board text removed: "v1.0"

Commit message: Updated Starlink PD supply
Fixed issues with pfet biasing.
Switched to a synchronous convertor.
Fixed nfet pinout.
Fixed paste under micro
Parts:
- added C35: 220pF, Capacitor_SMD:C_0805_2012Metric, F.Cu at (90.0, 77.0)
- added C36: 22uF 35V, Capacitor_SMD:C_1206_3216Metric, F.Cu at (88.0, 89.4)
- added C5: 1uF 60V, Capacitor_SMD:C_0805_2012Metric, F.Cu at (92.1, 88.3)
- added Q8: PSMN014-80YL, Package_TO_SOT_SMD:LFPAK56, F.Cu at (87.8, 96.7)
- added R38: 47k, Resistor_SMD:R_0805_2012Metric, F.Cu at (100.3, 95.0)
- added R39: 47k, Resistor_SMD:R_0805_2012Metric, F.Cu at (103.2, 84.7)
- C18: value 0.1uF -> 4.7uF
- C19: value 4.7nF -> 0.1uF
- C20: value 4.7uF 10v -> 15nF
- D2, D6, D7: value D_Schottky -> CDBA240LL-G; footprint Diode_SMD:D_SMB -> Custom:SMA
- D4: value D_Schottky -> PMEG10020ELRX; footprint Custom:CFP15B -> Custom:SOD-123W
- R27: value 41.2k 1% -> 48.7k 1%
- R30: value 28k 1% -> 8.66k 1%
- R31: value 0.010 1% 1W -> 8m 1% 1W
- R32: value 580k 1% -> 397k 1%
- R33: value 20k 1% -> 10k 1%
- U10: value LT3757 -> LTC3786; footprint Custom:DFN-10-3X3mm -> Custom:QFN-16
- moved R31 25.9 mm to (83.7, 71.2), turned to 90 degrees
- moved C21 24.3 mm to (107.1, 111.0)
- moved R33 23.8 mm to (94.3, 83.5), turned to -90 degrees
- moved R32 23.4 mm to (94.3, 87.0), turned to -90 degrees
- moved C22 22.3 mm to (84.5, 111.0)
- moved R27 22.0 mm to (87.3, 80.7), turned to -90 degrees
- moved C20 19.5 mm to (92.1, 77.0)
- moved R30 19.2 mm to (91.3, 79.8), turned to 0 degrees
- moved C19 16.8 mm to (87.9, 77.0), turned to 90 degrees
- moved C18 16.4 mm to (87.7, 92.1)
- moved U10 16.1 mm to (89.6, 84.6), turned to 180 degrees
- moved R20 14.3 mm to (108.2, 98.0)
- moved D5 14.2 mm to (108.2, 101.4)
- moved L2 10.6 mm to (77.3, 84.7)
- moved Q3 6.81 mm to (81.1, 97.4)
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Connections:
- C18 pad 1: Net-(C18-Pad1) -> /INTVcc
- C19 pad 1: Net-(C19-Pad1) -> /SOFT_START
- C20 pad 1: Net-(C20-Pad1) -> /CURRENT_THRESH
- D4 pad 1: +48V -> /BOOST
- D4 pad 2: /BOOST_SW -> /INTVcc
- L2 pad 1: /VBUS_OR -> /L_HIGH
- Q3 pad 1: Net-(Q3-Pad1) -> GND
- Q3 pad 2: Net-(Q3-Pad1) -> GND
- Q3 pad 3: Net-(Q3-Pad1) -> GND
- Q3 pad 4: Net-(Q3-Pad4) -> /BOT_GATE
- Q4 pad 2: Net-(Q4-Pad2) -> GND
- Q4 pad 3: GND -> Net-(Q4-D)
- Q6 pad 2: Net-(Q6-Pad2) -> GND
- Q6 pad 3: GND -> Net-(Q6-D)
- R15 pad 1: Net-(Q4-Pad2) -> Net-(Q4-D)
- R27 pad 2: Net-(R27-Pad2) -> /FREQ
- R30 pad 1: Net-(C19-Pad1) -> Net-(C35-Pad1)
- R30 pad 2: Net-(R30-Pad2) -> /CURRENT_THRESH
- R31 pad 1: GND -> /L_HIGH
- R31 pad 2: Net-(Q3-Pad1) -> /VBUS_OR
- R32 pad 1: Net-(R32-Pad1) -> /FB
- R33 pad 2: Net-(R32-Pad1) -> /FB
- R35 pad 1: Net-(Q6-Pad2) -> Net-(Q6-D)
- U10 pad 1: Net-(R30-Pad2) -> /BOOST_SW
- U10 pad 10: /VBUS_OR -> /48V_EN
- U10 pad 2: Net-(R32-Pad1) -> GND
- U10 pad 3: Net-(C18-Pad1) -> /FB
- U10 pad 4: Net-(R27-Pad2) -> /VBUS_OR
- U10 pad 5: GND -> /L_HIGH
- U10 pad 6: Net-(Q3-Pad1) -> /CURRENT_THRESH
- U10 pad 7: Net-(Q3-Pad4) -> /SOFT_START
- U10 pad 8: Net-(C20-Pad1) -> GND
- U10 pad 9: /48V_EN -> /FREQ
Routing:
- net /VBUS_OR: track 28.9 -> 64.1 mm
- net /BOOST_SW: track 0.00 -> 25.6 mm, vias 0 -> 2
- net /L_HIGH: track 0.00 -> 25.0 mm
- net /TOP_GATE: track 0.00 -> 23.0 mm
- net /BOT_GATE: track 0.00 -> 18.4 mm
- net /DISHY_48V: track 90.0 -> 101.6 mm
- net Net-(Q3-Pad4): track 10.6 -> 0.00 mm
- net /INTVcc: track 0.00 -> 8.04 mm
- net /BOOST: track 0.00 -> 7.97 mm
- net Net-(Q3-Pad1): track 7.74 -> 0.00 mm
- net /CURRENT_THRESH: track 0.00 -> 7.16 mm
- net /SOFT_START: track 0.00 -> 5.80 mm
- net Net-(R32-Pad1): track 5.79 -> 0.00 mm
- net /48V_EN: track 30.3 -> 35.7 mm
- net /FB: track 0.00 -> 4.98 mm
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- added copper zone on F.Cu, net /L_HIGH
- removed copper zone on F.Cu, net Net-(Q3-Pad1)
Other:
- board text added: "v1.2"
- board text removed: "v1.1"
