File: starlink-pd-supply/starlink-pd-supply.kicad_sch (KiCad schematic)
At the start: 62 parts

Commit message: WIP
Parts:
- added C?: 4.7uF 10v, Capacitor_SMD:C_0805_2012Metric, symbol Device:C
- added C?: 0.1uF, Capacitor_SMD:C_0805_2012Metric, symbol Device:C
- added C?: 56uF 60V, symbol Device:C_Polarized_US
- added C?: 4.7uF 100V, Capacitor_SMD:C_0805_2012Metric, symbol Device:C
- added C?: 100pF, Capacitor_SMD:C_0805_2012Metric, symbol Device:C
- added C?: 4.7nF, Capacitor_SMD:C_0805_2012Metric, symbol Device:C
- added D?: D_Schottky, symbol Device:D_Schottky
- added L?: 22uH, symbol Device:L
- added Q?: PSMN014-80YL, Package_TO_SOT_SMD:LFPAK56, symbol Custom:PSMN014-80YL
- added R? (x2): 165k 1%, Resistor_SMD:R_0805_2012Metric, symbol Device:R
- added R?: 0.006 1% 1W, Resistor_SMD:R_0805_2012Metric, symbol Device:R
- added R?: 28k 1%, Resistor_SMD:R_0805_2012Metric, symbol Device:R
- added R?: 20k 1%, Resistor_SMD:R_0805_2012Metric, symbol Device:R
- added R?: 580k 1%, Resistor_SMD:R_0805_2012Metric, symbol Device:R
- added R?: 41.2k 1%, Resistor_SMD:R_0805_2012Metric, symbol Device:R
Connections:
- net GND: now also U?.11 (GND), U?.5 (SYNC), C?.2, C?.2, C?.2, C?.2, C?.2, C?.2, R?.1, R?.1, R?.1, R?.1
- net VBUS_A_SW: now also Q?.1 (S), Q?.2 (S), Q?.3 (S); no longer Q?.5 (D)
- net VBUS_B_SW: now also Q?.1 (S), Q?.2 (S), Q?.3 (S); no longer Q?.5 (D)
- net VBUS_OR: now also Q?.5 (D), Q?.5 (D), U?.10 (Vin), L?.1, R?.2; no longer Q?.1 (S), Q?.1 (S), Q?.2 (S), Q?.2 (S), Q?.3 (S), Q?.3 (S)
- net at U?.1 (Vc): now also C?.1, R?.2
- net at U?.2 (FBX): now also R?.1, R?.2
- net at U?.3 (SS): now also C?.1
- net at U?.4 (RT): now also R?.2
- net at U?.6 (SENSE): now also Q?.1 (S), Q?.2 (S), Q?.3 (S), R?.2
- net at U?.7 (GATE): now also Q?.4 (G)
- net at U?.8 (INTVcc): now also C?.1
- net at U?.9 (~{SHDN}/UVLO): now also R?.1, R?.2
- new net: D?.2 (A), L?.2, Q?.5 (D)
- new net: C?.1, R?.1
- new net +48V: C?.1, C?.1, D?.1 (K), R?.2
Other:
- moved on the sheet: Q?, R?, U?

Commit message: WIP
Parts:
- removed C?: 100pF, Capacitor_SMD:C_0805_2012Metric, symbol Device:C
- added C22, C23, C24: 15uF 60V, Custom:Panasonic-F8, symbol Device:C_Polarized_US
- C1, C2, C4, C5, C6, C7: renamed from C?; footprint (none) -> Capacitor_SMD:C_0805_2012Metric
- C21: renamed from C?; value 56uF 60V -> 15uF 60V; footprint (none) -> Custom:Panasonic-F8
- D4: renamed from D?; footprint (none) -> Custom:CFP15B
- J1, J2: renamed from J?; footprint (none) -> Custom:Wurth_632723300011
- L2: renamed from L?; value 22uH -> 15uH; footprint (none) -> Custom:PQ2614BLA-BHA
- R31: renamed from R?; value 0.006 1% 1W -> 0.010 1% 1W; footprint Resistor_SMD:R_0805_2012Metric -> Resistor_SMD:R_1206_3216Metric
- R6, R7: renamed from R?; footprint (none) -> Resistor_SMD:R_0805_2012Metric
- U10: renamed from U?; footprint (none) -> Custom:DFN-10-3X3mm
- U9: renamed from U?; footprint (none) -> Custom:DE14
- gave numbers to parts that had none: 61
Connections:
- net +48V: now also C22.1, C23.1, C24.1
- net GND: now also U9.15 (GND), C22.2, C23.2, C24.2
Other:
- moved on the sheet: C18, C19, C20, C21, C25, D4, L2, Q3, R27, R28, R29, R30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

Commit message: WIP
Parts:
- removed R21, R23: 12.7k 1%, Resistor_SMD:R_0805_2012Metric, symbol Device:R
- removed R22, R29: 165k 1%, Resistor_SMD:R_0805_2012Metric, symbol Device:R
- added D5: LED, LED_SMD:LED_0805_2012Metric, symbol Device:LED
- added H1, H2, H3, H4: MountingHole, MountingHole:MountingHole_4mm_Pad_Via, symbol Mechanical:MountingHole
- R20, R28: value 165k 1% -> 10k
Connections:
- net OUT_EN is gone; now on net ~{OUT_EN}: U5.7 (PA4)
- net +3V3: now also R28.2
- net +48V: now also D5.1 (K)
- net GND: now also R20.1, U9.10 (~{PWRFLT2}), U9.11 (~{FUSEFLT2}), U9.12 (~{FUSEFLT1}), U9.13 (~{PWRFLT1}), U9.14 (MON1), U9.6 (~{VDSFLT}), U9.8 (SET), U9.9 (MON2)
- net VBUS_A_SW: no longer R20.2
- net VBUS_OR: no longer R28.2
- net BOOST_SW: now reaches D4.2 (A), L2.2, Q3.5 (D)
- net ~{OUT_EN}: now reaches R28.1, U10.9 (~{SHDN}/UVLO)
- net EN_SINK_B: now reaches R13.1, U4.2 (EN_SNK1), U7.5 (EN)
- net CC2_A: now reaches J1.B5 (CC2), U3.14 (CC2)
- net CC2_A: now also U1.2; no longer U1.1
- net CC1_A: now reaches J1.A5 (CC1), U3.13 (CC1)
- net CC1_A: now also U1.1; no longer U1.2
- net CC2_B: now reaches J2.B5 (CC2), U4.14 (CC2)
- net CC2_B: now also U2.2; no longer U2.1
- net CC1_B: now reaches J2.A5 (CC1), U4.13 (CC1)
- net CC1_B: now also U2.1; no longer U2.2
- net EN_SINK_A: now reaches R12.1, U3.2 (EN_SNK1), U6.5 (EN)
- new net: D5.2 (A), R20.2

Commit message: Dishy supply rev 1 complete
Parts:
- added C26, C27, C28: 1000p 2kV, Capacitor_SMD:C_1206_3216Metric, symbol Device:C
- added J3: TC2030-SWD, Custom:TC2030-IDC-FP, symbol Custom:TC2030-SWD
- added J4, J5: RJE59-188-54A1, Custom:RJE59-188-54A1, symbol Custom:RJE59-188-54A1
- added R21, R22, R23, R29: 75, Resistor_SMD:R_0805_2012Metric, symbol Device:R
- added U11: 7490220123, Custom:7490220123, symbol Custom:7490220123
Connections:
- net +3V3: now also J3.1 (VCC)
- net +48V: now also U11.21 (CX2), U11.24 (CX1)
- net GND: now also C26.2, C27.2, C28.2, J3.3 (GND), U11.15 (CX4), U11.18 (CX3)
- net SWDCLK: now also J3.5 (SWDCLK)
- net SWDIO: now also J3.6 (SWDIO)
- net nRESET: now also J3.2 (nRESET)
- new net: C26.1, J4.S (SHIELD)
- new net: C28.1, J5.S (SHIELD)
- new net: R23.1, U11.7 (CD3)
- new net: C27.1, R21.2, R22.2, R23.2, R29.2
- new net: R22.1, U11.4 (CD2)
- new net: R21.1, U11.1 (CD1)
- new net: R29.1, U11.10 (CD4)
- new net CPE_1_N: J4.2 (O), U11.3 (D1-)
- new net CPE_1_P: J4.1 (O/W), U11.2 (D1+)
- new net CPE_2_N: J4.4 (B), U11.8 (D3+)
- new net CPE_2_P: J4.3 (G/W), U11.5 (D2+)
- new net CPE_3_N: J4.6 (G), U11.6 (D2-)
- new net CPE_3_P: J4.5 (B/W), U11.9 (D3-)
- new net CPE_4_N: J4.8 (Br), U11.12 (D4-)
- new net CPE_4_P: J4.7 (Br/W), U11.11 (D4+)
- new net Dishy_1_N: J5.2 (O), U11.22 (X1-)
- new net Dishy_1_P: J5.1 (O/W), U11.23 (X1+)
- new net Dishy_2_N: J5.4 (B), U11.17 (X3+)
- new net Dishy_2_P: J5.3 (G/W), U11.20 (X2+)
- new net Dishy_3_N: J5.6 (G), U11.19 (X2-)
- new net Dishy_3_P: J5.5 (B/W), U11.16 (X3-)
- new net Dishy_4_N: J5.8 (Br), U11.13 (X4-)
- new net Dishy_4_P: J5.7 (Br/W), U11.14 (X4+)
Other:
- moved on the sheet: C14, C15, C16, C17, D2, D3, L1, R18, R19, R24, R25, R26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

Commit message: Fixes
Parts:
- added R34: NP, Resistor_SMD:R_0805_2012Metric, symbol Device:R
- added R35: 10k, Resistor_SMD:R_0805_2012Metric, symbol Device:R
Connections:
- net +3V3: now also R34.1
- net GND: now also R35.2
- net at U5.20 (PB9/BOOT0): now also R34.2, R35.1
Changed lines of the file:
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@@
   (junction (at 391.795 90.805) (diameter 0) (color 0 0 0 0)
   )
+  (junction (at 98.425 206.375) (diameter 0) (color 0 0 0 0)
+  )
   (junction (at 185.42 26.035) (diameter 0) (color 0 0 0 0)
   )
@@
     (stroke (width 0) (type default) (color 0 0 0 0))
   )
+  (wire (pts (xy 98.425 206.375) (xy 98.425 208.28))
+    (stroke (width 0) (type default) (color 0 0 0 0))
+  )
   (wire (pts (xy 66.675 132.715) (xy 66.675 135.255))
     (stroke (width 0) (type default) (color 0 0 0 0))
@@
     (stroke (width 0) (type default) (color 0 0 0 0))
   )
+  (wire (pts (xy 98.425 193.675) (xy 98.425 197.485))
+    (stroke (width 0) (type default) (color 0 0 0 0))
+  )
   (wire (pts (xy 99.06 283.21) (xy 99.06 285.75))
     (stroke (width 0) (type default) (color 0 0 0 0))
@@
     (stroke (width 0) (type default) (color 0 0 0 0))
   )
+  (wire (pts (xy 108.585 233.045) (xy 106.68 233.045))
+    (stroke (width 0) (type default) (color 0 0 0 0))
+  )
   (wire (pts (xy 246.38 51.435) (xy 246.38 26.035))
     (stroke (width 0) (type default) (color 0 0 0 0))
@@
     (stroke (width 0) (type default) (color 0 0 0 0))
   )
+  (wire (pts (xy 98.425 206.375) (xy 108.585 206.375))
+    (stroke (width 0) (type default) (color 0 0 0 0))
+  )
   (wire (pts (xy 346.71 53.975) (xy 351.155 53.975))
     (stroke (width 0) (type default) (color 0 0 0 0))
@@
     (stroke (width 0) (type default) (color 0 0 0 0))
   )
+  (wire (pts (xy 108.585 206.375) (xy 108.585 233.045))
+    (stroke (width 0) (type default) (color 0 0 0 0))
+  )
   (wire (pts (xy 51.435 31.115) (xy 51.435 57.785))
     (stroke (width 0) (type default) (color 0 0 0 0))
@@
     (stroke (width 0) (type default) (color 0 0 0 0))
   )
+  (wire (pts (xy 98.425 205.105) (xy 98.425 206.375))
+    (stroke (width 0) (type default) (color 0 0 0 0))
+  )
   (wire (pts (xy 434.975 38.735) (xy 449.58 38.735))
     (stroke (width 0) (type default) (color 0 0 0 0))
@@
     (stroke (width 0) (type default) (color 0 0 0 0))
   )
+  (wire (pts (xy 98.425 215.9) (xy 98.425 219.075))
+    (stroke (width 0) (type default) (color 0 0 0 0))
+  )
   (wire (pts (xy 98.425 160.02) (xy 101.6 160.02))
     (stroke (width 0) (type default) (color 0 0 0 0))
@@
     (pin "2")
   )
+  (symbol (lib_id "power:+3V3") (at 98.425 193.675 0) (unit 1)
+    (in_bom yes) (on_board yes) (fields_autoplaced)
+    (property "Reference" "#PWR0103" (id 0) (at 98.425 197.485 0)
+      (effects (font (size 1.27 1.27)) hide)
+    )
+    (property "Value" "+3V3" (id 1) (at 98.425 190.0705 0))
+    (property "Footprint" "" (id 2) (at 98.425 193.675 0)
+      (effects (font (size 1.27 1.27)) hide)
+    )
+    (property "Datasheet" "" (id 3) (at 98.425 193.675 0)
+      (effects (font (size 1.27 1.27)) hide)
+    )
+    (pin "1")
+  )
   (symbol (lib_id "power:GND") (at 57.15 187.96 0) (unit 1)
     (in_bom yes) (on_board yes) (fields_autoplaced)
@@
     (pin "2")
   )
+  (symbol (lib_id "power:GND") (at 98.425 219.075 0) (unit 1)
+    (in_bom yes) (on_board yes) (fields_autoplaced)
+    (property "Reference" "#PWR0104" (id 0) (at 98.425 225.425 0)
+      (effects (font (size 1.27 1.27)) hide)
+    )
+    (property "Value" "GND" (id 1) (at 98.425 223.6375 0))
+    (property "Footprint" "" (id 2) (at 98.425 219.075 0)
+      (effects (font (size 1.27 1.27)) hide)
+    )
+    (property "Datasheet" "" (id 3) (at 98.425 219.075 0)
+      (effects (font (size 1.27 1.27)) hide)
+    )
+    (pin "1")
+  )
   (symbol (lib_id "power:+3V3") (at 185.42 56.515 0) (unit 1)
     (in_bom yes) (on_board yes) (fields_autoplaced)
@@
     (pin "9")
   )
+  (symbol (lib_id "Device:R") (at 98.425 212.09 0) (unit 1)
+    (in_bom yes) (on_board yes) (fields_autoplaced)
+    (property "Reference" "R35" (id 0) (at 100.203 211.1815 0)
+      (effects (font (size 1.27 1.27)) (justify left))
+    )
+    (property "Value" "10k" (id 1) (at 100.203 213.9566 0)
+      (effects (font (size 1.27 1.27)) (justify left))
+    )
+    (property "Footprint" "Resistor_SMD:R_0805_2012Metric" (id 2) (at 96.647 212.09 90)
+      (effects (font (size 1.27 1.27)) hide)
+    )
+    (property "Datasheet" "~" (id 3) (at 98.425 212.09 0)
+      (effects (font (size 1.27 1.27)) hide)
+    )
+    (pin "1")
+    (pin "2")
+  )
   (symbol (lib_id "Device:R") (at 344.805 171.45 0) (unit 1)
     (in_bom yes) (on_board yes) (fields_autoplaced)
@@
     (pin "5")
   )
+  (symbol (lib_id "Device:R") (at 98.425 201.295 0) (unit 1)
+    (in_bom yes) (on_board yes) (fields_autoplaced)
+    (property "Reference" "R34" (id 0) (at 100.203 200.3865 0)
+      (effects (font (size 1.27 1.27)) (justify left))
+    )
+    (property "Value" "NP" (id 1) (at 100.203 203.1616 0)
+      (effects (font (size 1.27 1.27)) (justify left))
+    )
+    (property "Footprint" "Resistor_SMD:R_0805_2012Metric" (id 2) (at 96.647 201.295 90)
+      (effects (font (size 1.27 1.27)) hide)
+    )
+    (property "Datasheet" "~" (id 3) (at 98.425 201.295 0)
+      (effects (font (size 1.27 1.27)) hide)
+    )
+    (pin "1")
+    (pin "2")
+  )
   (symbol (lib_id "power:GND") (at 130.81 262.255 0) (unit 1)
     (in_bom yes) (on_board yes) (fields_autoplaced)
@@
       (reference "#PWR0102") (unit 1) (value "GND") (footprint "")
     )
+    (path "/09e41b55-2ad8-4dc9-bacd-b18f0e252339"
+      (reference "#PWR0103") (unit 1) (value "+3V3") (footprint "")
+    )
+    (path "/45d57b7f-869c-4644-bdd2-d94ece7dc45e"
+      (reference "#PWR0104") (unit 1) (value "GND") (footprint "")
+    )
     (path "/cc2181ef-0a25-4bc5-81dc-d0104cbb5d54"
       (reference "C1") (unit 1) (value "2.2uF") (footprint "Capacitor_SMD:C_0805_2012Metric")
@@
       (reference "R33") (unit 1) (value "20k 1%") (footprint "Resistor_SMD:R_0805_2012Metric")
     )
+    (path "/aea2edfd-e787-4e87-b031-d101d21f1827"
+      (reference "R34") (unit 1) (value "NP") (footprint "Resistor_SMD:R_0805_2012Metric")
+    )
+    (path "/63ae8269-8404-4c00-a98a-b1210b0ec8bd"
+      (reference "R35") (unit 1) (value "10k") (footprint "Resistor_SMD:R_0805_2012Metric")
+    )
     (path "/4f350a4f-2e5d-4159-b03a-ceba2207cf9b"
