File: starlink-pd-supply/starlink-pd-supply.kicad_sch (KiCad schematic)
At the start: 97 parts, among them J1 USB_C_Receptacle, J2 USB_C_Receptacle, J3 TC2030-SWD, J4 RJE59-188-54A1, J5 RJE59-188-54A1, Q1 PSMN014-80YL, Q2 PSMN014-80YL, Q3 PSMN014-80YL, U1 CDSOT23-0502B, U10 LT3757, U11 7490220123, U2 CDSOT23-0502B, U8 LT3685, U9 LT4355

Commit message: Updates to starlink PD design
Parts:
- added C1, C2, C32, C5, C8: 0.1uF, Capacitor_SMD:C_0805_2012Metric, symbol Device:C
- added C10: 1uF, Capacitor_SMD:C_0805_2012Metric, symbol Device:C
- added C9: 4.7uF, Capacitor_SMD:C_0805_2012Metric, symbol Device:C
- added R1, R10, R11, R9: 10k, Resistor_SMD:R_0805_2012Metric, symbol Device:R
- added R13: 10K, Resistor_SMD:R_0805_2012Metric, symbol Device:R
- added R2, R6: 3k, Resistor_SMD:R_0805_2012Metric, symbol Device:R
- added U12: MAX4080SAUA+, Custom:uMAX-8, symbol Custom:MAX4080SAUA+
- C11, C12, C13, C29, C6, C7: renamed from C?; footprint (none) -> Capacitor_SMD:C_0805_2012Metric
- C3, C30, C31, C4: renamed from C?; footprint (none) -> Capacitor_SMD:C_1210_3225Metric
- Q5: renamed from Q?; footprint (none) -> Package_TO_SOT_SMD:LFPAK56
- R12: renamed from R?; value 0.010 1% 1W -> 0.025 1% 1W
- R7, R8: renamed from R?; footprint (none) -> Resistor_SMD:R_0805_2012Metric
- gave numbers to parts that had none: 25
Connections:
- net ~{OUT_EN} is gone; now on net 48V_EN: U10.9 (~{SHDN}/UVLO)
- net +3V3: now also U5.32 (VDDIO2), U5.4 (VBAT), U5.5 (VREF+), U5.6 (VDD/VDDA), C10.1, C2.1, C5.1, C8.1, C9.1, R1.1, R2.1, R6.1; no longer U13.3 (EN)
- net +48V: now also C32.1, U12.1 (RS+), U12.2 (VCC)
- net CC1_A: now also U5.28 (PA8), U5.29 (PA9)
- net CC1_B: now also U5.38 (PD0), U5.39 (PD1)
- net CC2_A: now also U5.27 (PB15), U5.32 (VDDIO2)
- net CC2_B: now also U5.40 (PD2), U5.41 (PD3)
- net DIGIPOT_SCL: now also U5.45 (PB6), R2.2
- net DIGIPOT_SDA: now also U5.46 (PB7), R6.2
- net DISHY_POWER_EN: now also U5.15 (PA4)
- net DISHY_SENSE_EN: now also U13.3 (EN), U5.16 (PA5)
- net DISHY_SENSE_HIGH_SIDE: now also U5.13 (PA2)
- net DISHY_SENSE_LOW_SIDE: now also U5.14 (PA3)
- net GND: now also U5.30 (VSS), U5.49 (VSS), U5.7 (VSS/VSSA), C1.2, C10.2, C2.2, C32.2, C5.2, C8.2, C9.2, R10.2, R11.2, R13.1, R9.2, U12.4 (GND)
- net IND_B: now also U5.23 (PB11)
- net IND_G: now also U5.22 (PB10)
- net IND_R: now also U5.42 (PB3)
- net SWDCLK: now also U5.36 (PA14-BOOT0), R9.1
- net SWDIO: now also U5.35 (PA13)
- net VBUS_A_EN: now also U5.17 (PA6), R10.1, R11.1
- net VBUS_B_EN: now also U5.18 (PA7)
- net nRESET: now also U5.10 (PF2-NRST), C1.1, R1.2
- net 48V_EN: now reaches U5.11 (PA0)
- net 48V_EN: now also R13.2
- net DISHY_CURRENT_SENSE: now reaches U5.12 (PA1)
- net DISHY_CURRENT_SENSE: now also U12.5 (OUT)
- net at D8.1 (K), Q5.1 (S), Q5.2 (S)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: now also U12.8 (RS-)
- new net: U12.3 (NC), U12.6 (NC), U12.7 (NC)
Other:
- moved on the sheet: C18, C19, C20, C21, C22, C23, C24, C25, C26, C34, D1, D4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

Commit message: Finish layout
Parts:
- removed C5: 0.1uF, Capacitor_SMD:C_0805_2012Metric, symbol Device:C
Connections:
- net +3V3: no longer U5.32 (VDDIO2)
- net DIGIPOT_SCL: now also U5.47 (PB8); no longer U5.45 (PB6)
- net DIGIPOT_SDA: now also U5.48 (PB9); no longer U5.46 (PB7)
- net GND: no longer U5.30 (VSS)
- net IND_B: now also U5.45 (PB6); no longer U5.23 (PB11)
- net IND_G: now also U5.44 (PB5); no longer U5.22 (PB10)
- net IND_R: now also U5.43 (PB4); no longer U5.42 (PB3)
- net VBUS_A_EN: now also U5.23 (PB11); no longer R10.1, U5.17 (PA6)
- net VBUS_B_EN: now also R10.1, U5.24 (PB12); no longer U5.18 (PA7)
- net DISHY_48V_HIGH: now reaches D8.1 (K), Q5.1 (S), Q5.2 (S), Q5.3 (S), R12.1, U12.8 (RS-)
- net 3V3_OR: now reaches C14.1, D6.1 (K), D7.1 (K), U8.4 (Vin), U8.5 (RUN/SS)
- now unconnected: U12.3 (NC), U12.6 (NC), U12.7 (NC), U6.11 (NC), U6.14 (NC), U6.8 (NC), U7.11 (NC), U7.14 (NC), U7.8 (NC)
Other:
- moved on the sheet: C1, C10, C2, C8, C9, R1, R10, R11, R2, R6

Commit message: Update Version
Connections:
- net SHIELD_C: now reaches C26.1, J4.S (SHIELD)
- net SHIELD_D: now reaches C28.1, J5.S (SHIELD)
Changed lines of the file:
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@@
+    (effects (font (size 1.27 1.27)) (justify left bottom))
+  )
+  (label "SHIELD_D" (at 452.12 246.38 0)
     (effects (font (size 1.27 1.27)) (justify left bottom))
   )
@@
     (effects (font (size 1.27 1.27)) (justify left bottom))
   )
+  (label "SHIELD_C" (at 302.26 244.475 0)
+    (effects (font (size 1.27 1.27)) (justify left bottom))
+  )

Commit message: Updated Starlink PD supply
Fixed issues with pfet biasing.
Switched to a synchronous convertor.
Fixed nfet pinout.
Fixed paste under micro
Parts:
- removed U10: LT3757, Custom:DFN-10-3X3mm, symbol Custom:LT3757
- added C35: 220pF, Capacitor_SMD:C_0805_2012Metric, symbol Device:C
- added C36: 22uF 35V, Capacitor_SMD:C_1206_3216Metric, symbol Device:C
- added C5: 1uF 60V, Capacitor_SMD:C_0805_2012Metric, symbol Device:C
- added Q8: PSMN014-80YL, Package_TO_SOT_SMD:LFPAK56, symbol Custom:PSMN014-80YL
- added R38, R39: 47k, Resistor_SMD:R_0805_2012Metric, symbol Device:R
- added U10: LTC3786, Custom:QFN-16, symbol Custom:LTC3786
- C18: value 0.1uF -> 4.7uF
- C19: value 4.7nF -> 0.1uF
- C20: value 4.7uF 10v -> 15nF
- D2, D6, D7: value D_Schottky -> CDBA240LL-G; footprint Diode_SMD:D_SMB -> Custom:SMA
- D4: value D_Schottky -> PMEG10020ELRX; footprint Custom:CFP15B -> Custom:SOD-123W
- Q4, Q6: symbol Device:Q_NMOS_GDS -> Device:Q_NMOS_GSD
- R27: value 41.2k 1% -> 48.7k 1%
- R30: value 28k 1% -> 8.66k 1%
- R31: value 0.010 1% 1W -> 8m 1% 1W
- R32: value 580k 1% -> 397k 1%
- R33: value 20k 1% -> 10k 1%
Connections:
- net +48V: now also Q8.5 (D); no longer D4.1 (K)
- net 48V_EN: now also U10.10 (RUN)
- net BOOST_SW: now also C5.2, Q8.1 (S), Q8.2 (S), Q8.3 (S), U10.1 (SW); no longer D4.2 (A)
- net DISHY_48V: now also R39.2
- net DISHY_48V_HIGH: now also R38.2
- net GND: now also Q3.1 (S), Q3.2 (S), Q3.3 (S), Q4.2 (S), Q6.2 (S), C35.2, C36.1, U10.11 (GND), U10.17 (GND), U10.2 (PGOOD), U10.8 (PLLIN/MODE); no longer Q4.3 (S), Q6.3 (S), R31.1
- net VBUS_OR: now also R31.2, C36.2, U10.14 (VBIAS), U10.4 (SENSE+); no longer L2.1
- net at D8.2 (A), Q5.4 (G), R15.2: now also R38.1
- net at R15.1: now also Q4.3 (D); no longer Q4.2 (D)
- net CURRENT_THRESH: now reaches C20.1
- net CURRENT_THRESH: now also R30.2, U10.6 (ITH)
- net INTVcc: now reaches C18.1
- net INTVcc: now also D4.2 (A), U10.13 (INTVcc)
- net at R30.1: now also C35.1; no longer C19.1
- net FB: now reaches R32.1, R33.2
- net FB: now also U10.3 (VFB)
- net BOT_GATE: now reaches Q3.4 (G)
- net BOT_GATE: now also U10.12 (BG)
- net at R35.1: now also Q6.3 (D); no longer Q6.2 (D)
- net at D10.2 (A), Q7.1 (G), R35.2: now also R39.1
- net FREQ: now reaches R27.2
- net FREQ: now also U10.9 (FREQ)
- new net BOOST: C5.1, D4.1 (K), U10.15 (BOOST)
- new net L_HIGH: L2.1, R31.1, U10.5 (SENSE-)
- new net SOFT_START: C19.1, U10.7 (SS)
- new net TOP_GATE: Q8.4 (G), U10.16 (TG)
Other:
- moved on the sheet: C21, C22, C23, C24, C25, D5, L2, Q3, R13, R20, R31, R32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

Commit message: Fix dumb bugs
Parts:
- C20: value 15nF -> 220pF
- C35: value 220pF -> 15nF
Changed lines of the file:
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@@
       (effects (font (size 1.27 1.27)) (justify left))
     )
-    (property "Value" "220pF" (at 346.075 62.23 0)
+    (property "Value" "15nF" (at 346.075 62.23 0)
       (effects (font (size 1.27 1.27)) (justify left))
     )
@@
   (symbol (lib_id "Device:C") (at 334.01 71.755 0) (unit 1)
     (in_bom yes) (on_board yes) (dnp no) (fields_autoplaced)
-    (property "Reference" "C20" (at 337.185 71.12 0)
-      (effects (font (size 1.27 1.27)) (justify left))
-    )
-    (property "Value" "15nF" (at 337.185 73.66 0)
-      (effects (font (size 1.27 1.27)) (justify left))
-    )
+    (property "Reference" "C20" (at 337.82 70.485 0)
+      (effects (font (size 1.27 1.27)) (justify left))
+    )
+    (property "Value" "220pF" (at 337.82 73.025 0)
+      (effects (font (size 1.27 1.27)) (justify left))
+    )
