File: bilge-vacuum/bilge-vacuum.kicad_sch (KiCad schematic)
At the start: 31 parts, among them J1 TC2030-SWD, SW1 SW_Push, U1 STM32G0B1CEU6, U2 TPS2660

Commit message: Part selections
Other:
- note added: "Display: NHD-C12864A1Z-FSW-FBW-HTT 3v3 Buck: LTC3851 24v Boost: LTC3786 FRAM: FM25V20A-DGQ 4-20ma Prot: MAX14626ETT+T High Side Switches: TPS1HC30-Q1"
Changed lines of the file:
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@@
   (junction (at 447.04 60.96) (diameter 0) (color 0 0 0 0)
   )
-  (junction (at 342.9 99.06) (diameter 0) (color 0 0 0 0)
-  )
   (junction (at 119.38 130.175) (diameter 0) (color 0 0 0 0)
   )
@@
     (stroke (width 0) (type default))
   )
-  (wire (pts (xy 342.9 99.06) (xy 342.9 97.79))
-    (stroke (width 0) (type default))
-  )
   (wire (pts (xy 279.4 78.74) (xy 261.62 78.74))
     (stroke (width 0) (type default))
@@
     (stroke (width 0) (type default))
   )
+  (text "Display: NHD-C12864A1Z-FSW-FBW-HTT\n3v3 Buck: LTC3851\n24v Boost: LTC3786\nFRAM: FM25V20A-DGQ\n4-20ma Prot: MAX14626ETT+T\nHigh Side Switches: TPS1HC30-Q1"
+    (at 186.69 43.815 0)
+    (effects (font (size 1.27 1.27)) (justify left bottom))
+  )
   (label "IND_R" (at 92.075 93.345 180) (fields_autoplaced)

Commit message: WIP
Parts:
- added C12, C13, C33: 0.1uF 25V, symbol Device:C_Small
- added C14: 330pF 25V, symbol Device:C_Small
- added C15: 2200pF 25V, symbol Device:C_Small
- added C16, C23, C29: 0.1uF 50V, symbol Device:C_Small
- added C17, C30: 4.7uF 50V, symbol Device:C_Small
- added C18, C19: 330uF 10V, symbol Device:C_Polarized_US
- added C20: 47pF 10V, symbol Device:C_Small
- added C21: 0.047uF 25V, symbol Device:C_Small
- added C22: 22uF 25V, symbol Device:C_Polarized_US
- added C24: 220uF 50V, symbol Device:C_Polarized_US
- added C25, C26, C27, C28: 22uF 50V, symbol Device:C_Small
- added C31: 220pF 25V, symbol Device:C_Small
- added C32: 15000pF 25V, symbol Device:C_Small
- added D4, D6: D_Schottky, symbol Device:D_Schottky
- added D5, D7: GREEN, symbol Device:LED
- added L1: 0.68uH 15A, symbol Device:L
- added L2: 10.2uH 8A, symbol Device:L
- added Q1, Q2, Q3, Q4: PSMN014-80YL, Package_TO_SOT_SMD:LFPAK56, symbol Custom Parts:PSMN014-80YL
- added R13: 82.5k, symbol Device:R
- added R14: 15k, symbol Device:R
- added R15: 154k 1%, symbol Device:R_Small
- added R16: 48.7k 1%, symbol Device:R_Small
- added R17: 3.01k, symbol Device:R_Small
- added R18: 30.1k, symbol Device:R_Small
- added R19: 500, symbol Device:R
- added R20: 26.1k 1%, symbol Device:R_Small
- added R21: 53.6k 1%, symbol Device:R_Small
- added R22: 232k 1%, symbol Device:R_Small
- added R23: 12.1k 1%, symbol Device:R_Small
- added R24: 8.87k 1%, symbol Device:R
- added R25, R27: 10k, symbol Device:R
- added R26: 2.2k, symbol Device:R
- added U3: LTC3786, Custom:QFN-16, symbol Custom Parts:LTC3786
- added U4: LTC3851, Custom Parts:QFN-16, symbol Custom Parts:LTC3851
Connections:
- net +12V: now also C22.1, C23.1, L2.1, Q1.5 (D), R20.1, U3.14 (VBIAS), U3.4 (SENSE+), U4.11 (VIN)
- net +3.3V: now also R27.2
- net GND: now also C12.1, C13.1, C14.1, C17.2, C18.2, C19.2, C22.2, C24.2, C25.2, C26.2, C27.2, C28.2, C30.1, C31.1, C32.1, C33.1, Q2.1 (S), Q2.2 (S), Q2.3 (S), Q3.1 (S), Q3.2 (S), Q3.3 (S), R13.1, R14.1, R16.2, R19.2, R23.1, R25.1, R26.2, U3.11 (GND), U3.17 (GND), U3.9 (FREQ), U4.17 (GND), U4.8 (GND)
- new net: C31.2, R24.2, U3.6 (ITH)
- new net: C16.1, D4.1 (K), U4.12 (BOOST)
- new net: C16.2, L1.1, Q1.1 (S), Q1.2 (S), Q1.3 (S), Q2.5 (D), R17.1, U4.14 (SW)
- new net: C33.2, U3.7 (SS)
- new net: Q2.4 (G), U4.9 (BG)
- new net: Q3.4 (G), U3.12 (BG)
- new net: C29.2, L2.2, Q3.5 (D), Q4.1 (S), Q4.2 (S), Q4.3 (S), R21.2, U3.1 (SW)
- new net: D7.1 (K), R26.1
- new net: D6.2 (A), U3.13 (INTVcc)
- new net: C20.1, R15.2, R16.1, U4.4 (FB)
- new net: C24.1, C25.1, C26.1, C27.1, C28.1, D7.2 (A), Q4.5 (D), R22.1
- new net: R22.2, R23.2, U3.3 (VFB)
- new net: C14.2, C15.2, U4.3 (ITH)
- new net: C21.1, R17.2, R18.1, U4.6 (SENSE_P)
- new net: Q4.4 (G), U3.16 (TG)
- new net: C23.2, R20.2, R21.1, U3.5 (SENSE-)
- new net: C17.1, D4.2 (A), U4.10 (INTVCC)
- new net: D5.1 (K), R19.1
- new net: C32.2, R24.1
- new net: C12.2, R13.2, U4.16 (FREQ/PLLFLTR)
- new net: Q1.4 (G), U4.13 (TG)
- new net: C13.2, U4.2 (TK/SS)
- new net: C15.1, R14.2
- new net +3V3: C18.1, C19.1, C20.2, C21.2, D5.2 (A), L1.2, R15.1, R18.2, U4.5 (SENSE_N)
- new net 24V_INTVCC: C29.1, C30.2, D6.1 (K), U3.15 (BOOST), U3.8 (PLLIN/MODE)
- new net 24V_PGOOD: R27.1, U3.2 (PGOOD)
- new net 24_SUP_EN: R25.2, U3.10 (RUN)
Other:
- note added: "12V to 24V Boost"
- note added: "12V to 3.3V Buck"
- note added: "Input Protection"
- note added: "Main uC"
- note added: "TODO: Display: NHD-C12864A1Z-FSW-FBW-HTT FRAM: FM25V20A-DGQ 4-20ma Prot: MAX14626ETT+T High Side Switches: TPS27S100"
- note removed: "Display: NHD-C12864A1Z-FSW-FBW-HTT 3v3 Buck: LTC3851 24v Boost: LTC3786 FRAM: FM25V20A-DGQ 4-20ma Prot: MAX14626ETT+T High Side Switches: TPS1HC30-Q1"
- moved on the sheet: C1, C10, C11, C2, C3, C4, C5, C6, C7, C8, C9, D1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

Commit message: More WIP
Parts:
- added C34, C35, C36, C37, C38, C39, C40, C41, C42, C43, C44: 100nF 50V, symbol Device:C_Small
- added D10, D11, D12, D8, D9: D_Schottky, symbol Device:D_Schottky
- added F2: Polyfuse, symbol Device:Polyfuse
- added J2, J3, J4, J5, J6, J7: Screw_Terminal_01x02, symbol Connector:Screw_Terminal_01x02
- added R28, R31, R33, R35, R37: 15k, symbol Device:R_Small
- added R29, R30, R32, R34: 5k 1%, symbol Device:R_Small
- added R36: 825 1%, symbol Device:R_Small
- added R38: 100 1%, symbol Device:R_Small
- added U10: MAX14626, Custom Parts:TDFN-6, symbol Custom Parts:MAX14626
- added U11: LMV321, symbol Amplifier_Operational:LMV321
- added U5, U6, U7, U8, U9: TPS27S100A, Custom Parts:WQFN-16, symbol Custom Parts:TPS27S100A
Connections:
- net +12V: now also C42.2, D12.2 (A), F2.1
- net +3V3: now also C44.2, U11.5 (V+)
- net GND: now also C34.1, C35.1, C36.1, C37.1, C38.1, C39.1, C40.1, C41.1, C42.1, C43.1, C44.1, J2.2 (Pin_2), J3.2 (Pin_2), J4.2 (Pin_2), J5.2 (Pin_2), J6.2 (Pin_2), R29.1, R30.1, R32.1, R34.1, R36.1, R38.1, U10.2 (GND), U10.3 (GND), U10.4 (GND), U10.5 (GND), U10.7 (GND), U11.2 (V-), U11.3 (-), U11.4, U5.17 (GND), U5.2 (GND), U6.17 (GND), U6.2 (GND), U7.17 (GND), U7.2 (GND), U8.17 (GND), U8.2 (GND), U9.17 (GND), U9.2 (GND)
- new net: D10.1 (K), R33.1, U7.10 (IN), U7.11 (IN), U7.12 (IN), U7.9 (IN)
- new net: C41.2, J4.1 (Pin_1), R33.2, U7.5 (OUT), U7.6 (OUT), U7.7 (OUT), U7.8 (OUT)
- new net: R36.2, U9.15 (ILIM)
- new net: D8.1 (K), R28.1, U5.10 (IN), U5.11 (IN), U5.12 (IN), U5.9 (IN)
- new net: U5.13 (NC), U5.4 (NC), U5.NC (1)
- new net: R29.2, U5.15 (ILIM)
- new net: C35.2, J2.1 (Pin_1), R28.2, U5.5 (OUT), U5.6 (OUT), U5.7 (OUT), U5.8 (OUT)
- new net: F2.2, J7.1 (Pin_1)
- new net: D11.1 (K), R35.1, U8.10 (IN), U8.11 (IN), U8.12 (IN), U8.9 (IN)
- new net: U8.13 (NC), U8.4 (NC), U8.NC (1)
- new net: R34.2, U8.15 (ILIM)
- new net: C39.2, J5.1 (Pin_1), R35.2, U8.5 (OUT), U8.6 (OUT), U8.7 (OUT), U8.8 (OUT)
- new net: U7.13 (NC), U7.4 (NC), U7.NC (1)
- new net: R32.2, U7.15 (ILIM)
- new net: R38.2, U10.6 (OUT), U11.1 (+)
- new net: C37.2, J3.1 (Pin_1), R31.2, U6.5 (OUT), U6.6 (OUT), U6.7 (OUT), U6.8 (OUT)
- new net: D9.1 (K), R31.1, U6.10 (IN), U6.11 (IN), U6.12 (IN), U6.9 (IN)
- new net: C43.2, J6.1 (Pin_1), R37.2, U9.5 (OUT), U9.6 (OUT), U9.7 (OUT), U9.8 (OUT)
- new net: U6.13 (NC), U6.4 (NC), U6.NC (1)
- new net: R30.2, U6.15 (ILIM)
- new net: J7.2 (Pin_2), U10.1 (IN)
- new net: D12.1 (K), R37.1, U9.10 (IN), U9.11 (IN), U9.12 (IN), U9.9 (IN)
- new net: U9.13 (NC), U9.4 (NC), U9.NC (1)
- new net +24V: C34.2, C36.2, C38.2, C40.2, D10.2 (A), D11.2 (A), D8.2 (A), D9.2 (A)
- new net PUMP_DIAG: U9.14 (DIAG_EN)
- new net PUMP_EN: U9.3 (EN)
- new net PUMP_FLT: U9.16 (~{FLT})
- new net SOL_1_DIAG: U5.14 (DIAG_EN)
- new net SOL_1_EN: U5.3 (EN)
- new net SOL_1_FLT: U5.16 (~{FLT})
- new net SOL_2_DIAG: U6.14 (DIAG_EN)
- new net SOL_2_EN: U6.3 (EN)
- new net SOL_2_FLT: U6.16 (~{FLT})
- new net SOL_3_DIAG: U7.14 (DIAG_EN)
- new net SOL_3_EN: U7.3 (EN)
- new net SOL_3_FLT: U7.16 (~{FLT})
- new net SOL_4_DIAG: U8.14 (DIAG_EN)
- new net SOL_4_EN: U8.3 (EN)
- new net SOL_4_FLT: U8.16 (~{FLT})
Other:
- note added: "Motor Control"
- note added: "Pressure Transducer"
- note added: "Solenoid Control"
- note added: "TODO: Display: NHD-C12864A1Z-FSW-FBW-HTT FRAM: FM25V20A-DGQ 4-20ma Prot: MAX14626ETT+T"
- note removed: "TODO: Display: NHD-C12864A1Z-FSW-FBW-HTT FRAM: FM25V20A-DGQ 4-20ma Prot: MAX14626ETT+T High Side Switches: TPS27S100"

Commit message: More WIP
Parts:
- added C45, C50: 0.1uF 25V, symbol Device:C_Small
- added C46, C48, C49, C51: 1uF 25V, symbol Device:C_Small
- added C47, C52: 10uF 25V, symbol Device:C_Small
- added D13: GREEN, symbol Device:LED
- added Q5: PMV65XP,215, symbol Device:Q_PMOS_GSD
- added R39: 10, symbol Device:R_Small
- added R40: 10K, symbol Device:R_Small
- added R41: 0, symbol Device:R_Small
- added R42: 500, symbol Device:R
- added U12: NHD-C12864A1Z-FSW-FBW-HTT, Custom Parts:NHD-C12864A1Z-FSW-FBW-HTT, symbol Custom Parts:NHD-C12864A1Z-FSW-FBW-HTT
- added U13: ADP151, Custom Parts:CP_6_3_ADI, symbol Custom Parts:ADP151ACPZ-3.0-R7
- added U14: FM25V20A, Custom Parts:WDFN-8, symbol Custom Parts:FM25V20A
Connections:
- net +3V3: now also C48.1, C50.1, C51.1, C52.1, Q5.2 (S), R40.2, U13.6 (VIN), U14. (~{WP}), U14.8 (VDD)
- net GND: now also C45.2, C46.2, C47.2, C48.2, C49.2, C50.2, C51.2, C52.2, R42.2, U12.10 (LED_GND), U12.7 (VSS), U12.9 (HEATER_GND), U13.3 (GND), U13.7 (GND), U14.4 (VSS)
- new net: Q5.1 (G), R39.2, R40.1
- new net: Q5.3 (D), R41.2
- new net: D13.1 (K), R42.1
- new net: R41.1, U12.11 (LED_3V3)
- new net: U13.2 (NC), U13.5 (NC)
- new net +3V0: C45.1, C46.1, C47.1, C49.1, D13.2 (A), U12.3 (VDD), U13.1 (VOUT)
- new net DISPLAY_BL: R39.1
- new net DISPLAY_CS: U12.6 (~{CS})
- new net DISPLAY_EN: U13.4 (EN)
- new net DISPLAY_MOSI: U12.2 (SI)
- new net DISPLAY_REG: U12.4 (A0)
- new net DISPLAY_RESET: U12.5 (~{RESET})
- new net DISPLAY_SCL: U12.1 (SCL)
- new net FRAM_CS: U14.1 (~{CS})
- new net FRAM_MISO: U14.2 (SO)
- new net FRAM_MOSI: U14.5 (SI)
- new net FRAM_SCLK: U14.6 (SCLK)
Other:
- note added: "Display + Supply"
- note added: "FRAM"
- note added: "Pump Control"
- note removed: "Motor Control"
- note removed: "TODO: Display: NHD-C12864A1Z-FSW-FBW-HTT FRAM: FM25V20A-DGQ 4-20ma Prot: MAX14626ETT+T"

Commit message: Updates
Parts:
- removed C10, C11, C9: 4.7uF 50V, symbol Device:C_Small
- removed C23: 0.1uF 50V, symbol Device:C_Small
- removed C6: 5.5uF 25V, symbol Device:C_Small
- removed C7, C8: 1000uF 50V, symbol Device:C_Polarized
- removed D2: GREEN, symbol Device:LED
- removed D3: RED, symbol Device:LED
- removed R10: 6.6k 1%, symbol Device:R
- removed R11, R12: 11k, symbol Device:R
- removed R21: 53.6k 1%, symbol Device:R_Small
- removed R6, R7, R8: FIX, symbol Device:R
- removed R9: 5.5k 1%, symbol Device:R
- removed U2: TPS2660, symbol Custom:TPS2660
- added R21: 10k, symbol Device:R
- L1: value 0.68uH 15A -> SRP1265A-R68M; footprint (none) -> Custom Parts:SRP1265A
- L2: value 10.2uH 8A -> B82559B6682A016; footprint (none) -> Custom Parts:TDK-ERU-16
- R20: value 26.1k 1% -> 8m 1%
Connections:
- net DISPLAY_SCL is gone; now on net DISPLAY_SCLK: U12.1 (SCL)
- net FRAM_MOSI is gone; now on net DISPLAY_MOSI: U14.5 (SI)
- net FRAM_SCLK is gone; now on net DISPLAY_SCLK: U14.6 (SCLK)
- net SOL_1_FLT is gone; now on net PUMP_FLT: U5.16 (~{FLT})
- net SOL_2_FLT is gone; now on net PUMP_FLT: U6.16 (~{FLT})
- net SOL_3_FLT is gone; now on net PUMP_FLT: U7.16 (~{FLT})
- net SOL_4_FLT is gone; now on net PUMP_FLT: U8.16 (~{FLT})
- net +12V: no longer L2.1
- net +3.3V: now also R21.1
- net DISPLAY_BL: now also U1.32 (PA10)
- net DISPLAY_CS: now also U1.28 (PA8)
- net DISPLAY_MOSI: now also U1.18 (PA7)
- net DISPLAY_REG: now also U1.29 (PA9)
- net DISPLAY_RESET: now also U1.33 (PA11)
- net FRAM_CS: now also U1.34 (PA12)
- net FRAM_MISO: now also U1.17 (PA6)
- net GND: no longer U11.3 (-), U11.4
- net PUMP_DIAG: now also U1.24 (PB12)
- net PUMP_EN: now also U1.25 (PB13)
- net PUMP_FLT: now also U1.46 (PB7), R21.2
- net SOL_1_DIAG: now also U1.47 (PB8)
- net SOL_1_EN: now also U1.19 (PB0)
- net SOL_2_DIAG: now also U1.48 (PB9)
- net SOL_2_EN: now also U1.20 (PB1)
- net SOL_3_DIAG: now also U1.22 (PB10)
- net SOL_3_EN: now also U1.21 (PB2)
- net SOL_4_DIAG: now also U1.23 (PB11)
- net SOL_4_EN: now also U1.42 (PB3)
- net PRESSURE_BUFFERED: now reaches U1.11 (PA0)
- net PRESSURE_BUFFERED: now also U11.3 (-), U11.4
- net DISPLAY_SCLK: now reaches U1.16 (PA5)
- net at R20.2, U3.5 (SENSE-): now also L2.1
Other:
- note added: "USE TPS24751"

Commit message: New high current e-fuse
Parts:
- added C10, C9: 1000uF 50V, symbol Device:C_Polarized_Small
- added C11, C23, C53: 4.7uF 50V, symbol Device:C_Small
- added C6: 0.047uF 25V, symbol Device:C_Small
- added C7: 0.1uF 50V, symbol Device:C_Small
- added D2: GREEN, symbol Device:LED
- added D3: RED, symbol Device:LED
- added Q10: Q_PMOS_GSD, symbol Device:Q_PMOS_GSD
- added Q6: PSMN014-80YL, Package_TO_SOT_SMD:LFPAK56, symbol Custom Parts:PSMN014-80YL
- added Q7, Q8: Q_NMOS_GSD, symbol Device:Q_NMOS_GSD
- added R10, R43, R44: 10k 1%, symbol Device:R_Small
- added R11: 64.9k 1%, symbol Device:R_Small
- added R12: 1.58k 1%, symbol Device:R_Small
- added R45, R46: 2.61k, symbol Device:R
- added R47: 16k, symbol Device:R
- added R6: 2m 1% 1/2W, symbol Device:R_Small
- added R7: 51.1 1%, symbol Device:R_Small
- added R8: 104k 1%, symbol Device:R_Small
- added R9: 5.42k 1%, symbol Device:R_Small
- added U2: ~, Custom Parts:VQFN-36, symbol Custom Parts:TPS24751RUVR
Connections:
- net +12V: now also C10.1, C11.1, C23.1, C53.1, C9.1, D2.2 (A), Q10.2 (S), Q6.5 (D), R43.2, R44.2, R47.1
- net GND: now also C10.2, C11.2, C23.2, C53.2, C6.1, C7.2, C9.2, Q7.2 (S), Q8.2 (S), R10.1, R11.1, R12.1, R46.2, U2.28 (GND), U2.32 (GND), U2.36 (GND), U2.37 (GND), U2.4 (GND)
- net at F1.2: now also C7.1, R6.1, R7.1, R8.2, U2.26 (SENSE), U2.29 (VCC)
- net 3V3_ENABLE: now reaches U4.1 (RUN)
- net 3V3_ENABLE: now also Q7.3 (D)
- new net: R8.1, R9.2, U2.33 (EN)
- new net: R10.2, R9.1, U2.1 (OV)
- new net: Q7.1 (G), Q8.1 (G), R44.1, U2.31 (~{PG})
- new net: Q8.3 (D), R45.2
- new net: R7.2, U2.3 (SET)
- new net: Q10.1 (G), R43.1, R47.2, U2.30 (~{FLT})
- new net: D3.2 (A), Q10.3 (D)
- new net: D2.1 (K), R45.1
- new net: C6.2, U2.35 (TIMER)
- new net: Q6.1 (S), Q6.2 (S), Q6.3 (S), U2.10 (OUT), U2.11 (OUT), U2.12 (OUT), U2.13 (OUT), U2.19 (OUT), U2.20 (OUT), U2.21 (OUT), U2.22 (OUT), U2.23 (OUT), U2.24 (OUT), U2.6 (OUT), U2.7 (OUT), U2.8 (OUT), U2.9 (OUT)
- new net: Q6.4 (G), U2.25 (GATE)
- new net: D3.1 (K), R46.1
- new net: R12.2, U2.2 (IMON)
- new net: R6.2, U2.14 (DRAIN), U2.15 (DRAIN), U2.16 (DRAIN), U2.17 (DRAIN), U2.18 (DRAIN), U2.27 (DRAIN), U2.38 (DRAIN), U2.5 (DRAIN)
- new net: R11.2, U2.34 (PROG)
Other:
- note removed: "USE TPS24751"
- moved on the sheet: C45, C46, C47, C48, C49, C50, C51, C52, D13, Q5, R39, R40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

Commit message: Breakup design into smaller hierarchical sheets
Parts:
- removed C1, C2, C5: 0.1uF 10V, symbol Device:C_Small
- removed C10, C9: 1000uF 50V, symbol Device:C_Polarized_Small
- removed C11, C17, C23, C30, C53: 4.7uF 50V, symbol Device:C_Small
- removed C12, C13, C33, C45, C50: 0.1uF 25V, symbol Device:C_Small
- removed C14: 330pF 25V, symbol Device:C_Small
- removed C15: 2200pF 25V, symbol Device:C_Small
- removed C16, C29, C7: 0.1uF 50V, symbol Device:C_Small
- removed C18, C19: 330uF 10V, symbol Device:C_Polarized_US
- removed C20: 47pF 10V, symbol Device:C_Small
- removed C21, C6: 0.047uF 25V, symbol Device:C_Small
- removed C22: 22uF 25V, symbol Device:C_Polarized_US
- removed C24: 220uF 50V, symbol Device:C_Polarized_US
- removed C25, C26, C27, C28: 22uF 50V, symbol Device:C_Small
- removed C3: 1uF 10V, symbol Device:C_Small
- removed C31: 220pF 25V, symbol Device:C_Small
- removed C32: 15000pF 25V, symbol Device:C_Small
- removed C34, C35, C36, C37, C38, C39, C40, C41, C42, C43, C44: 100nF 50V, symbol Device:C_Small
- removed C4: 4.7uF 10V, symbol Device:C_Small
- removed C46, C48, C49, C51: 1uF 25V, symbol Device:C_Small
- removed C47, C52: 10uF 25V, symbol Device:C_Small
- removed D1: LED_RABG, symbol Device:LED_RABG
- removed D10, D11, D12, D4, D6, D8, D9: D_Schottky, symbol Device:D_Schottky
- removed D13, D2, D5, D7: GREEN, symbol Device:LED
- removed D3: RED, symbol Device:LED
- removed F1: Fuse, Custom:Keystone-3568, symbol Device:Fuse
- removed F2: Polyfuse, symbol Device:Polyfuse
- removed J1: TC2030-SWD, Custom:TC2030-IDC-FP, symbol Custom:TC2030-SWD
- removed J2, J3, J4, J5, J6, J7: Screw_Terminal_01x02, symbol Connector:Screw_Terminal_01x02
- removed L1: SRP1265A-R68M, Custom Parts:SRP1265A, symbol Device:L
- removed L2: B82559B6682A016, Custom Parts:TDK-ERU-16, symbol Device:L
- removed Q1, Q2, Q3, Q4, Q6: PSMN014-80YL, Package_TO_SOT_SMD:LFPAK56, symbol Custom Parts:PSMN014-80YL
- removed Q10: Q_PMOS_GSD, symbol Device:Q_PMOS_GSD
- removed Q5: PMV65XP,215, symbol Device:Q_PMOS_GSD
- removed Q7, Q8: Q_NMOS_GSD, symbol Device:Q_NMOS_GSD
- removed R1, R21, R25, R27: 10k, symbol Device:R
- removed R10, R43, R44: 10k 1%, symbol Device:R_Small
- removed R11: 64.9k 1%, symbol Device:R_Small
- removed R12: 1.58k 1%, symbol Device:R_Small
- removed R13: 82.5k, symbol Device:R
- removed R14: 15k, symbol Device:R
- removed R15: 154k 1%, symbol Device:R_Small
- removed R16: 48.7k 1%, symbol Device:R_Small
- removed R17: 3.01k, symbol Device:R_Small
- removed R18: 30.1k, symbol Device:R_Small
- removed R19, R3, R4, R42, R5: 500, symbol Device:R
- removed R2: NP, symbol Device:R
- removed R20: 8m 1%, symbol Device:R_Small
- removed R22: 232k 1%, symbol Device:R_Small
- removed R23: 12.1k 1%, symbol Device:R_Small
- removed R24: 8.87k 1%, symbol Device:R
- removed R26: 2.2k, symbol Device:R
- removed R28, R31, R33, R35, R37: 15k, symbol Device:R_Small
- removed R29, R30, R32, R34: 5k 1%, symbol Device:R_Small
- removed R36: 825 1%, symbol Device:R_Small
- removed R38: 100 1%, symbol Device:R_Small
- removed R39: 10, symbol Device:R_Small
- removed R40: 10K, symbol Device:R_Small
- removed R41: 0, symbol Device:R_Small
- removed R45, R46: 2.61k, symbol Device:R
- removed R47: 16k, symbol Device:R
- removed R6: 2m 1% 1/2W, symbol Device:R_Small
- removed R7: 51.1 1%, symbol Device:R_Small
- removed R8: 104k 1%, symbol Device:R_Small
- removed R9: 5.42k 1%, symbol Device:R_Small
- removed SW1: SW_Push, symbol Switch:SW_Push
- removed U1: STM32G0B1CEU6, Custom:UFQFPN-48, symbol Custom:STM32G0B1CEU6
- removed U10: MAX14626, Custom Parts:TDFN-6, symbol Custom Parts:MAX14626
- removed U11: LMV321, symbol Amplifier_Operational:LMV321
- removed U12: NHD-C12864A1Z-FSW-FBW-HTT, Custom Parts:NHD-C12864A1Z-FSW-FBW-HTT, symbol Custom Parts:NHD-C12864A1Z-FSW-FBW-HTT
- removed U13: ADP151, Custom Parts:CP_6_3_ADI, symbol Custom Parts:ADP151ACPZ-3.0-R7
- removed U14: FM25V20A, Custom Parts:WDFN-8, symbol Custom Parts:FM25V20A
- removed U2: ~, Custom Parts:VQFN-36, symbol Custom Parts:TPS24751RUVR
- removed U3: LTC3786, Custom:QFN-16, symbol Custom Parts:LTC3786
- removed U4: LTC3851, Custom Parts:QFN-16, symbol Custom Parts:LTC3851
- removed U5, U6, U7, U8, U9: TPS27S100A, Custom Parts:WQFN-16, symbol Custom Parts:TPS27S100A
Other:
- added sheet Display (display.kicad_sch)
- added sheet FRAM (fram.kicad_sch)
- added sheet Main uC (main_uc.kicad_sch)
- added sheet Output Control (output_control.kicad_sch)
- added sheet Power (power.kicad_sch)
- added sheet Pressure Transducer (4-20ma_frontend.kicad_sch)
- note removed: "12V to 24V Boost"
- note removed: "12V to 3.3V Buck"
- note removed: "Display + Supply"
- note removed: "FRAM"
- note removed: "Input Protection"
- note removed: "Main uC"
- note removed: "Pressure Transducer"
- note removed: "Pump Control"
- note removed: "Solenoid Control"
