File: bilge-vacuum/bilge-vacuum.kicad_sch (KiCad schematic)
At the start: 0 parts

Commit message: bilge vac 1v0
Parts:
- added H1, H2, H3, H4: MountingHole_Pad, MountingHole:MountingHole_3.5mm_Pad, symbol Mechanical:MountingHole_Pad
Connections:
- new net GND: H1.1, H2.1, H3.1, H4.1
Changed lines of the file:
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@@
 (kicad_sch (version 20230121) (generator eeschema)
   (paper "A4")
+  (junction (at 27.305 51.435) (diameter 0) (color 0 0 0 0)
+  )
   (junction (at 171.45 88.265) (diameter 0) (color 0 0 0 0)
   )
   (junction (at 167.64 92.075) (diameter 0) (color 0 0 0 0)
   )
+  (junction (at 27.305 41.275) (diameter 0) (color 0 0 0 0)
+  )
+  (junction (at 27.305 46.355) (diameter 0) (color 0 0 0 0)
+  )
   (wire (pts (xy 171.45 88.265) (xy 181.61 88.265))
     (stroke (width 0) (type default))
@@
     (stroke (width 0) (type default))
   )
+  (wire (pts (xy 27.305 51.435) (xy 27.305 55.245))
+    (stroke (width 0) (type default))
+  )
   (wire (pts (xy 169.545 128.27) (xy 169.545 90.17))
     (stroke (width 0) (type default))
   )
+  (wire (pts (xy 29.845 36.195) (xy 27.305 36.195))
+    (stroke (width 0) (type default))
+  )
   (wire (pts (xy 151.765 44.45) (xy 181.61 44.45))
     (stroke (width 0) (type default))
@@
     (stroke (width 0) (type default))
   )
+  (wire (pts (xy 27.305 41.275) (xy 29.845 41.275))
+    (stroke (width 0) (type default))
+  )
   (wire (pts (xy 151.765 81.28) (xy 181.61 81.28))
     (stroke (width 0) (type default))
@@
     (stroke (width 0) (type default))
   )
+  (wire (pts (xy 27.305 36.195) (xy 27.305 41.275))
+    (stroke (width 0) (type default))
+  )
   (wire (pts (xy 151.765 88.265) (xy 171.45 88.265))
     (stroke (width 0) (type default))
@@
     (stroke (width 0) (type default))
   )
+  (wire (pts (xy 27.305 46.355) (xy 27.305 51.435))
+    (stroke (width 0) (type default))
+  )
+  (wire (pts (xy 27.305 51.435) (xy 29.845 51.435))
+    (stroke (width 0) (type default))
+  )
   (wire (pts (xy 181.61 132.715) (xy 165.735 132.715))
     (stroke (width 0) (type default))
@@
     (stroke (width 0) (type default))
   )
+  (wire (pts (xy 27.305 46.355) (xy 29.845 46.355))
+    (stroke (width 0) (type default))
+  )
   (wire (pts (xy 151.765 36.83) (xy 181.61 36.83))
     (stroke (width 0) (type default))
@@
     (stroke (width 0) (type default))
   )
+  (wire (pts (xy 27.305 41.275) (xy 27.305 46.355))
+    (stroke (width 0) (type default))
+  )
   (wire (pts (xy 105.41 114.935) (xy 118.11 114.935))
     (stroke (width 0) (type default))
@@
     (stroke (width 0) (type default))
   )
+  (symbol (lib_id "Mechanical:MountingHole_Pad") (at 32.385 36.195 270) (unit 1)
+    (in_bom yes) (on_board yes) (dnp no) (fields_autoplaced)
+    (property "Reference" "H1" (at 36.195 34.9829 90)
+      (effects (font (size 1.27 1.27)) (justify left))
+    )
+    (property "Value" "MountingHole_Pad" (at 36.195 37.4071 90)
+      (effects (font (size 1.27 1.27)) (justify left))
+    )
+    (property "Footprint" "MountingHole:MountingHole_3.5mm_Pad" (at 32.385 36.195 0)
+      (effects (font (size 1.27 1.27)) hide)
+    )
+    (property "Datasheet" "~" (at 32.385 36.195 0)
+      (effects (font (size 1.27 1.27)) hide)
+    )
+    (pin "1")
+    (instances
+      (project "bilge-vacuum"
+        (path "/08405ba3-6912-4dc1-869a-b11176a5bc8a"
+          (reference "H1") (unit 1)
+        )
+      )
+    )
+  )
+  (symbol (lib_id "Mechanical:MountingHole_Pad") (at 32.385 46.355 270) (unit 1)
+    (in_bom yes) (on_board yes) (dnp no) (fields_autoplaced)
+    (property "Reference" "H3" (at 36.195 45.1429 90)
+      (effects (font (size 1.27 1.27)) (justify left))
+    )
+    (property "Value" "MountingHole_Pad" (at 36.195 47.5671 90)
+      (effects (font (size 1.27 1.27)) (justify left))
+    )
+    (property "Footprint" "MountingHole:MountingHole_3.5mm_Pad" (at 32.385 46.355 0)
+      (effects (font (size 1.27 1.27)) hide)
+    )
+    (property "Datasheet" "~" (at 32.385 46.355 0)
+      (effects (font (size 1.27 1.27)) hide)
+    )
+    (pin "1")
+    (instances
+      (project "bilge-vacuum"
+        (path "/08405ba3-6912-4dc1-869a-b11176a5bc8a"
+          (reference "H3") (unit 1)
+        )
+      )
+    )
+  )
+  (symbol (lib_id "power:GND") (at 27.305 55.245 0) (unit 1)
+    (in_bom yes) (on_board yes) (dnp no) (fields_autoplaced)
+    (property "Reference" "#PWR064" (at 27.305 61.595 0)
+      (effects (font (size 1.27 1.27)) hide)
+    )
+    (property "Value" "GND" (at 27.305 59.3781 0)
+      (effects (font (size 1.27 1.27)))
+    )
+    (property "Footprint" "" (at 27.305 55.245 0)
+      (effects (font (size 1.27 1.27)) hide)
+    )
+    (property "Datasheet" "" (at 27.305 55.245 0)
+      (effects (font (size 1.27 1.27)) hide)
+    )
+    (pin "1")
+    (instances
+      (project "bilge-vacuum"
+        (path "/08405ba3-6912-4dc1-869a-b11176a5bc8a"
+          (reference "#PWR064") (unit 1)
+        )
+      )
+    )
+  )
+  (symbol (lib_id "Mechanical:MountingHole_Pad") (at 32.385 51.435 270) (unit 1)
+    (in_bom yes) (on_board yes) (dnp no) (fields_autoplaced)
+    (property "Reference" "H4" (at 36.195 50.2229 90)
+      (effects (font (size 1.27 1.27)) (justify left))
+    )
+    (property "Value" "MountingHole_Pad" (at 36.195 52.6471 90)
+      (effects (font (size 1.27 1.27)) (justify left))
+    )
+    (property "Footprint" "MountingHole:MountingHole_3.5mm_Pad" (at 32.385 51.435 0)
+      (effects (font (size 1.27 1.27)) hide)
+    )
+    (property "Datasheet" "~" (at 32.385 51.435 0)
+      (effects (font (size 1.27 1.27)) hide)
+    )
+    (pin "1")
+    (instances
+      (project "bilge-vacuum"
+        (path "/08405ba3-6912-4dc1-869a-b11176a5bc8a"
+          (reference "H4") (unit 1)
+        )
+      )
+    )
+  )
+  (symbol (lib_id "Mechanical:MountingHole_Pad") (at 32.385 41.275 270) (unit 1)
+    (in_bom yes) (on_board yes) (dnp no) (fields_autoplaced)
+    (property "Reference" "H2" (at 36.195 40.0629 90)
+      (effects (font (size 1.27 1.27)) (justify left))
+    )
+    (property "Value" "MountingHole_Pad" (at 36.195 42.4871 90)
+      (effects (font (size 1.27 1.27)) (justify left))
+    )
+    (property "Footprint" "MountingHole:MountingHole_3.5mm_Pad" (at 32.385 41.275 0)
+      (effects (font (size 1.27 1.27)) hide)
+    )
+    (property "Datasheet" "~" (at 32.385 41.275 0)
+      (effects (font (size 1.27 1.27)) hide)
+    )
+    (pin "1")
+    (instances
+      (project "bilge-vacuum"
+        (path "/08405ba3-6912-4dc1-869a-b11176a5bc8a"
+          (reference "H2") (unit 1)
+        )
+      )
+    )
+  )
   (sheet (at 181.61 76.2) (size 29.21 30.48) (fields_autoplaced)
