File: bilge-vacuum/bilge-vacuum.kicad_sch (KiCad schematic)
At the start: 4 parts

Commit message: Fixes
Other:
- sheet Main uC ports: added DISPLAY_3V0_ENABLE; removed none
- sheet Power ports: added DISP_3V0_ENABLE; removed none
Changed lines of the file:
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@@
+    (stroke (width 0) (type default))
+  )
+  (wire (pts (xy 105.41 117.475) (xy 118.11 117.475))
     (stroke (width 0) (type default))
   )
@@
       (effects (font (size 1.27 1.27)) (justify right))
     )
+    (pin "DISPLAY_3V0_ENABLE" input (at 118.11 117.475 180)
+      (effects (font (size 1.27 1.27)) (justify left))
+    )
     (instances
       (project "bilge-vacuum"
@@
       (effects (font (size 1.27 1.27)) (justify right))
     )
+    (pin "DISP_3V0_ENABLE" input (at 105.41 117.475 0)
+      (effects (font (size 1.27 1.27)) (justify right))
+    )
