File: bilge-vacuum/24v_boost.kicad_sch (KiCad schematic)
At the start: 21 parts, among them Q3 PSMN014-80YL, Q4 PSMN014-80YL, U3 LTC3786

Commit message: Assign the bulk of parts, some passives still need custom footprints.
Parts:
- C25, C26, C27, C28: value 22uF 50V -> 10uF 50V; footprint (none) -> Capacitor_SMD:C_1206_3216Metric
- C29, C30, C31, C32: footprint (none) -> Capacitor_SMD:C_0805_2012Metric
- C33: value 0.1uF 25V -> 0.1uF 50V; footprint (none) -> Capacitor_SMD:C_0805_2012Metric
- D6: footprint (none) -> Custom Parts:SMA
- R20: footprint (none) -> Resistor_SMD:R_1206_3216Metric
- R22, R23, R24, R25, R27: footprint (none) -> Resistor_SMD:R_0805_2012Metric
Changed lines of the file:
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@@
       (effects (font (size 1.27 1.27)) (justify left))
     )
-    (property "Value" "22uF 50V" (at 240.4491 89.4834 0)
-      (effects (font (size 1.27 1.27)) (justify left))
-    )
-    (property "Footprint" "" (at 238.125 88.265 0)
+    (property "Value" "10uF 50V" (at 240.4491 89.4834 0)
+      (effects (font (size 1.27 1.27)) (justify left))
+    )
+    (property "Footprint" "Capacitor_SMD:C_1206_3216Metric" (at 238.125 88.265 0)
       (effects (font (size 1.27 1.27)) hide)
     )
@@
       (effects (font (size 1.27 1.27)) (justify right))
     )
-    (property "Footprint" "" (at 97.663 80.645 90)
+    (property "Footprint" "Resistor_SMD:R_0805_2012Metric" (at 97.663 80.645 90)
       (effects (font (size 1.27 1.27)) hide)
     )
@@
       (effects (font (size 1.27 1.27)) (justify right))
     )
-    (property "Footprint" "" (at 61.595 81.915 0)
+    (property "Footprint" "Capacitor_SMD:C_0805_2012Metric" (at 61.595 81.915 0)
       (effects (font (size 1.27 1.27)) hide)
     )
@@
       (effects (font (size 1.27 1.27)) (justify right))
     )
-    (property "Footprint" "" (at 149.86 72.39 0)
+    (property "Footprint" "Capacitor_SMD:C_0805_2012Metric" (at 149.86 72.39 0)
       (effects (font (size 1.27 1.27)) hide)
     )
@@
       (effects (font (size 1.27 1.27)) (justify right))
     )
-    (property "Footprint" "" (at 47.625 75.565 0)
+    (property "Footprint" "Capacitor_SMD:C_0805_2012Metric" (at 47.625 75.565 0)
       (effects (font (size 1.27 1.27)) hide)
     )
@@
       (effects (font (size 1.27 1.27)))
     )
-    (property "Footprint" "" (at 156.845 66.04 0)
+    (property "Footprint" "Capacitor_SMD:C_0805_2012Metric" (at 156.845 66.04 0)
       (effects (font (size 1.27 1.27)) hide)
     )
@@
       (effects (font (size 1.27 1.27)) (justify left))
     )
-    (property "Footprint" "" (at 211.455 78.105 0)
+    (property "Footprint" "Resistor_SMD:R_0805_2012Metric" (at 211.455 78.105 0)
       (effects (font (size 1.27 1.27)) hide)
     )
@@
       (effects (font (size 1.27 1.27)) (justify left))
     )
-    (property "Value" "22uF 50V" (at 247.4341 80.5934 0)
-      (effects (font (size 1.27 1.27)) (justify left))
-    )
-    (property "Footprint" "" (at 245.11 79.375 0)
+    (property "Value" "10uF 50V" (at 247.4341 80.5934 0)
+      (effects (font (size 1.27 1.27)) (justify left))
+    )
+    (property "Footprint" "Capacitor_SMD:C_1206_3216Metric" (at 245.11 79.375 0)
       (effects (font (size 1.27 1.27)) hide)
     )
@@
       (effects (font (size 1.27 1.27)) (justify right))
     )
-    (property "Footprint" "" (at 211.455 86.995 0)
+    (property "Footprint" "Resistor_SMD:R_0805_2012Metric" (at 211.455 86.995 0)
       (effects (font (size 1.27 1.27)) hide)
     )
@@
       (effects (font (size 1.27 1.27)) (justify left))
     )
-    (property "Value" "22uF 50V" (at 226.4791 89.4834 0)
-      (effects (font (size 1.27 1.27)) (justify left))
-    )
-    (property "Footprint" "" (at 224.155 88.265 0)
+    (property "Value" "10uF 50V" (at 226.4791 89.4834 0)
+      (effects (font (size 1.27 1.27)) (justify left))
+    )
+    (property "Footprint" "Capacitor_SMD:C_1206_3216Metric" (at 224.155 88.265 0)
       (effects (font (size 1.27 1.27)) hide)
     )
@@
       (effects (font (size 1.27 1.27)) (justify right))
     )
-    (property "Value" "0.1uF 25V" (at 80.4291 78.0407 0)
-      (effects (font (size 1.27 1.27)) (justify right))
-    )
-    (property "Footprint" "" (at 78.105 76.835 0)
+    (property "Value" "0.1uF 50V" (at 80.4291 78.0407 0)
+      (effects (font (size 1.27 1.27)) (justify right))
+    )
+    (property "Footprint" "Capacitor_SMD:C_0805_2012Metric" (at 78.105 76.835 0)
       (effects (font (size 1.27 1.27)) hide)
     )
@@
       (effects (font (size 1.27 1.27)))
     )
-    (property "Footprint" "" (at 142.24 68.58 0)
+    (property "Footprint" "Custom Parts:SMA" (at 142.24 68.58 0)
       (effects (font (size 1.27 1.27)) hide)
     )
@@
       (effects (font (size 1.27 1.27)) (justify left))
     )
-    (property "Footprint" "" (at 182.88 45.72 0)
+    (property "Footprint" "Resistor_SMD:R_1206_3216Metric" (at 182.88 45.72 0)
       (effects (font (size 1.27 1.27)) hide)
     )
@@
       (effects (font (size 1.27 1.27)) (justify right))
     )
-    (property "Footprint" "" (at 36.703 71.12 90)
+    (property "Footprint" "Resistor_SMD:R_0805_2012Metric" (at 36.703 71.12 90)
       (effects (font (size 1.27 1.27)) hide)
     )
@@
       (effects (font (size 1.27 1.27)) (justify left))
     )
-    (property "Value" "22uF 50V" (at 233.4641 80.5934 0)
-      (effects (font (size 1.27 1.27)) (justify left))
-    )
-    (property "Footprint" "" (at 231.14 79.375 0)
+    (property "Value" "10uF 50V" (at 233.4641 80.5934 0)
+      (effects (font (size 1.27 1.27)) (justify left))
+    )
+    (property "Footprint" "Capacitor_SMD:C_1206_3216Metric" (at 231.14 79.375 0)
       (effects (font (size 1.27 1.27)) hide)
     )
@@
       (effects (font (size 1.27 1.27)) (justify right))
     )
-    (property "Footprint" "" (at 63.373 73.025 90)
-      (effects (font (size 1.27 1.27)) hide)
-    )
+    (property "Footprint" "Resistor_SMD:R_0805_2012Metric" (at 63.373 73.025 90)
+      (effects (font (size 1.27 1.27)) hide)
+    )

Commit message: Vac progress
Parts:
- C24: value 220uF 50V -> EEEFT1H221GV; footprint (none) -> Custom Parts:Panasonic - F - Vibe
- U3: footprint Custom:QFN-16 -> Custom Parts:QFN-16
Changed lines of the file:
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@@
       (effects (font (size 1.27 1.27)))
     )
-    (property "Footprint" "Custom:QFN-16" (at 122.555 43.18 0)
+    (property "Footprint" "Custom Parts:QFN-16" (at 122.555 43.18 0)
       (effects (font (size 1.27 1.27)) hide)
     )
@@
       (effects (font (size 1.27 1.27)) (justify left))
     )
-    (property "Value" "220uF 50V" (at 255.016 87.5721 0)
-      (effects (font (size 1.27 1.27)) (justify left))
-    )
-    (property "Footprint" "" (at 252.095 86.995 0)
-      (effects (font (size 1.27 1.27)) hide)
-    )
+    (property "Value" "EEEFT1H221GV" (at 255.016 87.5721 0)
+      (effects (font (size 1.27 1.27)) (justify left))
+    )
+    (property "Footprint" "Custom Parts:Panasonic - F - Vibe" (at 252.095 86.995 0)
+      (effects (font (size 1.27 1.27)) hide)
+    )

Commit message: bilge vac 1v0
Connections:
- net BOOST_BG: now reaches Q3.4 (G), U3.12 (BG)
- net BOOST_TG: now reaches Q4.4 (G), U3.16 (TG)
Changed lines of the file:
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@@
     (effects (font (size 5 5) bold) (justify left bottom))
+  )
+  (label "BOOST_TG" (at 139.065 58.42 0) (fields_autoplaced)
+    (effects (font (size 1.27 1.27)) (justify left bottom))
   )
   (label "24V_INTVCC" (at 106.68 60.96 180) (fields_autoplaced)
@@
     (effects (font (size 1.27 1.27) bold) (justify left bottom))
   )
+  (label "BOOST_BG" (at 138.43 72.39 0) (fields_autoplaced)
+    (effects (font (size 1.27 1.27)) (justify left bottom))
+  )
   (hierarchical_label "PGOOD" (shape input) (at 103.505 90.17 0) (fields_autoplaced)

Commit message: Fixes
Parts:
- R25, R27: value 10k -> 10k 1%
Changed lines of the file:
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@@
       (effects (font (size 1.27 1.27)) (justify right))
     )
-    (property "Value" "10k" (at 97.663 81.8571 0)
+    (property "Value" "10k 1%" (at 97.663 81.8571 0)
       (effects (font (size 1.27 1.27)) (justify right))
     )
@@
       (effects (font (size 1.27 1.27)) (justify right))
     )
-    (property "Value" "10k" (at 36.703 72.3321 0)
-      (effects (font (size 1.27 1.27)) (justify right))
-    )
+    (property "Value" "10k 1%" (at 36.703 72.3321 0)
+      (effects (font (size 1.27 1.27)) (justify right))
+    )

Commit message: Fixes
Parts:
- D6: value D_Schottky -> B260AQ-13-F
Connections:
- net 24V_INTVCC: now also D6.2 (A), U3.13 (INTVcc); no longer C29.1, D6.1 (K), U3.15 (BOOST)
- new net: C29.1, D6.1 (K), U3.15 (BOOST)
Other:
- moved on the sheet: C29, C30, D6
