File: bilge-vacuum/output_control.kicad_sch (KiCad schematic)
At the start: 10 parts, among them J10 Screw_Terminal_01x02, J11 Screw_Terminal_01x02, J6 Screw_Terminal_01x02, J8 Screw_Terminal_01x02, J9 Screw_Terminal_01x02

Commit message: Assign the bulk of parts, some passives still need custom footprints.
Parts:
- R36, R49, R50, R52, R54: footprint (none) -> Resistor_SMD:R_0805_2012Metric
Changed lines of the file:
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@@
       (effects (font (size 1.27 1.27)))
     )
-    (property "Footprint" "" (at 234.315 63.5 0)
+    (property "Footprint" "Resistor_SMD:R_0805_2012Metric" (at 234.315 63.5 0)
       (effects (font (size 1.27 1.27)) hide)
     )
@@
       (effects (font (size 1.27 1.27)))
     )
-    (property "Footprint" "" (at 125.73 116.84 0)
+    (property "Footprint" "Resistor_SMD:R_0805_2012Metric" (at 125.73 116.84 0)
       (effects (font (size 1.27 1.27)) hide)
     )
@@
       (effects (font (size 1.27 1.27)))
     )
-    (property "Footprint" "" (at 125.73 73.025 0)
+    (property "Footprint" "Resistor_SMD:R_0805_2012Metric" (at 125.73 73.025 0)
       (effects (font (size 1.27 1.27)) hide)
     )
@@
       (effects (font (size 1.27 1.27)))
     )
-    (property "Footprint" "" (at 36.83 116.84 0)
+    (property "Footprint" "Resistor_SMD:R_0805_2012Metric" (at 36.83 116.84 0)
       (effects (font (size 1.27 1.27)) hide)
     )
@@
       (effects (font (size 1.27 1.27)))
     )
-    (property "Footprint" "" (at 36.83 71.755 0)
-      (effects (font (size 1.27 1.27)) hide)
-    )
+    (property "Footprint" "Resistor_SMD:R_0805_2012Metric" (at 36.83 71.755 0)
+      (effects (font (size 1.27 1.27)) hide)
+    )

Commit message: Vac progress
Parts:
- J10, J11, J6, J8, J9: footprint (none) -> Custom Parts:2604-1102
Changed lines of the file:
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@@
       (effects (font (size 1.27 1.27)) (justify left))
     )
-    (property "Footprint" "" (at 175.26 99.695 0)
+    (property "Footprint" "Custom Parts:2604-1102" (at 175.26 99.695 0)
       (effects (font (size 1.27 1.27)) hide)
     )
@@
       (effects (font (size 1.27 1.27)) (justify left))
     )
-    (property "Footprint" "" (at 86.36 99.695 0)
+    (property "Footprint" "Custom Parts:2604-1102" (at 86.36 99.695 0)
       (effects (font (size 1.27 1.27)) hide)
     )
@@
       (effects (font (size 1.27 1.27)) (justify left))
     )
-    (property "Footprint" "" (at 86.36 54.61 0)
+    (property "Footprint" "Custom Parts:2604-1102" (at 86.36 54.61 0)
       (effects (font (size 1.27 1.27)) hide)
     )
@@
       (effects (font (size 1.27 1.27)) (justify left))
     )
-    (property "Footprint" "" (at 285.115 46.355 0)
+    (property "Footprint" "Custom Parts:2604-1102" (at 285.115 46.355 0)
       (effects (font (size 1.27 1.27)) hide)
     )
@@
       (effects (font (size 1.27 1.27)) (justify left))
     )
-    (property "Footprint" "" (at 175.26 55.88 0)
-      (effects (font (size 1.27 1.27)) hide)
-    )
+    (property "Footprint" "Custom Parts:2604-1102" (at 175.26 55.88 0)
+      (effects (font (size 1.27 1.27)) hide)
+    )

Commit message: bilge vac 1v0
Changed lines of the file:
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@@
     (effects (font (size 1.27 1.27)) (justify left bottom))
   )
-  (label "PUMP_ENABLE" (at 238.76 51.435 180) (fields_autoplaced)
+  (label "PUMP_EN" (at 238.76 51.435 180) (fields_autoplaced)
     (effects (font (size 1.27 1.27)) (justify right bottom))
   )

Commit message: Fixes
Parts:
- R36: value 5k 1% -> 1.2k 1%
Changed lines of the file:
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@@
       (effects (font (size 1.27 1.27)))
     )
-    (property "Value" "5k 1%" (at 234.315 61.0433 90)
+    (property "Value" "1.2k 1%" (at 234.315 61.0433 90)
       (effects (font (size 1.27 1.27)))
     )

Commit message: Fixes
Other:
- sheet Pump Switch ports: added IO_VDD; removed none
- sheet Solenoid 1 ports: added IO_VDD; removed none
- sheet Solenoid 2 ports: added IO_VDD; removed none
- sheet Solenoid 3 ports: added IO_VDD; removed none
- sheet Solenoid 4 ports: added IO_VDD; removed none
Changed lines of the file:
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@@
+    (stroke (width 0) (type default))
+  )
+  (wire (pts (xy 228.6 42.545) (xy 228.6 48.895))
     (stroke (width 0) (type default))
   )
@@
     (stroke (width 0) (type default))
   )
+  (wire (pts (xy 114.935 92.71) (xy 114.935 102.235))
+    (stroke (width 0) (type default))
+  )
   (wire (pts (xy 39.37 71.755) (xy 43.815 71.755))
     (stroke (width 0) (type default))
@@
     (stroke (width 0) (type default))
   )
+  (wire (pts (xy 26.67 57.15) (xy 43.815 57.15))
+    (stroke (width 0) (type default))
+  )
   (wire (pts (xy 67.945 168.91) (xy 67.945 170.815))
     (stroke (width 0) (type default))
@@
     (stroke (width 0) (type default))
   )
+  (wire (pts (xy 26.67 47.625) (xy 26.67 57.15))
+    (stroke (width 0) (type default))
+  )
+  (wire (pts (xy 228.6 48.895) (xy 242.57 48.895))
+    (stroke (width 0) (type default))
+  )
   (wire (pts (xy 39.37 173.355) (xy 42.545 173.355))
     (stroke (width 0) (type default))
@@
     (stroke (width 0) (type default))
   )
+  (wire (pts (xy 114.935 48.895) (xy 114.935 58.42))
+    (stroke (width 0) (type default))
+  )
+  (wire (pts (xy 26.67 102.235) (xy 43.815 102.235))
+    (stroke (width 0) (type default))
+  )
+  (wire (pts (xy 26.67 92.71) (xy 26.67 102.235))
+    (stroke (width 0) (type default))
+  )
   (wire (pts (xy 30.48 116.84) (xy 34.29 116.84))
     (stroke (width 0) (type default))
@@
     (stroke (width 0) (type default))
   )
+  (wire (pts (xy 114.935 58.42) (xy 132.715 58.42))
+    (stroke (width 0) (type default))
+  )
   (wire (pts (xy 39.37 179.07) (xy 42.545 179.07))
     (stroke (width 0) (type default))
@@
   )
   (wire (pts (xy 66.04 165.1) (xy 67.945 165.1))
+    (stroke (width 0) (type default))
+  )
+  (wire (pts (xy 114.935 102.235) (xy 132.715 102.235))
     (stroke (width 0) (type default))
   )
@@
     )
   )
+  (symbol (lib_id "power:+3V3") (at 26.67 92.71 0) (unit 1)
+    (in_bom yes) (on_board yes) (dnp no) (fields_autoplaced)
+    (property "Reference" "#PWR023" (at 26.67 96.52 0)
+      (effects (font (size 1.27 1.27)) hide)
+    )
+    (property "Value" "+3V3" (at 26.67 88.5769 0)
+      (effects (font (size 1.27 1.27)))
+    )
+    (property "Footprint" "" (at 26.67 92.71 0)
+      (effects (font (size 1.27 1.27)) hide)
+    )
+    (property "Datasheet" "" (at 26.67 92.71 0)
+      (effects (font (size 1.27 1.27)) hide)
+    )
+    (pin "1")
+    (instances
+      (project "bilge-vacuum"
+        (path "/08405ba3-6912-4dc1-869a-b11176a5bc8a"
+          (reference "#PWR023") (unit 1)
+        )
+        (path "/08405ba3-6912-4dc1-869a-b11176a5bc8a/8a95e837-e0e7-4b78-93e7-7ab95e7c82dc"
+          (reference "#PWR026") (unit 1)
+        )
+        (path "/08405ba3-6912-4dc1-869a-b11176a5bc8a/16850e27-1e2e-4e85-af36-1238f6162217"
+          (reference "#PWR066") (unit 1)
+        )
+      )
+    )
+  )
+  (symbol (lib_id "power:+3V3") (at 114.935 48.895 0) (unit 1)
+    (in_bom yes) (on_board yes) (dnp no) (fields_autoplaced)
+    (property "Reference" "#PWR023" (at 114.935 52.705 0)
+      (effects (font (size 1.27 1.27)) hide)
+    )
+    (property "Value" "+3V3" (at 114.935 44.7619 0)
+      (effects (font (size 1.27 1.27)))
+    )
+    (property "Footprint" "" (at 114.935 48.895 0)
+      (effects (font (size 1.27 1.27)) hide)
+    )
+    (property "Datasheet" "" (at 114.935 48.895 0)
+      (effects (font (size 1.27 1.27)) hide)
+    )
+    (pin "1")
+    (instances
+      (project "bilge-vacuum"
+        (path "/08405ba3-6912-4dc1-869a-b11176a5bc8a"
+          (reference "#PWR023") (unit 1)
+        )
+        (path "/08405ba3-6912-4dc1-869a-b11176a5bc8a/8a95e837-e0e7-4b78-93e7-7ab95e7c82dc"
+          (reference "#PWR026") (unit 1)
+        )
+        (path "/08405ba3-6912-4dc1-869a-b11176a5bc8a/16850e27-1e2e-4e85-af36-1238f6162217"
+          (reference "#PWR068") (unit 1)
+        )
+      )
+    )
+  )
   (symbol (lib_id "power:GND") (at 278.13 50.8 0) (unit 1)
     (in_bom yes) (on_board yes) (dnp no) (fields_autoplaced)
@@
     )
   )
+  (symbol (lib_id "power:+3V3") (at 114.935 92.71 0) (unit 1)
+    (in_bom yes) (on_board yes) (dnp no) (fields_autoplaced)
+    (property "Reference" "#PWR023" (at 114.935 96.52 0)
+      (effects (font (size 1.27 1.27)) hide)
+    )
+    (property "Value" "+3V3" (at 114.935 88.5769 0)
+      (effects (font (size 1.27 1.27)))
+    )
+    (property "Footprint" "" (at 114.935 92.71 0)
+      (effects (font (size 1.27 1.27)) hide)
+    )
+    (property "Datasheet" "" (at 114.935 92.71 0)
+      (effects (font (size 1.27 1.27)) hide)
+    )
+    (pin "1")
+    (instances
+      (project "bilge-vacuum"
+        (path "/08405ba3-6912-4dc1-869a-b11176a5bc8a"
+          (reference "#PWR023") (unit 1)
+        )
+        (path "/08405ba3-6912-4dc1-869a-b11176a5bc8a/8a95e837-e0e7-4b78-93e7-7ab95e7c82dc"
+          (reference "#PWR026") (unit 1)
+        )
+        (path "/08405ba3-6912-4dc1-869a-b11176a5bc8a/16850e27-1e2e-4e85-af36-1238f6162217"
+          (reference "#PWR067") (unit 1)
+        )
+      )
+    )
+  )
   (symbol (lib_id "power:+24V") (at 121.92 48.895 0) (unit 1)
     (in_bom yes) (on_board yes) (dnp no) (fields_autoplaced)
@@
     )
   )
+  (symbol (lib_id "power:+3V3") (at 26.67 47.625 0) (unit 1)
+    (in_bom yes) (on_board yes) (dnp no) (fields_autoplaced)
+    (property "Reference" "#PWR023" (at 26.67 51.435 0)
+      (effects (font (size 1.27 1.27)) hide)
+    )
+    (property "Value" "+3V3" (at 26.67 43.4919 0)
+      (effects (font (size 1.27 1.27)))
+    )
+    (property "Footprint" "" (at 26.67 47.625 0)
+      (effects (font (size 1.27 1.27)) hide)
+    )
+    (property "Datasheet" "" (at 26.67 47.625 0)
+      (effects (font (size 1.27 1.27)) hide)
+    )
+    (pin "1")
+    (instances
+      (project "bilge-vacuum"
+        (path "/08405ba3-6912-4dc1-869a-b11176a5bc8a"
+          (reference "#PWR023") (unit 1)
+        )
+        (path "/08405ba3-6912-4dc1-869a-b11176a5bc8a/8a95e837-e0e7-4b78-93e7-7ab95e7c82dc"
+          (reference "#PWR026") (unit 1)
+        )
+        (path "/08405ba3-6912-4dc1-869a-b11176a5bc8a/16850e27-1e2e-4e85-af36-1238f6162217"
+          (reference "#PWR065") (unit 1)
+        )
+      )
+    )
+  )
   (symbol (lib_id "power:GND") (at 168.275 104.775 0) (unit 1)
     (in_bom yes) (on_board yes) (dnp no) (fields_autoplaced)
@@
         (path "/08405ba3-6912-4dc1-869a-b11176a5bc8a/16850e27-1e2e-4e85-af36-1238f6162217"
           (reference "R43") (unit 1)
+        )
+      )
+    )
+  )
+  (symbol (lib_id "power:+3V3") (at 228.6 42.545 0) (unit 1)
+    (in_bom yes) (on_board yes) (dnp no) (fields_autoplaced)
+    (property "Reference" "#PWR023" (at 228.6 46.355 0)
+      (effects (font (size 1.27 1.27)) hide)
+    )
+    (property "Value" "+3V3" (at 228.6 38.4119 0)
+      (effects (font (size 1.27 1.27)))
+    )
+    (property "Footprint" "" (at 228.6 42.545 0)
+      (effects (font (size 1.27 1.27)) hide)
+    )
+    (property "Datasheet" "" (at 228.6 42.545 0)
+      (effects (font (size 1.27 1.27)) hide)
+    )
+    (pin "1")
+    (instances
+      (project "bilge-vacuum"
+        (path "/08405ba3-6912-4dc1-869a-b11176a5bc8a"
+          (reference "#PWR023") (unit 1)
+        )
+        (path "/08405ba3-6912-4dc1-869a-b11176a5bc8a/8a95e837-e0e7-4b78-93e7-7ab95e7c82dc"
+          (reference "#PWR026") (unit 1)
+        )
+        (path "/08405ba3-6912-4dc1-869a-b11176a5bc8a/16850e27-1e2e-4e85-af36-1238f6162217"
+          (reference "#PWR069") (unit 1)
         )
       )
@@
       (effects (font (size 1.27 1.27)) (justify left))
     )
+    (pin "IO_VDD" input (at 132.715 102.235 180)
+      (effects (font (size 1.27 1.27)) (justify left))
+    )
     (instances
       (project "bilge-vacuum"
@@
       (effects (font (size 1.27 1.27)) (justify left))
     )
+    (pin "IO_VDD" input (at 242.57 48.895 180)
+      (effects (font (size 1.27 1.27)) (justify left))
+    )
     (instances
       (project "bilge-vacuum"
@@
       (effects (font (size 1.27 1.27)) (justify left))
     )
+    (pin "IO_VDD" input (at 132.715 58.42 180)
+      (effects (font (size 1.27 1.27)) (justify left))
+    )
     (instances
       (project "bilge-vacuum"
@@
       (effects (font (size 1.27 1.27)) (justify left))
     )
+    (pin "IO_VDD" input (at 43.815 57.15 180)
+      (effects (font (size 1.27 1.27)) (justify left))
+    )
     (instances
       (project "bilge-vacuum"
@@
       (effects (font (size 1.27 1.27)) (justify left))
     )
+    (pin "IO_VDD" input (at 43.815 102.235 180)
+      (effects (font (size 1.27 1.27)) (justify left))
+    )
