File: bilge-vacuum/bilge-vacuum.kicad_pcb (KiCad board)
At the start: 2 copper layers, 159 parts, among them J1 TC2030-SWD, J3 Screw_Terminal_01x02, J4 Screw_Terminal_01x02, J5 Screw_Terminal_01x02, J6 Screw_Terminal_01x02, J7 Screw_Terminal_01x02, J8 Screw_Terminal_01x02, Q1 PSMN014-80YL, Q10 Q_NMOS_GSD, Q2 PSMN014-80YL, Q3 PSMN014-80YL, Q4 PSMN014-80YL, Q5 PMV65XP,215, Q6 PSMN014-80YL, Q7 Q_NMOS_GSD, Q8 Q_NMOS_GSD, Q9 Q_PMOS_GSD, SW1 B3F-1000, U1 STM32G0B1CEU6, U10 TPS27S100A, U11 TPS27S100A, U12 NHD-C12864A1Z-FSW-FBW-HTT, U13 ADP151, U14 FM25V20A, U2 LTC3851, U3 LTC3786, U4 MAX14626, U6 LMV321, U7 TPS27S100A, U8 TPS27S100A, U9 TPS27S100A

Commit message: WIP
Parts:
- added J2: Screw_Terminal_01x02, Custom Parts:2604-1102, F.Cu at (134.1, 176.8)
- moved U14 211.1 mm to (260.0, 51.3)
- moved F1 174.1 mm to (95.4, 185.6)
- moved J8 172.7 mm to (276.5, 103.5)
- moved F3 163.1 mm to (275.8, 91.4)
- moved J7 158.9 mm to (250.0, 103.8)
- moved BZ1 158.3 mm to (276.7, 42.6)
- moved J6 156.7 mm to (234.3, 104.0)
- moved J5 155.7 mm to (219.8, 104.1)
- moved J4 154.4 mm to (205.0, 103.7)
- moved J3 152.5 mm to (189.5, 104.2)
- moved S1 152.2 mm to (272.8, 20.6)
- moved Q10 135.6 mm to (280.4, 54.2)
- moved D1 124.5 mm to (259.0, 28.3)
- moved D12 123.8 mm to (205.4, 91.1)
- moved U11 123.8 mm to (203.9, 86.2)
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Connections:
- F1 pad 1: +BATT -> /Power/Input Protection/VIN

Commit message: bilge vac 1v0
Parts:
- added C53: 0.1uF 50V, Capacitor_SMD:C_0805_2012Metric, F.Cu at (149.2, 66.2)
- added D15: GREEN, LED_SMD:LED_0805_2012Metric, F.Cu at (154.9, 145.1)
- added D16: GREEN, LED_SMD:LED_0805_2012Metric, F.Cu at (154.8, 119.4)
- added D17: GREEN, LED_SMD:LED_0805_2012Metric, F.Cu at (155.2, 106.1)
- added D18: GREEN, LED_SMD:LED_0805_2012Metric, F.Cu at (155.2, 131.7)
- added H1: MountingHole_Pad, MountingHole:MountingHole_3.5mm_Pad, F.Cu at (30.0, 30.0)
- added H2: MountingHole_Pad, MountingHole:MountingHole_3.5mm_Pad, F.Cu at (30.0, 155.0)
- added H3: MountingHole_Pad, MountingHole:MountingHole_3.5mm_Pad, F.Cu at (185.0, 30.0)
- added H4: MountingHole_Pad, MountingHole:MountingHole_3.5mm_Pad, F.Cu at (185.0, 155.0)
- added R21: NP, Resistor_SMD:R_0805_2012Metric, F.Cu at (170.6, 34.6)
- added R57: 0, Resistor_SMD:R_0805_2012Metric, F.Cu at (148.4, 69.1)
- added R58: 2.2k, Resistor_SMD:R_0805_2012Metric, F.Cu at (154.9, 141.5)
- added R59: 2.2k, Resistor_SMD:R_0805_2012Metric, F.Cu at (154.8, 115.8)
- added R60: 2.2k, Resistor_SMD:R_0805_2012Metric, F.Cu at (155.2, 102.5)
- added R61: 2.2k, Resistor_SMD:R_0805_2012Metric, F.Cu at (155.2, 128.1)
- R48: value 499 -> 2.2k
- U5: value ~ -> TPS24751RUVR
- moved S1 194.5 mm to (97.5, 104.8)
- moved Q4 190.8 mm to (31.2, 63.6)
- moved Q6 182.0 mm to (38.7, 63.6)
- moved C35 174.4 mm to (34.3, 46.1), turned to -90 degrees
- moved L2 156.1 mm to (37.2, 78.6), turned to 180 degrees
- moved U3 149.2 mm to (51.2, 54.5)
- moved D6 146.1 mm to (56.0, 49.9), turned to -90 degrees
- moved C50 125.2 mm to (159.7, 60.1), turned to -90 degrees
- moved D7 124.2 mm to (42.8, 46.8), turned to -90 degrees
- moved F3 124.2 mm to (152.8, 74.1)
- moved C52 121.5 mm to (164.1, 59.5), turned to -90 degrees
- moved R27 119.3 mm to (42.8, 43.1), turned to 90 degrees
- moved C51 117.9 mm to (162.0, 59.5), turned to -90 degrees
- moved R47 116.4 mm to (144.6, 89.1), turned to 180 degrees
- moved R43 116.4 mm to (144.7, 140.9)
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Connections:
- net Net-(Q2-G) renamed /Power/3.3V Buck/BUCK_TG
- net Net-(Q3-G) renamed /Power/3.3V Buck/BUCK_BG
- net Net-(Q4-G) renamed /Power/24V Boost/BOOST_BG
- net Net-(Q6-G) renamed /Power/24V Boost/BOOST_TG
- C1 pad 1: +3.3V -> +3V3
- C12 pad 2: +3.3V -> +3V3
- C3 pad 1: +3.3V -> +3V3
- C4 pad 1: +3.3V -> +3V3
- C5 pad 1: +3.3V -> +3V3
- D1 pad 2: +3.3V -> +3V3
- D14 pad 2: +3V3 -> /Output Control/Pump Switch/OUT
- J1 pad 1: +3.3V -> +3V3
- R23 pad 2: +3.3V -> +3V3
- R4 pad 1: +3.3V -> +3V3
- R49 pad 1: +3.3V -> +3V3
- R5 pad 1: +3.3V -> +3V3
- R50 pad 1: +3.3V -> +3V3
- R51 pad 1: +3.3V -> +3V3
- R52 pad 1: +3.3V -> +3V3
- R53 pad 1: +3.3V -> +3V3
- R54 pad 1: +3.3V -> +3V3
- S1 pad 1: (no net) -> GND
- U1 pad 4: +3.3V -> +3V3
- U1 pad 5: +3.3V -> +3V3
- U1 pad 6: +3.3V -> +3V3
- U10 pad 1: (no net) -> unconnected-(U10-NC-Pad1)
- U10 pad 13: Net-(U10-1) -> unconnected-(U10-NC-Pad13)
- U10 pad 4: Net-(U10-1) -> unconnected-(U10-NC-Pad4)
- U11 pad 1: (no net) -> unconnected-(U11-NC-Pad1)
- U11 pad 13: Net-(U11-1) -> unconnected-(U11-NC-Pad13)
- U11 pad 4: Net-(U11-1) -> unconnected-(U11-NC-Pad4)
- U13 pad 2: Net-(U13-NC-Pad2) -> unconnected-(U13-NC-Pad2)
- U13 pad 5: Net-(U13-NC-Pad2) -> unconnected-(U13-NC-Pad5)
- U14 pad 3: (no net) -> +3V3
- U6 pad 1: Net-(U4-OUT) -> Net-(U6-+)
- U6 pad 5: +3.3V -> +3V3
- U7 pad 1: (no net) -> unconnected-(U7-NC-Pad1)
- U7 pad 13: Net-(U7-1) -> unconnected-(U7-NC-Pad13)
- U7 pad 3: /Output Control/PUMP_ENABLE -> /Output Control/PUMP_EN
- U7 pad 4: Net-(U7-1) -> unconnected-(U7-NC-Pad4)
- U8 pad 1: (no net) -> unconnected-(U8-NC-Pad1)
- U8 pad 13: Net-(U8-1) -> unconnected-(U8-NC-Pad13)
- U8 pad 4: Net-(U8-1) -> unconnected-(U8-NC-Pad4)
- U9 pad 1: (no net) -> unconnected-(U9-NC-Pad1)
- U9 pad 13: Net-(U9-1) -> unconnected-(U9-NC-Pad13)
- U9 pad 4: Net-(U9-1) -> unconnected-(U9-NC-Pad4)
Routing:
- net +12V: track 0.00 -> 680.0 mm, vias 0 -> 4
- net +24V: track 0.00 -> 262.0 mm, vias 0 -> 2
- net /Main uC/24V_ENABLE: track 0.00 -> 156.9 mm, vias 0 -> 2
- net /Main uC/24V_PGOOD: track 0.00 -> 143.3 mm, vias 0 -> 2
- net /Output Control/PUMP_FLT: track 0.00 -> 134.2 mm, vias 0 -> 7
- net /Output Control/SOL_1_EN: track 0.00 -> 133.2 mm, vias 0 -> 2
- net /Display/REG: track 0.00 -> 128.9 mm, vias 0 -> 3
- net /Display/SCLK: track 0.00 -> 128.3 mm, vias 0 -> 2
- net /Display/MOSI: track 0.00 -> 127.2 mm, vias 0 -> 2
- net /Display/RESET: track 0.00 -> 125.4 mm, vias 0 -> 3
- net /Main uC/NAV_C: track 0.00 -> 122.4 mm, vias 0 -> 4
- net /Main uC/NAV_SEL: track 0.00 -> 121.2 mm, vias 0 -> 4
- net /Output Control/SOL_1_DIAG: track 0.00 -> 121.1 mm, vias 0 -> 2
- net /Display/CS: track 0.00 -> 118.2 mm, vias 0 -> 3
- net /Output Control/SOL_2_EN: track 0.00 -> 118.0 mm, vias 0 -> 2
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- added copper zone on F.Cu, net +12V
- added copper zone on F.Cu, net +24V
- added copper zone on F.Cu, net +3V0
- added copper zone on F.Cu, net +3V3
- added copper zone on In2.Cu, net +3V3
- added copper zone on F.Cu, net /Output Control/Pump Switch/OUT
- added copper zone on F.Cu, net /Output Control/Solenoid 1/OUT
- added copper zone on F.Cu, net /Output Control/Solenoid 2/OUT
- added copper zone on F.Cu, net /Output Control/Solenoid 3/OUT
- added copper zone on F.Cu, net /Output Control/Solenoid 4/OUT
- added copper zone on B.Cu, net GND
- added copper zone on F.Cu, net GND
- added copper zone on In1.Cu, net GND
- added copper zone on F.Cu, net Net-(D10-K)
- added copper zone on F.Cu, net Net-(D11-K)
- added copper zone on F.Cu, net Net-(D12-K)
- added copper zone on F.Cu, net Net-(D8-K)
- added copper zone on F.Cu, net Net-(D9-K)
- added copper zone on F.Cu, net Net-(Q1-S-Pad1)
- added copper zone on F.Cu, net Net-(Q3-D)
- added copper zone on F.Cu, net Net-(Q4-D)
- added copper zone on F.Cu, net Net-(R18-Pad2)
- added copper zone on F.Cu, net Net-(U3-SENSE-)
- added copper zone on F.Cu, net Net-(U5-SENSE)
Other:
- board outline added: 163 x 133 mm
- copper layers 2 -> 4
- board text added: "+"
- board text added: "-"
- board text added: "12V IN"
- board text added: "Bilge Vac 1v0"
- board text added: "Drain"
- board text added: "Nav"
- board text added: "Press."
- board text added: "Pump"
- board text added: "Push To Select"
- board text added: "Zone 1"
- board text added: "Zone 2"
- board text added: "Zone 3"

Commit message: Fixes
Parts:
- C47, C50: value 10uF 25V -> 10uF 50V
- R20, R23, R4, R41, R49, R5, R50, R51, R52, R53: value 10k -> 10k 1%
- R47: value 5k 1% -> 1.2k 1%
Changed lines of the file:
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@@
         (effects (font (size 1 1) (thickness 0.15)))
     )
-    (fp_text value "10uF 25V" (at -0.095 2.305 90) (layer "F.Fab")
+    (fp_text value "10uF 50V" (at -0.095 2.305 90) (layer "F.Fab")
         (effects (font (size 1 1) (thickness 0.15)))
     )
@@
         (effects (font (size 1 1) (thickness 0.15)))
     )
-    (fp_text value "10k" (at 0 1.65) (layer "F.Fab")
+    (fp_text value "10k 1%" (at 0 1.65) (layer "F.Fab")
         (effects (font (size 1 1) (thickness 0.15)))
     )
@@
         (effects (font (size 1 1) (thickness 0.15)))
     )
-    (fp_text value "10k" (at 0 1.65) (layer "F.Fab")
+    (fp_text value "10k 1%" (at 0 1.65) (layer "F.Fab")
         (effects (font (size 1 1) (thickness 0.15)))
     )
@@
         (effects (font (size 1 1) (thickness 0.15)))
     )
-    (fp_text value "10k" (at 0 1.65) (layer "F.Fab")
+    (fp_text value "10k 1%" (at 0 1.65) (layer "F.Fab")
         (effects (font (size 1 1) (thickness 0.15)))
     )
@@
         (effects (font (size 1 1) (thickness 0.15)))
     )
-    (fp_text value "10k" (at 0 1.65) (layer "F.Fab")
+    (fp_text value "10k 1%" (at 0 1.65) (layer "F.Fab")
         (effects (font (size 1 1) (thickness 0.15)))
     )
@@
         (effects (font (size 1 1) (thickness 0.15)))
     )
-    (fp_text value "10k" (at 0 1.65) (layer "F.Fab")
+    (fp_text value "10k 1%" (at 0 1.65) (layer "F.Fab")
         (effects (font (size 1 1) (thickness 0.15)))
     )
@@
         (effects (font (size 1 1) (thickness 0.15)))
     )
-    (fp_text value "5k 1%" (at 0 1.65) (layer "F.Fab")
+    (fp_text value "1.2k 1%" (at 0 1.65) (layer "F.Fab")
         (effects (font (size 1 1) (thickness 0.15)))
     )
@@
         (effects (font (size 1 1) (thickness 0.15)))
     )
-    (fp_text value "10k" (at 0 1.65 90) (layer "F.Fab")
+    (fp_text value "10k 1%" (at 0 1.65 90) (layer "F.Fab")
         (effects (font (size 1 1) (thickness 0.15)))
     )
@@
         (effects (font (size 1 1) (thickness 0.15)))
     )
-    (fp_text value "10k" (at 0 1.65 90) (layer "F.Fab")
+    (fp_text value "10k 1%" (at 0 1.65 90) (layer "F.Fab")
         (effects (font (size 1 1) (thickness 0.15)))
     )
@@
         (effects (font (size 1 1) (thickness 0.15)))
     )
-    (fp_text value "10uF 25V" (at 0 1.85 90) (layer "F.Fab")
+    (fp_text value "10uF 50V" (at 0 1.85 90) (layer "F.Fab")
         (effects (font (size 1 1) (thickness 0.15)))
     )
@@
         (effects (font (size 1 1) (thickness 0.15)))
     )
-    (fp_text value "10k" (at 0 1.65) (layer "F.Fab")
+    (fp_text value "10k 1%" (at 0 1.65) (layer "F.Fab")
         (effects (font (size 1 1) (thickness 0.15)))
     )
@@
         (effects (font (size 1 1) (thickness 0.15)))
     )
-    (fp_text value "10k" (at 0 1.65) (layer "F.Fab")
+    (fp_text value "10k 1%" (at 0 1.65) (layer "F.Fab")
         (effects (font (size 1 1) (thickness 0.15)))
     )
@@
         (effects (font (size 1 1) (thickness 0.15)))
     )
-    (fp_text value "10k" (at 0 1.65) (layer "F.Fab")
+    (fp_text value "10k 1%" (at 0 1.65) (layer "F.Fab")
         (effects (font (size 1 1) (thickness 0.15)))
     )

Commit message: Fixes
Parts:
- removed R32: 16k, Resistor_SMD:R_0805_2012Metric
- added C54: 10uF 50V, Capacitor_SMD:C_1206_3216Metric, F.Cu at (233.0, 41.4)
- added C55: 10uF 50V, Capacitor_SMD:C_1206_3216Metric, F.Cu at (233.0, 44.8)
- added D19: 5.0SMDJ18CA, Custom Parts:DO-214AB, F.Cu at (216.2, 32.6)
- added D20: B260AQ-13-F, Custom Parts:SMA, F.Cu at (214.8, 38.5)
- added R62: 10k 1%, Resistor_SMD:R_0805_2012Metric, F.Cu at (219.2, 44.0)
- added R63: 10k 1%, Resistor_SMD:R_0805_2012Metric, F.Cu at (232.4, 30.4)
- added R64: 10k 1%, Resistor_SMD:R_0805_2012Metric, F.Cu at (226.0, 30.4)
- added R65: 10k 1%, Resistor_SMD:R_0805_2012Metric, F.Cu at (212.8, 44.0)
- added R66: 10k 1%, Resistor_SMD:R_0805_2012Metric, F.Cu at (226.0, 41.2)
- added R67: 10k 1%, Resistor_SMD:R_0805_2012Metric, F.Cu at (219.2, 46.9)
- added R68: 10k 1%, Resistor_SMD:R_0805_2012Metric, F.Cu at (232.4, 33.3)
- added R69: 10k 1%, Resistor_SMD:R_0805_2012Metric, F.Cu at (226.0, 33.3)
- added R70: 10k 1%, Resistor_SMD:R_0805_2012Metric, F.Cu at (212.8, 46.9)
- added R71: 10k 1%, Resistor_SMD:R_0805_2012Metric, F.Cu at (226.0, 44.1)
- added R72: 10k 1%, Resistor_SMD:R_0805_2012Metric, F.Cu at (219.2, 49.9)
- added R73: 10k 1%, Resistor_SMD:R_0805_2012Metric, F.Cu at (232.4, 36.2)
- added R74: 10k 1%, Resistor_SMD:R_0805_2012Metric, F.Cu at (226.0, 36.2)
- added R75: 10k 1%, Resistor_SMD:R_0805_2012Metric, F.Cu at (212.8, 49.9)
- added R76: 10k 1%, Resistor_SMD:R_0805_2012Metric, F.Cu at (226.0, 47.1)
- D10, D11, D12, D4, D6, D8, D9: value D_Schottky -> B260AQ-13-F
- F3: footprint Resistor_SMD:R_2010_5025Metric -> Custom Parts:SMD_2016
- Q8: value Q_NMOS_GSD -> Q_PMOS_GSD
- R27, R48, R58, R59, R60, R61: value 2.2k -> 10k 1%
- R31, R33: value 2.61k -> 5k 1%
- moved Q8 156.3 mm to (232.7, 50.6), turned to 0 degrees
Connections:
- C30 pad 1: /Power/24V Boost/24V_INTVCC -> Net-(D6-K)
- D2 pad 2: +12V -> Net-(D2-A)
- D6 pad 1: /Power/24V Boost/24V_INTVCC -> Net-(D6-K)
- D6 pad 2: Net-(D6-A) -> /Power/24V Boost/24V_INTVCC
- Q8 pad 2: GND -> +12V
- Q8 pad 3: Net-(Q8-D) -> Net-(D2-A)
- R31 pad 2: Net-(Q8-D) -> GND
- U1 pad 31: unconnected-(U1-PC7-Pad31) -> /Main uC/DISPLAY_3V0_ENABLE
- U13 pad 4: /Power/DISPLAY_EN -> /Main uC/DISPLAY_3V0_ENABLE
- U3 pad 13: Net-(D6-A) -> /Power/24V Boost/24V_INTVCC
- U3 pad 15: /Power/24V Boost/24V_INTVCC -> Net-(D6-K)
Routing:
- net /Power/24V Boost/24V_INTVCC: track 19.2 -> 23.8 mm
- net Net-(D6-A): track 4.53 -> 0.00 mm
- net Net-(Q8-D): track 2.05 -> 0.00 mm
- net GND: track 0.00 -> 2.05 mm

Commit message: Updates
Parts:
- removed R28: 1.58k 1%, Resistor_SMD:R_0805_2012Metric
- added C56: 0.1uF 50V, Capacitor_SMD:C_0805_2012Metric, F.Cu at (213.3, 68.8)
- added Q11: PSMN014-80YL, Package_TO_SOT_SMD:LFPAK56, F.Cu at (215.2, 61.0)
- C14: value 0.047uF 25V -> 0.1uF 50V
- R14: value 104k 1% -> 21.5k 1%
- R15: value 5.42k 1% -> 1.1k 1%
- R16: value 10k 1% -> 2k 1%
- R17: value 51.1 1% -> 3m 1% 1/2W; footprint Resistor_SMD:R_0805_2012Metric -> Resistor_SMD:R_1206_3216Metric
- R18: value 2m 1% 1/2W -> 15k; footprint Resistor_SMD:R_1206_3216Metric -> Resistor_SMD:R_0805_2012Metric
- R19: value 64.9k 1% -> 2k
- U5: value TPS24751RUVR -> LTC4229; footprint Custom Parts:VQFN-36 -> Custom Parts:WFQFN-24
- moved U5 136.8 mm to (222.8, 60.5)
- moved R19 134.6 mm to (217.8, 68.7)
- moved C14 133.3 mm to (213.3, 65.8), turned to 0 degrees
- moved R17 132.3 mm to (222.8, 65.9), turned to 0 degrees
- moved R18 122.9 mm to (217.8, 65.8), turned to 0 degrees
Connections:
- C13 pad 1: Net-(D19-A2) -> /Power/Input Protection/VIN
- C14 pad 1: GND -> Net-(U5-FTMR)
- C14 pad 2: Net-(U5-TIMER) -> GND
- F1 pad 2: Net-(D19-A2) -> /Power/Input Protection/VIN
- Q1 pad 1: Net-(Q1-S-Pad1) -> +12V
- Q1 pad 2: Net-(Q1-S-Pad1) -> +12V
- Q1 pad 3: Net-(Q1-S-Pad1) -> +12V
- Q1 pad 4: Net-(Q1-G) -> /Power/Input Protection/HOTSWAP_GATE
- Q1 pad 5: +12V -> /Power/Input Protection/SENSE_N
- R14 pad 1: Net-(U5-EN) -> /Power/Input Protection/UNDERVOLT_SENSE
- R14 pad 2: Net-(D19-A2) -> /Power/Input Protection/VIN
- R15 pad 1: Net-(U5-OV) -> /Power/Input Protection/OVERVOLT_SENSE
- R15 pad 2: Net-(U5-EN) -> /Power/Input Protection/UNDERVOLT_SENSE
- R16 pad 2: Net-(U5-OV) -> /Power/Input Protection/OVERVOLT_SENSE
- R17 pad 1: Net-(D19-A2) -> /Power/Input Protection/SENSE_N
- R17 pad 2: Net-(U5-SET) -> /Power/Input Protection/SENSE_N
- R18 pad 1: Net-(D19-A2) -> +12V
- R18 pad 2: Net-(R18-Pad2) -> /Power/Input Protection/FOLDBACK_SENSE
- R19 pad 1: GND -> /Power/Input Protection/FOLDBACK_SENSE
- R19 pad 2: Net-(U5-PROG) -> GND
- U5 pad 1: Net-(U5-OV) -> /Power/Input Protection/VIN
- U5 pad 10: Net-(Q1-S-Pad1) -> Net-(U5-FTMR)
- U5 pad 11: Net-(Q1-S-Pad1) -> GND
- U5 pad 12: Net-(Q1-S-Pad1) -> /Power/Input Protection/UNDERVOLT_SENSE
- U5 pad 13: Net-(Q1-S-Pad1) -> /Power/Input Protection/OVERVOLT_SENSE
- U5 pad 14: Net-(R18-Pad2) -> GND
- U5 pad 15: Net-(R18-Pad2) -> GND
- U5 pad 16: Net-(R18-Pad2) -> unconnected-(U5-~{DFLT}-Pad16)
- U5 pad 17: Net-(R18-Pad2) -> unconnected-(U5-~{DSTAT}-Pad17)
- U5 pad 18: Net-(R18-Pad2) -> /Power/Input Protection/~{FAULT}
- U5 pad 19: Net-(Q1-S-Pad1) -> /Power/Input Protection/~{PGOOD}
- U5 pad 2: Net-(U5-IMON) -> /Power/Input Protection/SENSE_N
- U5 pad 20: Net-(Q1-S-Pad1) -> /Power/Input Protection/FOLDBACK_SENSE
- U5 pad 21: Net-(Q1-S-Pad1) -> +12V
- U5 pad 22: Net-(Q1-S-Pad1) -> /Power/Input Protection/HOTSWAP_GATE
- U5 pad 23: Net-(Q1-S-Pad1) -> unconnected-(U5-CPO-Pad23)
- U5 pad 24: Net-(Q1-S-Pad1) -> /Power/Input Protection/DIODE_GATE
- U5 pad 25: Net-(Q1-G) -> GND
- U5 pad 3: Net-(U5-SET) -> /Power/Input Protection/SENSE_N
- U5 pad 4: GND -> /Power/Input Protection/VIN
- U5 pad 5: Net-(R18-Pad2) -> /Power/Input Protection/SENSE_N
- U5 pad 6: Net-(Q1-S-Pad1) -> Net-(U5-DTMR)
- U5 pad 7: Net-(Q1-S-Pad1) -> GND
- U5 pad 8: Net-(Q1-S-Pad1) -> Net-(U5-DTMR)
- U5 pad 9: Net-(Q1-S-Pad1) -> unconnected-(U5-RTMR-Pad9)
Routing:
- net (no net): track 0.00 -> 20.6 mm, vias 0 -> 2
- net Net-(U5-OV): track 19.1 -> 0.00 mm, vias 2 -> 0
- net /Power/Input Protection/OVERVOLT_SENSE: track 0.00 -> 19.1 mm, vias 0 -> 2
- net /Power/Input Protection/VIN: track 17.1 -> 33.9 mm, vias 0 -> 2
- net Net-(D19-A2): track 16.7 -> 0.00 mm, vias 2 -> 0
- net Net-(U5-EN): track 13.5 -> 0.00 mm, vias 2 -> 0
- net /Power/Input Protection/UNDERVOLT_SENSE: track 0.00 -> 13.5 mm, vias 0 -> 2
- net Net-(U5-SET): track 8.96 -> 0.00 mm, vias 2 -> 0
- net Net-(Q1-G): track 7.29 -> 0.00 mm, vias 2 -> 0
- net /Power/Input Protection/HOTSWAP_GATE: track 0.00 -> 7.29 mm, vias 0 -> 2
- net Net-(U5-PROG): track 4.69 -> 0.00 mm
- net Net-(U5-TIMER): track 4.39 -> 0.00 mm
- net Net-(U5-IMON): track 2.56 -> 0.00 mm
- added copper zone on F.Cu, net (none)
- added copper zone on F.Cu, net /Power/Input Protection/VIN
- removed copper zone on F.Cu, net Net-(D19-A2)
- removed copper zone on F.Cu, net Net-(Q1-S-Pad1)
- removed copper zone on F.Cu, net Net-(R18-Pad2)
