File: bilge-vacuum/e-fuse.kicad_sch (KiCad schematic)
At the start: 19 parts, among them Q6 PSMN014-80YL

Commit message: Assign the bulk of parts, some passives still need custom footprints.
Parts:
- C11, C23, C53, C6, C7: footprint (none) -> Capacitor_SMD:C_0805_2012Metric
- R10, R11, R12, R43, R44, R7, R8, R9: footprint (none) -> Resistor_SMD:R_0805_2012Metric
- R6: footprint (none) -> Resistor_SMD:R_1206_3216Metric
Changed lines of the file:
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@@
       (effects (font (size 1.27 1.27)) (justify left))
     )
-    (property "Footprint" "" (at 209.55 70.485 0)
+    (property "Footprint" "Capacitor_SMD:C_0805_2012Metric" (at 209.55 70.485 0)
       (effects (font (size 1.27 1.27)) hide)
     )
@@
       (effects (font (size 1.27 1.27)) (justify left))
     )
-    (property "Footprint" "" (at 204.47 64.77 0)
+    (property "Footprint" "Capacitor_SMD:C_0805_2012Metric" (at 204.47 64.77 0)
       (effects (font (size 1.27 1.27)) hide)
     )
@@
       (effects (font (size 1.27 1.27)) (justify right))
     )
-    (property "Footprint" "" (at 158.75 50.165 0)
+    (property "Footprint" "Resistor_SMD:R_0805_2012Metric" (at 158.75 50.165 0)
       (effects (font (size 1.27 1.27)) hide)
     )
@@
       (effects (font (size 1.27 1.27)) (justify right))
     )
-    (property "Footprint" "" (at 59.69 69.215 0)
+    (property "Footprint" "Resistor_SMD:R_0805_2012Metric" (at 59.69 69.215 0)
       (effects (font (size 1.27 1.27)) hide)
     )
@@
       (effects (font (size 1.27 1.27)) (justify right))
     )
-    (property "Footprint" "" (at 59.69 50.165 0)
+    (property "Footprint" "Resistor_SMD:R_0805_2012Metric" (at 59.69 50.165 0)
       (effects (font (size 1.27 1.27)) hide)
     )
@@
       (effects (font (size 1.27 1.27)) (justify right))
     )
-    (property "Footprint" "" (at 59.69 59.69 0)
+    (property "Footprint" "Resistor_SMD:R_0805_2012Metric" (at 59.69 59.69 0)
       (effects (font (size 1.27 1.27)) hide)
     )
@@
       (effects (font (size 1.27 1.27)))
     )
-    (property "Footprint" "" (at 89.535 64.77 0)
+    (property "Footprint" "Resistor_SMD:R_0805_2012Metric" (at 89.535 64.77 0)
       (effects (font (size 1.27 1.27)) hide)
     )
@@
       (effects (font (size 1.27 1.27)) (justify right))
     )
-    (property "Footprint" "" (at 147.955 50.165 0)
+    (property "Footprint" "Resistor_SMD:R_0805_2012Metric" (at 147.955 50.165 0)
       (effects (font (size 1.27 1.27)) hide)
     )
@@
       (effects (font (size 1.27 1.27)))
     )
-    (property "Footprint" "" (at 89.535 43.18 0)
+    (property "Footprint" "Resistor_SMD:R_1206_3216Metric" (at 89.535 43.18 0)
       (effects (font (size 1.27 1.27)) hide)
     )
@@
       (effects (font (size 1.27 1.27)))
     )
-    (property "Footprint" "" (at 80.01 52.07 0)
+    (property "Footprint" "Resistor_SMD:R_0805_2012Metric" (at 80.01 52.07 0)
       (effects (font (size 1.27 1.27)) hide)
     )
@@
       (effects (font (size 1.27 1.27)) (justify right))
     )
-    (property "Footprint" "" (at 121.285 66.675 0)
+    (property "Footprint" "Resistor_SMD:R_0805_2012Metric" (at 121.285 66.675 0)
       (effects (font (size 1.27 1.27)) hide)
     )
@@
       (effects (font (size 1.27 1.27)) (justify left))
     )
-    (property "Footprint" "" (at 200.025 58.42 0)
+    (property "Footprint" "Capacitor_SMD:C_0805_2012Metric" (at 200.025 58.42 0)
       (effects (font (size 1.27 1.27)) hide)
     )
@@
       (effects (font (size 1.27 1.27)) (justify left))
     )
-    (property "Footprint" "" (at 45.085 59.69 0)
+    (property "Footprint" "Capacitor_SMD:C_0805_2012Metric" (at 45.085 59.69 0)
       (effects (font (size 1.27 1.27)) hide)
     )
@@
       (effects (font (size 1.27 1.27)))
     )
-    (property "Footprint" "" (at 81.28 68.58 0)
-      (effects (font (size 1.27 1.27)) hide)
-    )
+    (property "Footprint" "Capacitor_SMD:C_0805_2012Metric" (at 81.28 68.58 0)
+      (effects (font (size 1.27 1.27)) hide)
+    )

Commit message: Vac progress
Parts:
- C10, C9: value 1000uF 50V -> EEE-FK1H102AV; footprint (none) -> Custom Parts:Panasonic - J - Vibe
- F1: footprint Custom:Keystone-3568 -> Custom Parts:Keystone-3568
Changed lines of the file:
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@@
       (effects (font (size 1.27 1.27)) (justify left))
     )
-    (property "Value" "1000uF 50V" (at 187.579 70.516 0)
-      (effects (font (size 1.27 1.27)) (justify left))
-    )
-    (property "Footprint" "" (at 185.42 69.85 0)
+    (property "Value" "EEE-FK1H102AV" (at 187.579 70.516 0)
+      (effects (font (size 1.27 1.27)) (justify left))
+    )
+    (property "Footprint" "Custom Parts:Panasonic - J - Vibe" (at 185.42 69.85 0)
       (effects (font (size 1.27 1.27)) hide)
     )
@@
       (effects (font (size 1.27 1.27)))
     )
-    (property "Footprint" "Custom:Keystone-3568" (at 38.1 44.958 90)
+    (property "Footprint" "Custom Parts:Keystone-3568" (at 38.1 44.958 90)
       (effects (font (size 1.27 1.27)) hide)
     )
@@
       (effects (font (size 1.27 1.27)) (justify left))
     )
-    (property "Value" "1000uF 50V" (at 181.864 60.356 0)
-      (effects (font (size 1.27 1.27)) (justify left))
-    )
-    (property "Footprint" "" (at 179.705 59.69 0)
-      (effects (font (size 1.27 1.27)) hide)
-    )
+    (property "Value" "EEE-FK1H102AV" (at 181.864 60.356 0)
+      (effects (font (size 1.27 1.27)) (justify left))
+    )
+    (property "Footprint" "Custom Parts:Panasonic - J - Vibe" (at 179.705 59.69 0)
+      (effects (font (size 1.27 1.27)) hide)
+    )

Commit message: bilge vac 1v0
Parts:
- U2: value ~ -> TPS24751RUVR
Changed lines of the file:
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@@
   )
   (symbol (lib_id "Custom Parts:TPS24751RUVR") (at 106.68 55.88 0) (unit 1)
-    (in_bom yes) (on_board yes) (dnp no) (fields_autoplaced)
-    (property "Reference" "U2" (at 106.68 40.3169 0)
+    (in_bom yes) (on_board yes) (dnp no)
+    (property "Reference" "U2" (at 114.3 40.64 0)
       (effects (font (size 1.27 1.27)))
     )
-    (property "Value" "~" (at 99.06 40.64 0)
+    (property "Value" "TPS24751RUVR" (at 104.775 40.64 0)
       (effects (font (size 1.27 1.27)))
     )

Commit message: Fixes
Parts:
- added D19: 5.0SMDJ18CA, Custom Parts:DO-214AB, symbol Device:D_TVS
- added D6: B260AQ-13-F, Custom Parts:SMA, symbol Device:D_Schottky
Connections:
- net GND: now also D19.1 (A1), D6.2 (A)
- net VOUT: now also D6.1 (K)
- net at C7.1, F1.2, R6.1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: now also D19.2 (A2)
Other:
- moved on the sheet: C10, C11, C23, C53, C6, C7, C9, F1, Q6, R10, R11, R12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

Commit message: Updates
Parts:
- removed C6: 0.047uF 25V, Capacitor_SMD:C_0805_2012Metric, symbol Device:C_Small
- removed R11: 64.9k 1%, Resistor_SMD:R_0805_2012Metric, symbol Device:R_Small
- removed R12: 1.58k 1%, Resistor_SMD:R_0805_2012Metric, symbol Device:R_Small
- removed R6: 2m 1% 1/2W, Resistor_SMD:R_1206_3216Metric, symbol Device:R_Small
- removed R7: 51.1 1%, Resistor_SMD:R_0805_2012Metric, symbol Device:R_Small
- removed U2: TPS24751RUVR, Custom Parts:VQFN-36, symbol Custom Parts:TPS24751RUVR
- added C7 (x2): 0.1uF 50V, Capacitor_SMD:C_0805_2012Metric, symbol Device:C_Small
- added Q6: PSMN014-80YL, Package_TO_SOT_SMD:LFPAK56, symbol Custom Parts:PSMN014-80YL
- added R17: 3m 1% 1/2W, Resistor_SMD:R_1206_3216Metric, symbol Device:R_Small
- added R18: 15k, Resistor_SMD:R_0805_2012Metric, symbol Device:R_Small
- added R19: 2k, Resistor_SMD:R_0805_2012Metric, symbol Device:R_Small
- added U5: LTC4229, Custom Parts:WFQFN-24, symbol Custom Parts:LTC4229
- R10: value 10k 1% -> 2k 1%
- R8: value 104k 1% -> 21.5k 1%
- R9: value 5.42k 1% -> 1.1k 1%
Connections:
- net GND: now also C7.2, C7.2, R19.2, U5.11 (~{EN}), U5.14 (DCFG), U5.15 (DOFF), U5.25 (GND), U5.7 (GND)
- net VIN: now also C7.1, D19.2 (A2), F1.2, R8.2, Q6.1 (S), Q6.2 (S), Q6.3 (S), U5.1 (DSRC), U5.4 (IN)
- net VOUT: now also Q6.1 (S), Q6.2 (S), Q6.3 (S), R18.1, U5.21 (OUT); no longer Q6.5 (D)
- net ~{FAULT}: now also U5.18 (~{FAULT})
- net ~{PGOOD}: now also U5.19 (~{PWRGD})
- net OVERVOLT_SENSE: now reaches R10.2, R9.1
- net OVERVOLT_SENSE: now also U5.13 (OV)
- net HOTSWAP_GATE: now reaches Q6.4 (G)
- net HOTSWAP_GATE: now also U5.22 (HGATE)
- net UNDERVOLT_SENSE: now reaches R8.1, R9.2
- net UNDERVOLT_SENSE: now also U5.12 (UV)
- new net: C7.1, U5.6 (INTVcc), U5.8 (DTMR)
- new net: C7.1, U5.10 (FTMR)
- new net DIODE_GATE: Q6.4 (G), U5.24 (DGATE)
- new net FOLDBACK_SENSE: R18.2, R19.1, U5.20 (FB)
- new net SENSE_N: Q6.5 (D), Q6.5 (D), R17.1, R17.2, U5.2 (SENSE_N), U5.3 (SENSE_P), U5.5 (DSNS)
Other:
- moved on the sheet: C10, C11, C23, C53, C7, C9, D6, F1, Q6, R10, R43, R44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
