File: epaper-hum-display/e-paper_display.kicad_sch (KiCad schematic)
At the start: 22 parts, among them Q1 Si1308EDL, Q2 PMV65XP,215

Commit message: WIP
Parts:
- added R1: 0, symbol Device:R_Small_US
Connections:
- net +3V3: now also R1.2; no longer Q2.2 (S), R1.2
- new net: Q2.2 (S), R1.1, R1.2
Changed lines of the file:
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@@
     (stroke (width 0) (type default))
   )
-  (wire (pts (xy 76.2 100.33) (xy 76.2 101.6))
+  (wire (pts (xy 76.2 96.52) (xy 76.2 101.6))
     (stroke (width 0) (type default))
   )
@@
   )
   (wire (pts (xy 180.975 120.015) (xy 180.975 124.46))
+    (stroke (width 0) (type default))
+  )
+  (wire (pts (xy 76.2 88.265) (xy 76.2 91.44))
     (stroke (width 0) (type default))
   )
@@
     )
   )
-  (symbol (lib_id "power:+3V3") (at 76.2 100.33 0) (unit 1)
+  (symbol (lib_id "power:+3V3") (at 76.2 88.265 0) (unit 1)
     (in_bom yes) (on_board yes) (dnp no)
-    (property "Reference" "#PWR05" (at 76.2 104.14 0)
-      (effects (font (size 1.27 1.27)) hide)
-    )
-    (property "Value" "+3V3" (at 76.2 95.885 0)
-      (effects (font (size 1.27 1.27)))
-    )
-    (property "Footprint" "" (at 76.2 100.33 0)
-      (effects (font (size 1.27 1.27)) hide)
-    )
-    (property "Datasheet" "" (at 76.2 100.33 0)
+    (property "Reference" "#PWR05" (at 76.2 92.075 0)
+      (effects (font (size 1.27 1.27)) hide)
+    )
+    (property "Value" "+3V3" (at 76.2 83.82 0)
+      (effects (font (size 1.27 1.27)))
+    )
+    (property "Footprint" "" (at 76.2 88.265 0)
+      (effects (font (size 1.27 1.27)) hide)
+    )
+    (property "Datasheet" "" (at 76.2 88.265 0)
       (effects (font (size 1.27 1.27)) hide)
     )
@@
         )
       )
+    )
+  )
+  (symbol (lib_id "Device:R_Small_US") (at 76.2 93.98 180) (unit 1)
+    (in_bom yes) (on_board yes) (dnp no) (fields_autoplaced)
+    (property "Reference" "R1" (at 77.851 92.7679 0)
+      (effects (font (size 1.27 1.27)) (justify right))
+    )
+    (property "Value" "0" (at 77.851 95.1921 0)
+      (effects (font (size 1.27 1.27)) (justify right))
+    )
+    (property "Footprint" "" (at 76.2 93.98 0)
+      (effects (font (size 1.27 1.27)) hide)
+    )
+    (property "Datasheet" "~" (at 76.2 93.98 0)
+      (effects (font (size 1.27 1.27)) hide)
+    )
+    (pin "1")
+    (pin "2")
+    (instances
+      (project "epaper-hum-display"
+        (path "/e8301e0c-f140-47c2-97ee-69a5a204efef"
+          (reference "R1") (unit 1)
+        )
+        (path "/e8301e0c-f140-47c2-97ee-69a5a204efef/3f5106e4-1b1e-45fa-91c4-dc93b9e9dbb4"
+          (reference "R28") (unit 1)
+        )
+      )

Commit message: WIP
Parts:
- C1, C10, C11, C12, C2, C3, C4, C5, C6, C7, C8, C9: footprint (none) -> Capacitor_SMD:C_0805_2012Metric
- D1, D2, D3: value MBR0530 -> MBR0530T1G; footprint (none) -> Custom:SOD-123W
- J1: symbol Custom:F31L-1A7H1-11024 -> Custom:WAVESHARE-2_13-E_Paper
- L1: value 68uH -> NLCV32T-680K-EF; footprint (none) -> Inductor_SMD:L_1210_3225Metric
- Q1, Q2: footprint (none) -> Custom:SOT-23-3
- R1, R2: footprint (none) -> Resistor_SMD:R_0805_2012Metric
Connections:
- net GND: now also J1.GND
Changed lines of the file:
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@@
       (effects (font (size 1.27 1.27)))
     )
-    (property "Footprint" "" (at 194.31 120.015 0)
+    (property "Footprint" "Capacitor_SMD:C_0805_2012Metric" (at 194.31 120.015 0)
       (effects (font (size 1.27 1.27)) hide)
     )
@@
     )
   )
-  (symbol (lib_id "Custom:F31L-1A7H1-11024") (at 225.425 90.805 0) (unit 1)
+  (symbol (lib_id "Custom:WAVESHARE-2_13-E_Paper") (at 225.425 90.805 0) (unit 1)
     (in_bom yes) (on_board yes) (dnp no)
     (property "Reference" "J1" (at 220.345 56.515 0)
@@
       (effects (font (size 1.27 1.27)))
     )
-    (property "Footprint" "Custom:F31L-1A7H1-11024" (at 220.345 76.835 0)
+    (property "Footprint" "Custom:F31L-1A7H1-11024" (at 225.425 55.245 0)
       (effects (font (size 1.27 1.27)) hide)
     )
@@
     (pin "8")
     (pin "9")
+    (pin "GND")
     (instances
       (project "epaper-hum-display"
@@
       (effects (font (size 1.27 1.27)) (justify left))
     )
-    (property "Value" "MBR0530" (at 154.305 106.045 90)
-      (effects (font (size 1.27 1.27)) (justify left))
-    )
-    (property "Footprint" "" (at 151.765 104.775 0)
+    (property "Value" "MBR0530T1G" (at 154.305 106.045 90)
+      (effects (font (size 1.27 1.27)) (justify left))
+    )
+    (property "Footprint" "Custom:SOD-123W" (at 151.765 104.775 0)
       (effects (font (size 1.27 1.27)) hide)
     )
@@
       (effects (font (size 1.27 1.27)))
     )
-    (property "Footprint" "" (at 185.42 112.395 0)
+    (property "Footprint" "Capacitor_SMD:C_0805_2012Metric" (at 185.42 112.395 0)
       (effects (font (size 1.27 1.27)) hide)
     )
@@
       (effects (font (size 1.27 1.27)))
     )
-    (property "Footprint" "" (at 69.215 101.6 0)
+    (property "Footprint" "Resistor_SMD:R_0805_2012Metric" (at 69.215 101.6 0)
       (effects (font (size 1.27 1.27)) hide)
     )
@@
       (effects (font (size 1.27 1.27)) (justify right))
     )
-    (property "Value" "MBR0530" (at 126.365 106.045 90)
+    (property "Value" "MBR0530T1G" (at 126.365 106.045 90)
       (effects (font (size 1.27 1.27)) (justify right))
     )
-    (property "Footprint" "" (at 123.825 104.775 0)
+    (property "Footprint" "Custom:SOD-123W" (at 123.825 104.775 0)
       (effects (font (size 1.27 1.27)) hide)
     )
@@
       (effects (font (size 1.27 1.27)))
     )
-    (property "Footprint" "" (at 145.415 99.06 0)
+    (property "Footprint" "Capacitor_SMD:C_0805_2012Metric" (at 145.415 99.06 0)
       (effects (font (size 1.27 1.27)) hide)
     )
@@
       (effects (font (size 1.27 1.27)))
     )
-    (property "Footprint" "" (at 194.31 104.775 0)
+    (property "Footprint" "Capacitor_SMD:C_0805_2012Metric" (at 194.31 104.775 0)
       (effects (font (size 1.27 1.27)) hide)
     )
@@
       (effects (font (size 1.27 1.27)))
     )
-    (property "Footprint" "" (at 185.42 107.315 0)
+    (property "Footprint" "Capacitor_SMD:C_0805_2012Metric" (at 185.42 107.315 0)
       (effects (font (size 1.27 1.27)) hide)
     )
@@
       (effects (font (size 1.27 1.27)))
     )
-    (property "Footprint" "" (at 185.42 71.755 0)
+    (property "Footprint" "Capacitor_SMD:C_0805_2012Metric" (at 185.42 71.755 0)
       (effects (font (size 1.27 1.27)) hide)
     )
@@
       (effects (font (size 1.27 1.27)) (justify left))
     )
-    (property "Value" "MBR0530" (at 139.7 106.045 90)
-      (effects (font (size 1.27 1.27)) (justify left))
-    )
-    (property "Footprint" "" (at 137.16 104.775 0)
+    (property "Value" "MBR0530T1G" (at 139.7 106.045 90)
+      (effects (font (size 1.27 1.27)) (justify left))
+    )
+    (property "Footprint" "Custom:SOD-123W" (at 137.16 104.775 0)
       (effects (font (size 1.27 1.27)) hide)
     )
@@
       (effects (font (size 1.27 1.27)))
     )
-    (property "Value" "68uH" (at 142.875 82.55 90)
-      (effects (font (size 1.27 1.27)))
-    )
-    (property "Footprint" "" (at 142.875 86.36 0)
+    (property "Value" "NLCV32T-680K-EF" (at 142.875 82.55 90)
+      (effects (font (size 1.27 1.27)))
+    )
+    (property "Footprint" "Inductor_SMD:L_1210_3225Metric" (at 142.875 86.36 0)
       (effects (font (size 1.27 1.27)) hide)
     )
@@
       (effects (font (size 1.27 1.27)))
     )
-    (property "Footprint" "" (at 194.31 109.855 0)
+    (property "Footprint" "Capacitor_SMD:C_0805_2012Metric" (at 194.31 109.855 0)
       (effects (font (size 1.27 1.27)) hide)
     )
@@
       (effects (font (size 1.27 1.27)))
     )
-    (property "Footprint" "" (at 185.42 117.475 0)
+    (property "Footprint" "Capacitor_SMD:C_0805_2012Metric" (at 185.42 117.475 0)
       (effects (font (size 1.27 1.27)) hide)
     )
@@
       (effects (font (size 1.27 1.27)))
     )
-    (property "Footprint" "" (at 194.31 114.935 0)
+    (property "Footprint" "Capacitor_SMD:C_0805_2012Metric" (at 194.31 114.935 0)
       (effects (font (size 1.27 1.27)) hide)
     )
@@
       (effects (font (size 1.27 1.27)) (justify left))
     )
-    (property "Footprint" "" (at 154.305 76.835 0)
+    (property "Footprint" "Custom:SOT-23-3" (at 154.305 76.835 0)
       (effects (font (size 1.27 1.27)) hide)
     )
@@
       (effects (font (size 1.27 1.27)))
     )
-    (property "Footprint" "" (at 185.42 97.155 0)
+    (property "Footprint" "Capacitor_SMD:C_0805_2012Metric" (at 185.42 97.155 0)
       (effects (font (size 1.27 1.27)) hide)
     )
@@
       (effects (font (size 1.27 1.27)) (justify right))
     )
-    (property "Footprint" "" (at 76.2 93.98 0)
+    (property "Footprint" "Resistor_SMD:R_0805_2012Metric" (at 76.2 93.98 0)
       (effects (font (size 1.27 1.27)) hide)
     )
@@
       (effects (font (size 1.27 1.27)))
     )
-    (property "Footprint" "" (at 123.19 86.36 0)
+    (property "Footprint" "Capacitor_SMD:C_0805_2012Metric" (at 123.19 86.36 0)
       (effects (font (size 1.27 1.27)) hide)
     )
@@
       (effects (font (size 1.27 1.27)))
     )
-    (property "Footprint" "" (at 127.635 74.295 0)
+    (property "Footprint" "Resistor_SMD:R_0805_2012Metric" (at 127.635 74.295 0)
       (effects (font (size 1.27 1.27)) hide)
     )
@@
       (effects (font (size 1.27 1.27)))
     )
-    (property "Footprint" "" (at 194.31 69.215 0)
+    (property "Footprint" "Capacitor_SMD:C_0805_2012Metric" (at 194.31 69.215 0)
       (effects (font (size 1.27 1.27)) hide)
     )
@@
       (effects (font (size 1.27 1.27)) (justify right))
     )
-    (property "Footprint" "" (at 151.765 62.23 0)
+    (property "Footprint" "Resistor_SMD:R_0805_2012Metric" (at 151.765 62.23 0)
       (effects (font (size 1.27 1.27)) hide)
     )
@@
       (effects (font (size 1.27 1.27)) (justify left))
     )
-    (property "Footprint" "" (at 78.74 111.125 0)
-      (effects (font (size 1.27 1.27)) hide)
-    )
+    (property "Footprint" "Custom:SOT-23-3" (at 78.74 111.125 0)
+      (effects (font (size 1.27 1.27)) hide)
+    )
