File: epaper-hum-display/epaper-hum-display.kicad_sch (KiCad schematic)
At the start: 2 parts, among them U1 STM32L011

Commit message: Add projects
Parts:
- added C1, C2, C6: 4.7uF 50V, symbol Device:C_Small
- added C10, C11, C12, C3, C4, C7, C8, C9: 1uF 16V, symbol Device:C_Small
- added C5: 0.1 uF 16V, symbol Device:C_Small
- added D1, D2, D3: MBR0530, symbol Device:D
- added L1: 68uH, symbol Device:L_Iron
- added Q1: Si1308EDL, symbol Simulation_SPICE:NMOS
- added R1: 10K, symbol Device:R_Small_US
- added R2: 3, symbol Device:R_Small_US
Connections:
- net RESET: now reaches J1.10 (RST)
- net DATA/COM_CTL: now reaches J1.11 (D/C)
- net EPAPER_CS: now reaches J1.12 (CS)
- net EPAPER_SCLK: now reaches J1.13 (SCLK)
- net EPAPER_SDI: now reaches J1.14 (SDI)
- net +3V3: now reaches J1.15 (VDDIO)
- net +3V3: now also J1.16 (VCI), C2.1, C5.1, L1.1
- net GND: now reaches J1.17 (VSS)
- net GND: now also C10.2, C11.2, C12.2, C2.2, C3.2, C4.2, C5.2, C6.2, C7.2, C8.2, C9.2, D1.1 (K), R1.1, R2.2
- net at J1.18 (VDD): now also C6.1
- net at J1.19 (VPP): now also C7.1
- net GDR: now reaches J1.2 (GDR)
- net GDR: now also Q1.2 (G), R1.2
- net PREVGH: now reaches J1.20 (VSH)
- net PREVGH: now also C8.1, D2.2 (A)
- net at J1.21 (PREVGH): now also C9.1
- net PREVGL: now reaches J1.22 (VSL)
- net PREVGL: now also C10.1, D3.2 (A)
- net at J1.23 (PREVGL): now also C11.1
- net at J1.24 (VCOM): now also C12.1
- net RESE: now reaches J1.3 (RESE)
- net RESE: now also Q1.3 (S), R2.1
- net at J1.4 (VGL): now also C3.1
- net at J1.5 (VGH): now also C4.1
- net BS: now reaches J1.8 (BS)
- net BUSY: now reaches J1.9 (BUSY)
- new net: C1.2, D3.1 (K), L1.2, Q1.1 (D)
- new net: C1.1, D1.2 (A), D2.1 (K)
Other:
- moved on the sheet: J1

Commit message: e-paper-hum-wip
Parts:
- removed C1, C2, C6: 4.7uF 50V, symbol Device:C_Small
- removed C10, C11, C12, C3, C4, C7, C8, C9: 1uF 16V, symbol Device:C_Small
- removed C5: 0.1 uF 16V, symbol Device:C_Small
- removed D1, D2, D3: MBR0530, symbol Device:D
- removed J1: ~, Custom:F31L-1A7H1-11024, symbol Custom:F31L-1A7H1-11024
- removed L1: 68uH, symbol Device:L_Iron
- removed Q1: Si1308EDL, symbol Simulation_SPICE:NMOS
- removed R1: 10K, symbol Device:R_Small_US
- removed R2: 3, symbol Device:R_Small_US
- added C37, C38, C39, C41: 0.1uF 10V, symbol Device:C_Small
- added C40: 1uF 10V, symbol Device:C_Small
- added D4: LED_RABG, symbol Device:LED_RABG
- added J2: TC2030-SWD, Custom:TC2030-IDC-FP, symbol Custom:TC2030-SWD
- added R15, R16, R17: 2.2k, symbol Device:R_Small
- added R18, R19, R7: 10k, symbol Device:R_Small
- added SW1: SW_Push, symbol Switch:SW_Push
- added U9: HDC3022, Custom Parts:WSON-8, symbol Custom:HDC3022
Connections:
- net GND: now also U1.12 (VSS), C37.2, C38.2, C39.2, C40.2, C41.2, J2.3 (GND), R18.2, R19.2, SW1.1, U9.2 (ADDR), U9.7 (ADDR1), U9.8 (GND)
- net HUM_ALERT: now reaches U1.1 (PC14/OSC32_IN)
- net HUM_ALERT: now also U9.3 (ALERT)
- net DISPLAY_MOSI: now reaches U1.10 (PA7)
- net ~{BATT_IRQ}: now reaches U1.11 (PB1)
- net +1V8: now reaches U1.13 (VDD)
- net +1V8: now also U1.4 (VDDA), C38.1, C39.1, C40.1, C41.1, J2.1 (VCC), R15.1, R16.1, R17.1, R7.1, U9.5 (VDD)
- net SWDIO: now reaches U1.16 (PA13)
- net SWDIO: now also J2.6 (SWDIO)
- net SWCLK: now reaches U1.17 (PA14)
- net SWCLK: now also J2.5 (SWDCLK)
- net I2C_SCL: now reaches U1.18 (PB6)
- net I2C_SCL: now also R15.2, U9.4 (SCL)
- net I2C_SDA: now reaches U1.19 (PB7)
- net I2C_SDA: now also R16.2, U9.1 (SDA)
- net HUM_RESET: now reaches U1.2 (PC15/OSC32_OUT)
- net HUM_RESET: now also R17.2, U9.6 (~{RESET})
- net at U1.20 (PB9/BOOT0): now also R18.1
- net nRESET: now reaches U1.3 (NRST)
- net nRESET: now also C37.1, J2.2 (nRESET), R7.2, SW1.2
- net 3V3_EN: now reaches U1.5 (PA0/CK_IN)
- net 3V3_EN: now also R19.1
- net DISPLAY_CS: now reaches U1.7 (PA4)
- net DISPLAY_SCLK: now reaches U1.8 (PA5)
Other:
- added sheet Battery (Battery.kicad_sch)
- added sheet E-Paper Display (e-paper_display.kicad_sch)
- moved on the sheet: U1

Commit message: WIP
Parts:
- removed C38: 0.1uF 10V, symbol Device:C_Small
- removed U1: STM32L011, Custom:UFQFPN-20, symbol Custom:STM32L011
- added R20, R21, R22: 500, symbol Device:R_Small
- added U1: STM32U575CIT, Custom:LQFP-48, symbol Custom:STM32U575CIT
Connections:
- net +1V8: now also U1.24 (VDD), U1.36 (VDD), U1.48 (VDD)
- net 3V3_EN: now also U1.10 (PA0)
- net DISPLAY_CS: now also U1.18 (PB0)
- net DISPLAY_MOSI: now also U1.41 (PB5)
- net DISPLAY_SCLK: now also U1.39 (PB3)
- net HUM_ALERT: now also U1.12 (PA2)
- net HUM_RESET: now also U1.11 (PA1)
- net I2C_SCL: now also U1.42 (PB6)
- net I2C_SDA: now also U1.43 (PB7)
- net SWCLK: now also U1.37 (PA14)
- net SWDIO: now also U1.34 (PA13)
- net nRESET: now also U1.7 (NRST)
- net ~{BATT_IRQ}: now also U1.45 (PB8)
- net at R18.1: now also U1.44 (PH3/BOOT0)
- net at D4.1 (RK): now also R20.1
- net +3V3: now reaches D4.2 (A)
- net at D4.3 (BK): now also R22.1
- net at D4.4 (GK): now also R21.1
- new net: U1.23 (VSS), U1.35 (VSS), U1.47 (VSS)
- new net CDSTOP: U1.16 (PA6)
- new net CSLEEP: U1.15 (PA5)
- new net IND_B: R22.2, U1.31 (PA10)
- new net IND_G: R21.2, U1.30 (PA9)
- new net IND_R: R20.2, U1.29 (PA8)
- new net SRDSTOP: U1.17 (PA7)
Other:
- moved on the sheet: C37, C39, C40, D4, R18, R7, SW1

Commit message: WIP
Parts:
- added C38, C42: 0.1uF 10V, symbol Device:C_Small
- added R23, R24, R25, R30: 10k, symbol Device:R_Small
- added R29, R31, R32: 0, symbol Device:R_Small
- added TP1, TP2, TP3: TestPoint, symbol Connector:TestPoint
- added U10: TCA9416DDF, Custom:SOT-23-8, symbol Custom:TCA9416DDF
- U1: value STM32U575CIT -> STM32U575CIT6Q
Connections:
- net +1V8: now also R29.1, R30.1, R31.2; no longer C39.1, C40.1, U1.24 (VDD), U1.36 (VDD), U1.48 (VDD)
- net +3V3: now also R23.1, R24.1, R25.1, R32.1
- net BATT_SCL: now also U10.1 (SCL_A)
- net BATT_SDA: now also U10.4 (SDA_A)
- net CDSTOP: now also TP2.1
- net CSLEEP: now also TP1.1
- net DISPLAY_BUSY: now also U1.26 (PB13)
- net DISPLAY_BUS_SEL: now also U1.25 (PB12), R25.2
- net DISPLAY_DATA_COMM_CTL: now also U1.28 (PB15)
- net DISPLAY_RESET: now also U1.27 (PB14), R23.2
- net GND: now also U1.23 (VSS), U1.35 (VSS), U1.47 (VSS), U1.8 (VSSA), C38.2, C42.2, U10.6 (GND)
- net HUM_RESET: now also R30.2
- net I2C_SCL: now also U10.8 (SCL_B)
- net I2C_SDA: now also U10.5 (SDA_B)
- net SRDSTOP: now also TP3.1
- net ~{BATT_IRQ}: now also R24.2
- net at U1.9 (VDDA): now also C39.1, C40.1, U1.24 (VDD), U1.36 (VDD), U1.48 (VDD), R29.2
- new net: C42.1, R31.1, U10.7 (VCCB)
- new net: C38.1, R32.2, U10.3 (VCCA)
Other:
- moved on the sheet: C37, J2, R19, R7, SW1

Commit message: WIP
Parts:
- added C43, C44, C46, C47, C48, C49: 0.1uF 10V, symbol Device:C_Small
- added C45: 4.7uF 10V, symbol Device:C_Small
- added R33, R34, R35: 0, symbol Device:R_Small
- added U11: TXU0104BQA, Custom:WQFN-14, symbol Custom:TXU0104BQA
- C40: value 1uF 10V -> 10uF 10V
Connections:
- net +1V8: now also R34.2
- net +3V3: now also R33.1
- net DISPLAY_CS: now also U11.2 (A1)
- net DISPLAY_DATA_COMM_CTL: now also U11.5 (A4)
- net DISPLAY_MOSI: now also U11.4 (A3)
- net DISPLAY_SCLK: now also U11.3 (A2)
- net GND: now also C43.2, C44.2, C45.1, C46.2, C47.2, C48.2, C49.2, R35.1, U11.15 (GND), U11.7 (NC)
- net at C39.1, C40.1, R29.2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: now also U1.1 (VBAT), C46.1, C47.1, C48.1, C49.1
- net at U1.22 (VCAP): now also C45.2
- new net: C43.1, R34.1, U11.1 (VCCA)
- new net: C44.1, R33.2, U11.14 (VCCB)
- new net DISPLAY_CS_S: U11.13 (B1Y)
- new net DISPLAY_DATA_COMM_CTL_S: U11.10 (B4Y)
- new net DISPLAY_LVL_OE: R35.2, U11.8 (OE)
- new net DISPLAY_MOSI_S: U11.12 (B2Y)
- new net DISPLAY_SCLK_S: U11.11 (B3Y)
Other:
- moved on the sheet: C37, C38, C39, C40, C41, C42, D4, J2, R15, R16, R17, R18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

Commit message: WIP
Parts:
- C37, C38, C39, C40, C41, C42, C43, C44, C45, C46, C47, C48, C49: footprint (none) -> Capacitor_SMD:C_0805_2012Metric
- D4: footprint (none) -> LED_SMD:LED_Cree-PLCC4_3.2x2.8mm_CCW
- R15, R16, R17, R18, R19, R20, R21, R22, R23, R24, R25, R29, R30, R31, R32, R33, R34, R35, R7: footprint (none) -> Resistor_SMD:R_0805_2012Metric
- SW1: value SW_Push -> B3F-1000; footprint (none) -> Button_Switch_THT:SW_PUSH_6mm
- TP1, TP2, TP3: footprint (none) -> TestPoint:TestPoint_Pad_D1.5mm
Other:
- moved on the sheet: SW1

Commit message: E Paper Hum WIP
Parts:
- added H1, H2, H3, H4: MountingHole_Pad, MountingHole:MountingHole_3.5mm_Pad_Via, symbol Mechanical:MountingHole_Pad
Connections:
- net GND: now also H1.1, H2.1, H3.1, H4.1
Changed lines of the file:
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@@
+    (stroke (width 0) (type default))
+  )
+  (wire (pts (xy 146.05 222.25) (xy 146.05 224.79))
     (stroke (width 0) (type default))
   )
@@
     (stroke (width 0) (type default))
   )
+  (wire (pts (xy 99.06 222.25) (xy 99.06 224.79))
+    (stroke (width 0) (type default))
+  )
   (wire (pts (xy 55.245 159.385) (xy 69.215 159.385))
     (stroke (width 0) (type default))
@@
     (stroke (width 0) (type default))
   )
+  (wire (pts (xy 122.555 222.25) (xy 122.555 224.79))
+    (stroke (width 0) (type default))
+  )
   (wire (pts (xy 222.885 132.715) (xy 222.885 136.525))
     (stroke (width 0) (type default))
@@
   )
   (wire (pts (xy 190.5 224.79) (xy 190.5 231.14))
+    (stroke (width 0) (type default))
+  )
+  (wire (pts (xy 72.39 222.25) (xy 72.39 224.155))
     (stroke (width 0) (type default))
   )
@@
     )
   )
+  (symbol (lib_id "Mechanical:MountingHole_Pad") (at 99.06 219.71 0) (unit 1)
+    (in_bom yes) (on_board yes) (dnp no) (fields_autoplaced)
+    (property "Reference" "H2" (at 101.6 217.2279 0)
+      (effects (font (size 1.27 1.27)) (justify left))
+    )
+    (property "Value" "MountingHole_Pad" (at 101.6 219.6521 0)
+      (effects (font (size 1.27 1.27)) (justify left))
+    )
+    (property "Footprint" "MountingHole:MountingHole_3.5mm_Pad_Via" (at 99.06 219.71 0)
+      (effects (font (size 1.27 1.27)) hide)
+    )
+    (property "Datasheet" "~" (at 99.06 219.71 0)
+      (effects (font (size 1.27 1.27)) hide)
+    )
+    (pin "1")
+    (instances
+      (project "epaper-hum-display"
+        (path "/e8301e0c-f140-47c2-97ee-69a5a204efef"
+          (reference "H2") (unit 1)
+        )
+      )
+    )
+  )
   (symbol (lib_id "power:+3V3") (at 278.13 161.925 0) (unit 1)
     (in_bom yes) (on_board yes) (dnp no) (fields_autoplaced)
@@
     )
   )
+  (symbol (lib_id "power:GND") (at 99.06 224.79 0) (mirror y) (unit 1)
+    (in_bom yes) (on_board yes) (dnp no) (fields_autoplaced)
+    (property "Reference" "#PWR055" (at 99.06 231.14 0)
+      (effects (font (size 1.27 1.27)) hide)
+    )
+    (property "Value" "GND" (at 99.06 228.9231 0)
+      (effects (font (size 1.27 1.27)))
+    )
+    (property "Footprint" "" (at 99.06 224.79 0)
+      (effects (font (size 1.27 1.27)) hide)
+    )
+    (property "Datasheet" "" (at 99.06 224.79 0)
+      (effects (font (size 1.27 1.27)) hide)
+    )
+    (pin "1")
+    (instances
+      (project "epaper-hum-display"
+        (path "/e8301e0c-f140-47c2-97ee-69a5a204efef"
+          (reference "#PWR055") (unit 1)
+        )
+      )
+    )
+  )
   (symbol (lib_id "Device:R_Small") (at 201.295 125.73 0) (unit 1)
     (in_bom yes) (on_board yes) (dnp no) (fields_autoplaced)
@@
         (path "/e8301e0c-f140-47c2-97ee-69a5a204efef"
           (reference "#PWR046") (unit 1)
+        )
+      )
+    )
+  )
+  (symbol (lib_id "Mechanical:MountingHole_Pad") (at 122.555 219.71 0) (unit 1)
+    (in_bom yes) (on_board yes) (dnp no) (fields_autoplaced)
+    (property "Reference" "H3" (at 125.095 217.2279 0)
+      (effects (font (size 1.27 1.27)) (justify left))
+    )
+    (property "Value" "MountingHole_Pad" (at 125.095 219.6521 0)
+      (effects (font (size 1.27 1.27)) (justify left))
+    )
+    (property "Footprint" "MountingHole:MountingHole_3.5mm_Pad_Via" (at 122.555 219.71 0)
+      (effects (font (size 1.27 1.27)) hide)
+    )
+    (property "Datasheet" "~" (at 122.555 219.71 0)
+      (effects (font (size 1.27 1.27)) hide)
+    )
+    (pin "1")
+    (instances
+      (project "epaper-hum-display"
+        (path "/e8301e0c-f140-47c2-97ee-69a5a204efef"
+          (reference "H3") (unit 1)
         )
       )
@@
         (path "/e8301e0c-f140-47c2-97ee-69a5a204efef"
           (reference "TP2") (unit 1)
+        )
+      )
+    )
+  )
+  (symbol (lib_id "power:GND") (at 122.555 224.79 0) (mirror y) (unit 1)
+    (in_bom yes) (on_board yes) (dnp no) (fields_autoplaced)
+    (property "Reference" "#PWR056" (at 122.555 231.14 0)
+      (effects (font (size 1.27 1.27)) hide)
+    )
+    (property "Value" "GND" (at 122.555 228.9231 0)
+      (effects (font (size 1.27 1.27)))
+    )
+    (property "Footprint" "" (at 122.555 224.79 0)
+      (effects (font (size 1.27 1.27)) hide)
+    )
+    (property "Datasheet" "" (at 122.555 224.79 0)
+      (effects (font (size 1.27 1.27)) hide)
+    )
+    (pin "1")
+    (instances
+      (project "epaper-hum-display"
+        (path "/e8301e0c-f140-47c2-97ee-69a5a204efef"
+          (reference "#PWR056") (unit 1)
         )
       )
@@
     )
   )
+  (symbol (lib_id "power:GND") (at 72.39 224.155 0) (mirror y) (unit 1)
+    (in_bom yes) (on_board yes) (dnp no) (fields_autoplaced)
+    (property "Reference" "#PWR054" (at 72.39 230.505 0)
+      (effects (font (size 1.27 1.27)) hide)
+    )
+    (property "Value" "GND" (at 72.39 228.2881 0)
+      (effects (font (size 1.27 1.27)))
+    )
+    (property "Footprint" "" (at 72.39 224.155 0)
+      (effects (font (size 1.27 1.27)) hide)
+    )
+    (property "Datasheet" "" (at 72.39 224.155 0)
+      (effects (font (size 1.27 1.27)) hide)
+    )
+    (pin "1")
+    (instances
+      (project "epaper-hum-display"
+        (path "/e8301e0c-f140-47c2-97ee-69a5a204efef"
+          (reference "#PWR054") (unit 1)
+        )
+      )
+    )
+  )
   (symbol (lib_id "Device:R_Small") (at 203.2 185.42 0) (mirror x) (unit 1)
     (in_bom yes) (on_board yes) (dnp no) (fields_autoplaced)
@@
     )
   )
+  (symbol (lib_id "power:GND") (at 146.05 224.79 0) (mirror y) (unit 1)
+    (in_bom yes) (on_board yes) (dnp no) (fields_autoplaced)
+    (property "Reference" "#PWR057" (at 146.05 231.14 0)
+      (effects (font (size 1.27 1.27)) hide)
+    )
+    (property "Value" "GND" (at 146.05 228.9231 0)
+      (effects (font (size 1.27 1.27)))
+    )
+    (property "Footprint" "" (at 146.05 224.79 0)
+      (effects (font (size 1.27 1.27)) hide)
+    )
+    (property "Datasheet" "" (at 146.05 224.79 0)
+      (effects (font (size 1.27 1.27)) hide)
+    )
+    (pin "1")
+    (instances
+      (project "epaper-hum-display"
+        (path "/e8301e0c-f140-47c2-97ee-69a5a204efef"
+          (reference "#PWR057") (unit 1)
+        )
+      )
+    )
+  )
   (symbol (lib_id "Device:R_Small") (at 332.105 163.195 0) (unit 1)
     (in_bom yes) (on_board yes) (dnp no) (fields_autoplaced)
@@
         (path "/e8301e0c-f140-47c2-97ee-69a5a204efef"
           (reference "R22") (unit 1)
+        )
+      )
+    )
+  )
+  (symbol (lib_id "Mechanical:MountingHole_Pad") (at 72.39 219.71 0) (unit 1)
+    (in_bom yes) (on_board yes) (dnp no) (fields_autoplaced)
+    (property "Reference" "H1" (at 74.93 217.2279 0)
+      (effects (font (size 1.27 1.27)) (justify left))
+    )
+    (property "Value" "MountingHole_Pad" (at 74.93 219.6521 0)
+      (effects (font (size 1.27 1.27)) (justify left))
+    )
+    (property "Footprint" "MountingHole:MountingHole_3.5mm_Pad_Via" (at 72.39 219.71 0)
+      (effects (font (size 1.27 1.27)) hide)
+    )
+    (property "Datasheet" "~" (at 72.39 219.71 0)
+      (effects (font (size 1.27 1.27)) hide)
+    )
+    (pin "1")
+    (instances
+      (project "epaper-hum-display"
+        (path "/e8301e0c-f140-47c2-97ee-69a5a204efef"
+          (reference "H1") (unit 1)
         )
       )
@@
         )
       )
+    )
+  )
+  (symbol (lib_id "Mechanical:MountingHole_Pad") (at 146.05 219.71 0) (unit 1)
+    (in_bom yes) (on_board yes) (dnp no) (fields_autoplaced)
+    (property "Reference" "H4" (at 148.59 217.2279 0)
+      (effects (font (size 1.27 1.27)) (justify left))
+    )
+    (property "Value" "MountingHole_Pad" (at 148.59 219.6521 0)
+      (effects (font (size 1.27 1.27)) (justify left))
+    )
+    (property "Footprint" "MountingHole:MountingHole_3.5mm_Pad_Via" (at 146.05 219.71 0)
+      (effects (font (size 1.27 1.27)) hide)
+    )
+    (property "Datasheet" "~" (at 146.05 219.71 0)
+      (effects (font (size 1.27 1.27)) hide)
+    )
+    (pin "1")
+    (instances
+      (project "epaper-hum-display"
+        (path "/e8301e0c-f140-47c2-97ee-69a5a204efef"
+          (reference "H4") (unit 1)
+        )
+      )

Commit message: Hum WIP
Connections:
- net DISPLAY_EN: now reaches U1.19 (PB1)
Changed lines of the file:
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@@
+    (stroke (width 0) (type default))
+  )
+  (wire (pts (xy 287.655 83.185) (xy 291.465 83.185))
     (stroke (width 0) (type default))
   )
@@
     (stroke (width 0) (type default))
   )
+  (wire (pts (xy 151.765 103.505) (xy 159.385 103.505))
+    (stroke (width 0) (type default))
+  )
   (wire (pts (xy 218.44 231.14) (xy 218.44 233.045))
     (stroke (width 0) (type default))
@@
     (effects (font (size 1.27 1.27)) (justify right bottom))
   )
+  (label "DISPLAY_EN" (at 159.385 103.505 0) (fields_autoplaced)
+    (effects (font (size 1.27 1.27)) (justify left bottom))
+  )
   (label "CSLEEP" (at 107.315 107.315 180) (fields_autoplaced)
     (effects (font (size 1.27 1.27)) (justify right bottom))
@@
     (effects (font (size 1.27 1.27)) (justify left bottom))
   )
+  (label "DISPLAY_EN" (at 287.655 83.185 180) (fields_autoplaced)
+    (effects (font (size 1.27 1.27)) (justify right bottom))
+  )
   (label "IND_R" (at 107.315 114.935 180) (fields_autoplaced)
