File: epaper-hum-display/Battery.kicad_sch (KiCad schematic)
At the start: 46 parts, among them J3 USB_C_Receptacle, Q2 PMV65XP,215, U2 TPS25750S, U3 BQ25798, U4 CDSOT23-0502B, U5 CDSOT23-0502B, U6 SISF00DN, U7 TPS7A2018PDBVR, U8 TPS7A2033PDBVR

Commit message: WIP
Parts:
- added R26, R27: 0, symbol Device:R_Small
Connections:
- net +3V3: now also R26.2, R27.1; no longer C17.2, Q2.2 (S), R13.1, R4.1, R5.1, R6.1, U2.32 (VIN_3V3)
- new net: Q2.2 (S), R13.1, R27.2
- new net PD_CTRLR_3V3: C17.2, R26.1, R4.1, R5.1, R6.1, U2.32 (VIN_3V3)
Changed lines of the file:
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@@
   (junction (at 424.815 65.405) (diameter 0) (color 0 0 0 0)
   )
+  (junction (at 391.795 103.505) (diameter 0) (color 0 0 0 0)
+  )
+  (junction (at 439.42 65.405) (diameter 0) (color 0 0 0 0)
+  )
+  (junction (at 200.025 55.245) (diameter 0) (color 0 0 0 0)
+  )
+  (junction (at 127 93.98) (diameter 0) (color 0 0 0 0)
+  )
+  (junction (at 290.83 73.025) (diameter 0) (color 0 0 0 0)
+  )
+  (junction (at 396.875 75.565) (diameter 0) (color 0 0 0 0)
+  )
+  (junction (at 354.33 65.405) (diameter 0) (color 0 0 0 0)
+  )
+  (junction (at 363.22 81.915) (diameter 0) (color 0 0 0 0)
+  )
+  (junction (at 368.935 75.565) (diameter 0) (color 0 0 0 0)
+  )
+  (junction (at 74.93 69.215) (diameter 0) (color 0 0 0 0)
+  )
+  (junction (at 290.83 62.865) (diameter 0) (color 0 0 0 0)
+  )
+  (junction (at 443.23 65.405) (diameter 0) (color 0 0 0 0)
+  )
+  (junction (at 132.08 41.91) (diameter 0) (color 0 0 0 0)
+  )
+  (junction (at 462.28 79.375) (diameter 0) (color 0 0 0 0)
+  )
+  (junction (at 451.485 111.76) (diameter 0) (color 0 0 0 0)
+  )
+  (junction (at 377.825 103.505) (diameter 0) (color 0 0 0 0)
+  )
+  (junction (at 377.825 81.915) (diameter 0) (color 0 0 0 0)
+  )
+  (junction (at 439.42 97.79) (diameter 0) (color 0 0 0 0)
+  )
+  (junction (at 222.885 93.345) (diameter 0) (color 0 0 0 0)
+  )
+  (junction (at 382.905 75.565) (diameter 0) (color 0 0 0 0)
+  )
+  (junction (at 264.795 45.085) (diameter 0) (color 0 0 0 0)
+  )
+  (junction (at 107.315 64.135) (diameter 0) (color 0 0 0 0)
+  )
+  (junction (at 208.28 55.245) (diameter 0) (color 0 0 0 0)
+  )
+  (junction (at 424.815 75.565) (diameter 0) (color 0 0 0 0)
+  )
+  (junction (at 151.765 47.625) (diameter 0) (color 0 0 0 0)
+  )
+  (junction (at 391.795 81.915) (diameter 0) (color 0 0 0 0)
+  )
+  (junction (at 294.64 41.275) (diameter 0) (color 0 0 0 0)
+  )
+  (junction (at 452.755 65.405) (diameter 0) (color 0 0 0 0)
+  )
+  (junction (at 65.405 69.215) (diameter 0) (color 0 0 0 0)
+  )
+  (junction (at 359.41 43.815) (diameter 0) (color 0 0 0 0)
+  )
+  (junction (at 237.49 45.085) (diameter 0) (color 0 0 0 0)
+  )
+  (junction (at 65.405 74.295) (diameter 0) (color 0 0 0 0)
+  )
+  (junction (at 100.965 61.595) (diameter 0) (color 0 0 0 0)
+  )
+  (junction (at 381 49.53) (diameter 0) (color 0 0 0 0)
+  )
+  (junction (at 363.22 103.505) (diameter 0) (color 0 0 0 0)
+  )
   (junction (at 222.885 55.245) (diameter 0) (color 0 0 0 0)
   )
-  (junction (at 391.795 103.505) (diameter 0) (color 0 0 0 0)
-  )
-  (junction (at 439.42 65.405) (diameter 0) (color 0 0 0 0)
-  )
-  (junction (at 200.025 55.245) (diameter 0) (color 0 0 0 0)
-  )
-  (junction (at 127 93.98) (diameter 0) (color 0 0 0 0)
-  )
-  (junction (at 290.83 73.025) (diameter 0) (color 0 0 0 0)
-  )
-  (junction (at 396.875 75.565) (diameter 0) (color 0 0 0 0)
-  )
-  (junction (at 354.33 65.405) (diameter 0) (color 0 0 0 0)
-  )
-  (junction (at 363.22 81.915) (diameter 0) (color 0 0 0 0)
-  )
-  (junction (at 237.49 45.085) (diameter 0) (color 0 0 0 0)
-  )
-  (junction (at 368.935 75.565) (diameter 0) (color 0 0 0 0)
-  )
-  (junction (at 74.93 69.215) (diameter 0) (color 0 0 0 0)
-  )
-  (junction (at 290.83 62.865) (diameter 0) (color 0 0 0 0)
-  )
-  (junction (at 443.23 65.405) (diameter 0) (color 0 0 0 0)
-  )
-  (junction (at 132.08 41.91) (diameter 0) (color 0 0 0 0)
-  )
-  (junction (at 462.28 79.375) (diameter 0) (color 0 0 0 0)
-  )
-  (junction (at 451.485 111.76) (diameter 0) (color 0 0 0 0)
-  )
-  (junction (at 377.825 103.505) (diameter 0) (color 0 0 0 0)
-  )
-  (junction (at 377.825 81.915) (diameter 0) (color 0 0 0 0)
-  )
-  (junction (at 439.42 97.79) (diameter 0) (color 0 0 0 0)
-  )
-  (junction (at 222.885 93.345) (diameter 0) (color 0 0 0 0)
-  )
-  (junction (at 382.905 75.565) (diameter 0) (color 0 0 0 0)
-  )
-  (junction (at 107.315 64.135) (diameter 0) (color 0 0 0 0)
-  )
-  (junction (at 208.28 55.245) (diameter 0) (color 0 0 0 0)
-  )
-  (junction (at 424.815 75.565) (diameter 0) (color 0 0 0 0)
-  )
-  (junction (at 151.765 47.625) (diameter 0) (color 0 0 0 0)
-  )
-  (junction (at 391.795 81.915) (diameter 0) (color 0 0 0 0)
-  )
-  (junction (at 294.64 41.275) (diameter 0) (color 0 0 0 0)
-  )
-  (junction (at 452.755 65.405) (diameter 0) (color 0 0 0 0)
-  )
-  (junction (at 264.795 45.085) (diameter 0) (color 0 0 0 0)
-  )
-  (junction (at 65.405 69.215) (diameter 0) (color 0 0 0 0)
-  )
-  (junction (at 359.41 43.815) (diameter 0) (color 0 0 0 0)
-  )
-  (junction (at 65.405 74.295) (diameter 0) (color 0 0 0 0)
-  )
-  (junction (at 100.965 61.595) (diameter 0) (color 0 0 0 0)
-  )
-  (junction (at 381 49.53) (diameter 0) (color 0 0 0 0)
-  )
-  (junction (at 363.22 103.505) (diameter 0) (color 0 0 0 0)
-  )
   (wire (pts (xy 134.62 81.28) (xy 134.62 78.105))
     (stroke (width 0) (type default))
@@
     (stroke (width 0) (type default))
   )
-  (wire (pts (xy 237.49 55.245) (xy 237.49 45.085))
-    (stroke (width 0) (type default))
-  )
   (wire (pts (xy 348.615 103.505) (xy 363.22 103.505))
     (stroke (width 0) (type default))
@@
     (stroke (width 0) (type default))
   )
+  (wire (pts (xy 222.885 55.245) (xy 228.6 55.245))
+    (stroke (width 0) (type default))
+  )
   (wire (pts (xy 452.755 65.405) (xy 454.66 65.405))
     (stroke (width 0) (type default))
@@
     (stroke (width 0) (type default))
   )
+  (wire (pts (xy 253.365 45.085) (xy 264.795 45.085))
+    (stroke (width 0) (type default))
+  )
   (wire (pts (xy 222.885 55.245) (xy 215.9 55.245))
     (stroke (width 0) (type default))
@@
     (stroke (width 0) (type default))
   )
+  (wire (pts (xy 233.68 55.245) (xy 237.49 55.245))
+    (stroke (width 0) (type default))
+  )
   (wire (pts (xy 363.22 103.505) (xy 377.825 103.505))
     (stroke (width 0) (type default))
@@
     (stroke (width 0) (type default))
   )
-  (wire (pts (xy 237.49 45.085) (xy 264.795 45.085))
-    (stroke (width 0) (type default))
-  )
   (wire (pts (xy 327.66 103.505) (xy 348.615 103.505))
     (stroke (width 0) (type default))
@@
     (stroke (width 0) (type default))
   )
-  (wire (pts (xy 222.885 55.245) (xy 237.49 55.245))
-    (stroke (width 0) (type default))
-  )
   (wire (pts (xy 439.42 97.79) (xy 439.42 65.405))
     (stroke (width 0) (type default))
@@
     (stroke (width 0) (type default))
   )
+  (wire (pts (xy 237.49 45.085) (xy 237.49 55.245))
+    (stroke (width 0) (type default))
+  )
   (wire (pts (xy 160.655 27.94) (xy 160.655 35.56))
     (stroke (width 0) (type default))
@@
     (stroke (width 0) (type default))
   )
+  (wire (pts (xy 237.49 45.085) (xy 248.285 45.085))
+    (stroke (width 0) (type default))
+  )
   (wire (pts (xy 191.135 55.245) (xy 200.025 55.245))
     (stroke (width 0) (type default))
@@
     (stroke (width 0) (type default))
   )
-  (wire (pts (xy 237.49 45.085) (xy 237.49 38.1))
+  (wire (pts (xy 237.49 38.1) (xy 237.49 45.085))
     (stroke (width 0) (type default))
   )
@@
         )
       )
+    )
+  )
+  (symbol (lib_id "Device:R_Small") (at 231.14 55.245 90) (unit 1)
+    (in_bom yes) (on_board yes) (dnp no) (fields_autoplaced)
+    (property "Reference" "R26" (at 231.14 50.3641 90)
+      (effects (font (size 1.27 1.27)))
+    )
+    (property "Value" "0" (at 231.14 52.7883 90)
+      (effects (font (size 1.27 1.27)))
+    )
+    (property "Footprint" "" (at 231.14 55.245 0)
+      (effects (font (size 1.27 1.27)) hide)
+    )
+    (property "Datasheet" "~" (at 231.14 55.245 0)
+      (effects (font (size 1.27 1.27)) hide)
+    )
+    (pin "1")
+    (pin "2")
+    (instances
+      (project "epaper-hum-display"
+        (path "/e8301e0c-f140-47c2-97ee-69a5a204efef/0e2f7551-c5c5-4ce9-b1ee-dbdaa7ffe02b"
+          (reference "R26") (unit 1)
+        )
+      )
+    )
+  )
+  (symbol (lib_id "Device:R_Small") (at 250.825 45.085 90) (unit 1)
+    (in_bom yes) (on_board yes) (dnp no) (fields_autoplaced)
+    (property "Reference" "R27" (at 250.825 40.2041 90)
+      (effects (font (size 1.27 1.27)))
+    )
+    (property "Value" "0" (at 250.825 42.6283 90)
+      (effects (font (size 1.27 1.27)))
+    )
+    (property "Footprint" "" (at 250.825 45.085 0)
+      (effects (font (size 1.27 1.27)) hide)
+    )
+    (property "Datasheet" "~" (at 250.825 45.085 0)
+      (effects (font (size 1.27 1.27)) hide)
+    )
+    (pin "1")
+    (pin "2")
+    (instances
+      (project "epaper-hum-display"
+        (path "/e8301e0c-f140-47c2-97ee-69a5a204efef/0e2f7551-c5c5-4ce9-b1ee-dbdaa7ffe02b"
+          (reference "R27") (unit 1)
+        )
+      )

Commit message: WIP
Parts:
- BT1: footprint (none) -> Custom:KEYSTONE-1043
- C13, C14, C15, C16, C17, C18, C19, C20, C21, C22, C23, C24, C25, C26, C27, C28, C29, C30, C31, C32, C33, C34, C35, C36: footprint (none) -> Capacitor_SMD:C_0805_2012Metric
- D5: footprint (none) -> LED_SMD:LED_0805_2012Metric
- J3: footprint (none) -> Custom:Wurth_632723300011
- L2: value 1uH 6A -> SRP0315-1R0K; footprint (none) -> Custom:SRP0315
- Q2: footprint (none) -> Custom:SOT-23-3
- R10, R11, R12, R13, R14, R26, R27, R4, R5, R6, R8, R9: footprint (none) -> Resistor_SMD:R_0805_2012Metric
Connections:
- net GND: now also U2.33 (GND)

Commit message: WIP
Parts:
- added R36, R37: 0, Resistor_SMD:R_0805_2012Metric, symbol Device:R_Small
Connections:
- net VSYS: now also R36.2, R37.2; no longer C33.1, C35.1, U7.1 (IN), U7.3 (EN), U8.1 (IN)
- new net: C35.1, R37.1, U8.1 (IN)
- new net: C33.1, R36.1, U7.1 (IN), U7.3 (EN)
Other:
- moved on the sheet: C33, C34, C35, C36, R14, U7, U8

Commit message: E Paper Hum Layout Complete
Parts:
- added F1: Fuse, Custom:01550900M, symbol Device:Fuse
Connections:
- net at C22.1, C23.1, C24.1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: now also F1.1; no longer BT1.1 (+)
- new net: BT1.1 (+), F1.2
Other:
- moved on the sheet: BT1
Changed lines of the file:
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@@
+    (stroke (width 0) (type default))
+  )
+  (wire (pts (xy 417.195 81.915) (xy 417.195 88.9))
     (stroke (width 0) (type default))
   )
@@
     (stroke (width 0) (type default))
   )
-  (wire (pts (xy 406.4 81.915) (xy 406.4 88.9))
-    (stroke (width 0) (type default))
-  )
   (wire (pts (xy 191.135 90.805) (xy 215.9 90.805))
     (stroke (width 0) (type default))
@@
     (stroke (width 0) (type default))
   )
-  (wire (pts (xy 406.4 103.505) (xy 406.4 96.52))
+  (wire (pts (xy 417.195 103.505) (xy 417.195 96.52))
     (stroke (width 0) (type default))
   )
@@
     (stroke (width 0) (type default))
   )
+  (wire (pts (xy 407.67 81.915) (xy 417.195 81.915))
+    (stroke (width 0) (type default))
+  )
   (wire (pts (xy 353.695 50.165) (xy 359.41 50.165))
     (stroke (width 0) (type default))
@@
     (stroke (width 0) (type default))
   )
-  (wire (pts (xy 391.795 81.915) (xy 406.4 81.915))
+  (wire (pts (xy 391.795 81.915) (xy 400.05 81.915))
     (stroke (width 0) (type default))
   )
@@
     (stroke (width 0) (type default))
   )
-  (wire (pts (xy 391.795 103.505) (xy 406.4 103.505))
+  (wire (pts (xy 391.795 103.505) (xy 417.195 103.505))
     (stroke (width 0) (type default))
   )
@@
         (path "/e8301e0c-f140-47c2-97ee-69a5a204efef/0e2f7551-c5c5-4ce9-b1ee-dbdaa7ffe02b"
           (reference "R37") (unit 1)
+        )
+      )
+    )
+  )
+  (symbol (lib_id "Device:Fuse") (at 403.86 81.915 90) (unit 1)
+    (in_bom yes) (on_board yes) (dnp no) (fields_autoplaced)
+    (property "Reference" "F1" (at 403.86 77.0087 90)
+      (effects (font (size 1.27 1.27)))
+    )
+    (property "Value" "Fuse" (at 403.86 79.4329 90)
+      (effects (font (size 1.27 1.27)))
+    )
+    (property "Footprint" "Custom:01550900M" (at 403.86 83.693 90)
+      (effects (font (size 1.27 1.27)) hide)
+    )
+    (property "Datasheet" "~" (at 403.86 81.915 0)
+      (effects (font (size 1.27 1.27)) hide)
+    )
+    (pin "1")
+    (pin "2")
+    (instances
+      (project "epaper-hum-display"
+        (path "/e8301e0c-f140-47c2-97ee-69a5a204efef/0e2f7551-c5c5-4ce9-b1ee-dbdaa7ffe02b"
+          (reference "F1") (unit 1)
         )
       )
@@
     )
   )
-  (symbol (lib_id "Device:Battery_Cell") (at 406.4 93.98 0) (unit 1)
-    (in_bom yes) (on_board yes) (dnp no) (fields_autoplaced)
-    (property "Reference" "BT1" (at 409.321 90.9264 0)
-      (effects (font (size 1.27 1.27)) (justify left))
-    )
-    (property "Value" "Battery_Cell" (at 409.321 93.3506 0)
-      (effects (font (size 1.27 1.27)) (justify left))
-    )
-    (property "Footprint" "Custom:KEYSTONE-1043" (at 406.4 92.456 90)
-      (effects (font (size 1.27 1.27)) hide)
-    )
-    (property "Datasheet" "~" (at 406.4 92.456 90)
-      (effects (font (size 1.27 1.27)) hide)
-    )
+  (symbol (lib_id "Device:Battery_Cell") (at 417.195 93.98 0) (unit 1)
+    (in_bom yes) (on_board yes) (dnp no) (fields_autoplaced)
+    (property "Reference" "BT1" (at 420.116 90.9264 0)
+      (effects (font (size 1.27 1.27)) (justify left))
+    )
+    (property "Value" "Battery_Cell" (at 420.116 93.3506 0)
+      (effects (font (size 1.27 1.27)) (justify left))
+    )
+    (property "Footprint" "Custom:KEYSTONE-1043" (at 417.195 92.456 90)
+      (effects (font (size 1.27 1.27)) hide)
+    )
+    (property "Datasheet" "~" (at 417.195 92.456 90)
+      (effects (font (size 1.27 1.27)) hide)
+    )
