File: epaper-hum-display/epaper-hum-display.kicad_pcb (KiCad board)
At the start: 2 copper layers, 113 parts, among them J2 TC2030-SWD, J3 USB_C_Receptacle, Q1 Si1308EDL, Q2 PMV65XP,215, Q4 PMV65XP,215, SW1 B3F-1000, U1 STM32U575CIT6Q, U10 TCA9416DDF, U11 TXU0104BQA, U2 TPS25750S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

Commit message: WIP
Parts:
- added R36: 0, Resistor_SMD:R_0805_2012Metric, F.Cu at (103.3, 53.1)
- added R37: 0, Resistor_SMD:R_0805_2012Metric, F.Cu at (101.5, 66.0)
- BT1: moved to B.Cu
- moved C3 91.7 mm to (142.1, 41.5)
- moved J1 89.0 mm to (146.2, 29.7), turned to 90 degrees
- moved R7 88.0 mm to (98.1, 116.9)
- moved R20 88.0 mm to (110.6, 107.9)
- moved C2 83.0 mm to (132.8, 39.8)
- moved C6 82.9 mm to (137.2, 39.8)
- moved SW1 80.9 mm to (101.8, 115.2)
- moved C37 79.7 mm to (98.2, 120.2)
- moved L1 79.6 mm to (131.0, 28.0)
- moved R22 79.0 mm to (97.5, 111.1)
- moved R21 78.4 mm to (97.1, 107.7)
- moved R25 78.2 mm to (107.8, 88.9)
- moved C11 77.5 mm to (116.5, 21.5)
- moved R28 76.7 mm to (137.6, 43.5)
- moved C12 76.6 mm to (132.9, 43.6)
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Connections:
- C33 pad 1: /Battery/VSYS -> Net-(U7-EN)
- C35 pad 1: /Battery/VSYS -> Net-(U8-IN)
- U7 pad 1: /Battery/VSYS -> Net-(U7-EN)
- U7 pad 3: /Battery/VSYS -> Net-(U7-EN)
- U8 pad 1: /Battery/VSYS -> Net-(U8-IN)

Commit message: E Paper Hum WIP
Parts:
- added H1: MountingHole_Pad, MountingHole:MountingHole_3.5mm_Pad_Via, F.Cu at (111.0, 24.0)
- added H2: MountingHole_Pad, MountingHole:MountingHole_3.5mm_Pad_Via, F.Cu at (24.0, 24.0)
- added H3: MountingHole_Pad, MountingHole:MountingHole_3.5mm_Pad_Via, F.Cu at (111.0, 56.0)
- added H4: MountingHole_Pad, MountingHole:MountingHole_3.5mm_Pad_Via, F.Cu at (24.0, 56.0)
- moved R33 104.3 mm to (92.1, 22.0), turned to 180 degrees
- moved C43 98.7 mm to (88.4, 22.0), turned to 180 degrees
- moved R34 93.9 mm to (88.4, 24.1), turned to 180 degrees
- moved R35 93.5 mm to (90.1, 30.4)
- moved U11 90.9 mm to (90.2, 27.2)
- moved C44 90.7 mm to (92.1, 24.1)
- moved R20 82.4 mm to (48.0, 54.3)
- moved TP3 80.6 mm to (70.2, 44.7), turned to -90 degrees
- moved D4 77.3 mm to (47.6, 57.1)
- moved R17 77.2 mm to (85.3, 38.4), turned to 90 degrees
- moved TP2 75.7 mm to (73.8, 44.7), turned to -90 degrees
- moved C46 74.9 mm to (59.2, 47.3), turned to -90 degrees
- moved C40 72.8 mm to (50.8, 47.3), turned to -90 degrees
- moved C45 71.3 mm to (64.9, 44.9), turned to -90 degrees
- moved TP1 70.7 mm to (77.3, 44.7), turned to -90 degrees
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Other:
- board outline added: 95 x 40 mm
- copper layers 2 -> 4

Commit message: WIP
Parts:
- moved U5 13.8 mm to (24.8, 39.7)
- moved R29 13.2 mm to (61.3, 43.7), turned to -90 degrees
- moved U4 7.76 mm to (36.9, 37.7)
- moved R36 6.70 mm to (67.2, 30.8)
- moved C33 6.70 mm to (70.1, 31.6)
- moved C22 5.73 mm to (62.3, 33.0), turned to -90 degrees
- moved R7 5.07 mm to (87.2, 57.0), turned to -90 degrees
- moved U6 4.71 mm to (40.4, 47.2)
- moved C15 4.71 mm to (37.3, 45.3)
- moved C16 4.71 mm to (35.2, 45.3)
- moved C43 4.39 mm to (84.5, 24.1)
- moved R34 4.39 mm to (84.5, 26.2)
- moved R33 4.39 mm to (88.2, 24.1)
- moved R35 4.39 mm to (86.2, 32.5)
- moved U11 4.39 mm to (86.4, 29.3)
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Routing:
- net +3V3: track 0.00 -> 179.4 mm
- net +1V8: track 0.00 -> 116.6 mm
- net /~{BATT_IRQ}: track 0.00 -> 64.5 mm, vias 0 -> 2
- net /Battery/~{BQ_I2C_IRQ}: track 0.00 -> 45.3 mm, vias 0 -> 2
- net Net-(BT1-+): track 0.00 -> 40.9 mm, vias 0 -> 11
- net /nRESET: track 0.00 -> 35.9 mm
- net /Battery/CC1: track 0.00 -> 33.6 mm, vias 0 -> 2
- net /Battery/CC2: track 0.00 -> 30.5 mm, vias 0 -> 1
- net /Battery/BQ_I2C_SDA: track 0.00 -> 29.6 mm, vias 0 -> 2
- net /Battery/BQ_I2C_SCL: track 0.00 -> 27.3 mm, vias 0 -> 2
- net Net-(U2-GATE_VBUS): track 0.00 -> 25.3 mm, vias 0 -> 2
- net /Battery/VBUS: track 0.00 -> 24.1 mm, vias 0 -> 2
- net /E-Paper Display/EPAPER_3V3: track 0.00 -> 22.2 mm
- net Net-(U2-GATE_VSYS): track 0.00 -> 20.7 mm, vias 0 -> 2
- net /Battery/USB_P: track 0.00 -> 19.9 mm
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- added copper zone on F.Cu, net /Battery/VBUS
- added copper zone on F.Cu, net /Battery/VSYS
- added copper zone on F.Cu, net /E-Paper Display/EPAPER_3V3
- added copper zone on B.Cu, net GND
- added copper zone on F.Cu, net GND
- added copper zone on In1.Cu, net GND
- added copper zone on In2.Cu, net GND
- added copper zone on B.Cu, net Net-(BT1-+)
- added copper zone on F.Cu, net Net-(BT1-+)
- added copper zone on F.Cu, net Net-(D3-K)
- added copper zone on F.Cu, net Net-(U1-VBAT)
- added copper zone on F.Cu, net Net-(U3-PMID)
- added copper zone on B.Cu, net Net-(U3-SW1)
- added copper zone on F.Cu, net Net-(U3-SW1)
- added copper zone on B.Cu, net Net-(U3-SW2)
- added copper zone on F.Cu, net Net-(U3-SW2)
- added copper zone on F.Cu, net Net-(U3-VAC1)

Commit message: Hum WIP
Parts:
- moved TP1 3.73 mm to (73.6, 44.5)
- moved TP2 2.91 mm to (70.9, 44.5)
- moved TP3 2.07 mm to (68.2, 44.5)
- moved R23 0.55 mm to (56.4, 52.1)
- moved R25 0.55 mm to (56.4, 50.2)
- turned R30 to 180 degrees
Connections:
- Q2 pad 1: /E-Paper Display/ENABLE -> /DISPLAY_EN
- R3 pad 1: /E-Paper Display/ENABLE -> /DISPLAY_EN
- U1 pad 19: unconnected-(U1-PB1-Pad19) -> /DISPLAY_EN
Routing:
- net /I2C_SDA: track 5.72 -> 88.2 mm, vias 0 -> 3
- net /I2C_SCL: track 2.37 -> 84.0 mm, vias 0 -> 3
- net /DISPLAY_MOSI: track 0.00 -> 72.1 mm, vias 0 -> 2
- net /DISPLAY_RESET: track 5.40 -> 77.2 mm, vias 0 -> 2
- net /DISPLAY_BUSY: track 0.00 -> 69.8 mm, vias 0 -> 2
- net /DISPLAY_SCLK: track 0.00 -> 69.6 mm, vias 0 -> 2
- net /DISPLAY_BUS_SEL: track 4.78 -> 71.6 mm, vias 0 -> 2
- net /E-Paper Display/PREVGL: track 11.0 -> 60.6 mm, vias 0 -> 2
- net /3V3_EN: track 4.38 -> 50.1 mm, vias 0 -> 2
- net /E-Paper Display/PREVGH: track 14.8 -> 56.7 mm, vias 0 -> 2
- net /DISPLAY_DATA_COMM_CTL: track 1.71 -> 42.6 mm, vias 1 -> 2
- net /DISPLAY_EN: track 0.00 -> 37.9 mm, vias 0 -> 2
- net /SWCLK: track 0.00 -> 35.4 mm, vias 0 -> 2
- net /BATT_SDA: track 0.82 -> 34.2 mm, vias 1 -> 2
- net /DISPLAY_CS: track 0.00 -> 32.4 mm, vias 0 -> 2
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
Commit message: E Paper Hum Layout Complete
Parts:
- added F1: Fuse, Custom:01550900M, F.Cu at (60.2, 37.9)
- moved C21 4.19 mm to (51.1, 41.4), turned to 180 degrees
- moved R24 1.05 mm to (58.2, 58.0)
- moved C23 0.60 mm to (59.6, 33.0)
- moved C24 0.60 mm to (57.5, 33.0)
- moved C22 0.60 mm to (61.7, 33.0)
- moved R9 0.50 mm to (55.5, 33.0)
Connections:
- C22 pad 1: Net-(BT1-+) -> Net-(C22-Pad1)
- C23 pad 1: Net-(BT1-+) -> Net-(C22-Pad1)
- C24 pad 1: Net-(BT1-+) -> Net-(C22-Pad1)
- R9 pad 1: Net-(BT1-+) -> Net-(C22-Pad1)
- U3 pad 22: Net-(BT1-+) -> Net-(C22-Pad1)
- U3 pad 23: Net-(BT1-+) -> Net-(C22-Pad1)
Routing:
- net Net-(BT1-+): track 40.0 -> 25.1 mm, vias 11 -> 9
- net Net-(U3-SDRV): track 9.05 -> 13.5 mm
- net /3V3_EN: track 50.1 -> 52.5 mm
- net +3V3: track 179.2 -> 177.3 mm
- net /Battery/~{BQ_I2C_IRQ}: track 45.3 -> 43.8 mm
- net Net-(U3-BTST1): track 10.1 -> 11.5 mm
- net Net-(U1-PH3/BOOT0): track 10.1 -> 8.98 mm
- net /DISPLAY_MOSI: track 72.1 -> 71.2 mm
- net GND: vias 249 -> 297
- added copper zone on F.Cu, net Net-(C22-Pad1)
Other:
- board text added: "E-Paper Humidity Display"
- board text added: "V1"
